File: input/input_board_rear.kicad_pcb (KiCad board)
At the start: 4 copper layers, 191 parts, among them J1 Sensor, J101 Gain, J2 C64AB, J3 Decimate, Q1 NSS1C300ET4G, Q2 2STD1665T4, Q3 NSS1C300ET4G, U1 FIN1048, U101 AD8599, U102 LTC2512-24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

Commit message: Progress on input board layout.  Have adopted 100x280mm eurocard format with connector at the back. Schematic changes are mostly cosmetic.  The working board file is now input/input_board_rear.kicad_pcb
Parts:
- moved U9 139.1 mm to (280.2, 142.7)
- moved C28 139.1 mm to (273.8, 142.7)
- moved C27 139.1 mm to (286.5, 142.7)
- moved J2 137.7 mm to (299.5, 60.5), turned to 270 degrees
- moved C101 127.7 mm to (160.2, 61.6)
- moved C109 127.7 mm to (167.8, 66.4)
- moved FB105 127.7 mm to (175.7, 70.8)
- moved R101 127.7 mm to (160.2, 57.5)
- moved R102 127.7 mm to (160.2, 65.7)
- moved C105 127.7 mm to (168.7, 58.4)
- moved C107 127.7 mm to (168.7, 60.3)
- moved C110 127.7 mm to (169.4, 75.3)
- moved D111 127.7 mm to (161.8, 76.2)
- moved U102 127.7 mm to (173.8, 62.2)
- moved C102 127.7 mm to (163.0, 59.4)
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Other:
- board outline added: 280 x 100 mm
