File: input/in_amp.sch (KiCad schematic (older format))
At the start: 16 parts

Commit message: Continuing work on input board, also added some design files and PDF documentation for the prototype source and sensor.  Deleted various spurious kicad project files.  The main project for the input board is now input_board.pro.
Parts:
- added C125, C126: 2.2n 1% C0G, Capacitor_SMD:C_0805_2012Metric, symbol Device:C_Small
- gave numbers to parts that had none: 16
Connections:
- wire segments 72 -> 79
Other:
- note added: "C125,C126 mainly there to swamp excess capacitance at the \ninverting input due to gain switching network, but also give\nsome band limiting, 144 kHz. The antialias filter gives plenty\nof rejection, so we are not risking compromising CMR by\ntaking a strong cut here (though to first order, mismatch should\nnot matter)."
- moved on the sheet: C101, C102, C103, C104, J101, R101, R102, R103, R104, R105, U102, U103

Commit message: Mainly work on the top level of the input board, attaching signals to the channels, digital I/O.  Decided to use Eurocard 64 pin type B connector for the connection to the main board.  See input_board_pinout.txt.
Parts:
- removed C102, C103, C105: 1u, Capacitor_SMD:C_0603_1608Metric, symbol Device:C_Small
- removed C125: 2.2n 1% C0G, Capacitor_SMD:C_0805_2012Metric, symbol Device:C_Small
- removed R104, R105: 499, Resistor_SMD:R_1206_3216Metric, symbol Device:R_US
- removed RN101: 1K, Resistor_SMD:R_Array_Convex_4x1206, symbol Device:R_Pack04
- removed U102, U104: LT1028, symbol ilemt_input:opamp_single
- added C129: 2.2n 1% C0G, Capacitor_SMD:C_0805_2012Metric, symbol Device:C_Small
- added C132, C133, C135: 1u, Capacitor_SMD:C_0603_1608Metric, symbol Device:C_Small
- added R129, R130: 499, Resistor_SMD:R_1206_3216Metric, symbol Device:R_US
- added RN103: 1K, Resistor_SMD:R_Array_Convex_4x1206, symbol Device:R_Pack04
- added U105, U107: LT1028, symbol ilemt_input:opamp_single
- renumbered C126 to C130, C101 to C131, C104 to C134, C106 to C136, R101 to R126, R102 to R127, R103 to R128, U103 to U106
Other:
- note added: "C195, C1230 mainly there to swamp excess capacitance at the \ninverting input due to gain switching network, but also give\nsome band limiting, 144 kHz. The antialias filter gives plenty\nof rejection, so we are not risking compromising CMR by\ntaking a strong cut here (though to first order, mismatch should\nnot matter)."
- note removed: "C125,C126 mainly there to swamp excess capacitance at the \ninverting input due to gain switching network, but also give\nsome band limiting, 144 kHz. The antialias filter gives plenty\nof rejection, so we are not risking compromising CMR by\ntaking a strong cut here (though to first order, mismatch should\nnot matter)."
Changed lines of the file:
@@
 EESchema Schematic File Version 4
+LIBS:input_board-cache
 LIBS:input_channel-cache
 EELAYER 29 0
@@
 $Descr A4 11693 8268
 encoding utf-8
-Sheet 3 5
+Sheet 6 10
 Title ""
 Date ""
@@
 $EndDescr
 $Comp
-L power:+15V #PWR0102
-U 1 1 5DE453A9
+L power:+15V #PWR0139
+U 1 1 5DFFAD16
 P 4000 900
-F 0 "#PWR0102" H 4000 750 50  0001 C CNN
+F 0 "#PWR0139" H 4000 750 50  0001 C CNN
 F 1 "+15V" H 4015 1073 50  0000 C CNN
 F 2 "" H 4000 900 50  0001 C CNN
@@
 	4000 900  4000 1000
 $Comp
-L Device:C_Small C101
+L Device:C_Small C131
 U 1 1 5DE6EE08
 P 4350 1000
-F 0 "C101" V 4121 1000 50  0000 C CNN
+F 0 "C131" V 4121 1000 50  0000 C CNN
 F 1 "1u" V 4212 1000 50  0000 C CNN
 F 2 "Capacitor_SMD:C_0603_1608Metric" H 4350 1000 50  0001 C CNN
@@
 	4000 1700 4000 1850
 $Comp
-L power:-15V #PWR0103
+L power:-15V #PWR0140
 U 1 1 5DE6EE07
 P 4000 1900
-F 0 "#PWR0103" H 4000 2000 50  0001 C CNN
+F 0 "#PWR0140" H 4000 2000 50  0001 C CNN
 F 1 "-15V" H 4015 2073 50  0000 C CNN
 F 2 "" H 4000 1900 50  0001 C CNN
@@
 	4000 1000 4000 1100
 $Comp
-L power:GNDA #PWR0106
-U 1 1 5DE6EE09
+L power:GNDA #PWR0143
+U 1 1 5DFFAD1A
 P 4600 1000
-F 0 "#PWR0106" H 4600 750 50  0001 C CNN
+F 0 "#PWR0143" H 4600 750 50  0001 C CNN
 F 1 "GNDA" V 4605 872 50  0000 R CNN
 F 2 "" H 4600 1000 50  0001 C CNN
@@
 	4450 1000 4600 1000
 $Comp
-L Device:C_Small C102
-U 1 1 5DE6EE0A
+L Device:C_Small C132
+U 1 1 5E195589
 P 4350 1850
-F 0 "C102" V 4121 1850 50  0000 C CNN
+F 0 "C132" V 4121 1850 50  0000 C CNN
 F 1 "1u" V 4212 1850 50  0000 C CNN
 F 2 "Capacitor_SMD:C_0603_1608Metric" H 4350 1850 50  0001 C CNN
@@
 $EndComp
 $Comp
-L power:GNDA #PWR0107
-U 1 1 5DE6EE0B
+L power:GNDA #PWR0144
+U 1 1 5E19558A
 P 4600 1850
-F 0 "#PWR0107" H 4600 1600 50  0001 C CNN
+F 0 "#PWR0144" H 4600 1600 50  0001 C CNN
 F 1 "GNDA" V 4605 1722 50  0000 R CNN
 F 2 "" H 4600 1850 50  0001 C CNN
@@
 	4450 1850 4600 1850
 $Comp
-L ilemt_input:opamp_single U102
-U 1 1 5DE44053
+L ilemt_input:opamp_single U105
+U 1 1 5DFFAD15
 P 3950 1400
-F 0 "U102" H 4294 1446 50  0000 L CNN
+F 0 "U105" H 4294 1446 50  0000 L CNN
 F 1 "LT1028" H 4294 1355 50  0000 L CNN
 F 2 "" H 4000 1450 50  0001 C CNN
@@
 $EndComp
 $Comp
-L Device:C_Small C103
-U 1 1 5DE57C96
+L Device:C_Small C133
+U 1 1 5E19556B
 P 4450 5850
-F 0 "C103" V 4221 5850 50  0000 C CNN
+F 0 "C133" V 4221 5850 50  0000 C CNN
 F 1 "1u" V 4312 5850 50  0000 C CNN
 F 2 "Capacitor_SMD:C_0603_1608Metric" H 4450 5850 50  0001 C CNN
@@
 $EndComp
 $Comp
-L power:GNDA #PWR0108
-U 1 1 5DE57CA6
+L power:GNDA #PWR0145
+U 1 1 5E19556C
 P 4700 5850
-F 0 "#PWR0108" H 4700 5600 50  0001 C CNN
+F 0 "#PWR0145" H 4700 5600 50  0001 C CNN
 F 1 "GNDA" V 4705 5722 50  0000 R CNN
 F 2 "" H 4700 5850 50  0001 C CNN
@@
 	4550 5850 4700 5850
 $Comp
-L Device:C_Small C104
+L Device:C_Small C134
 U 1 1 5DE57CAD
 P 4450 6700
-F 0 "C104" V 4221 6700 50  0000 C CNN
+F 0 "C134" V 4221 6700 50  0000 C CNN
 F 1 "1u" V 4312 6700 50  0000 C CNN
 F 2 "Capacitor_SMD:C_0603_1608Metric" H 4450 6700 50  0001 C CNN
@@
 $EndComp
 $Comp
-L power:GNDA #PWR0109
+L power:GNDA #PWR0146
 U 1 1 5DE57CB3
 P 4700 6700
-F 0 "#PWR0109" H 4700 6450 50  0001 C CNN
+F 0 "#PWR0146" H 4700 6450 50  0001 C CNN
 F 1 "GNDA" V 4705 6572 50  0000 R CNN
 F 2 "" H 4700 6700 50  0001 C CNN
@@
 	4350 6700 4100 6700
 $Comp
-L ilemt_input:opamp_single U103
+L ilemt_input:opamp_single U106
 U 1 1 5DE57CBD
 P 4050 6250
-F 0 "U103" H 4394 6296 50  0000 L CNN
+F 0 "U106" H 4394 6296 50  0000 L CNN
 F 1 "LT1028" H 4394 6205 50  0000 L CNN
 F 2 "" H 4100 6300 50  0001 C CNN
@@
 $EndComp
 $Comp
-L power:+15V #PWR0105
+L power:+15V #PWR0142
 U 1 1 5DE6EE11
 P 4100 6850
-F 0 "#PWR0105" H 4100 6700 50  0001 C CNN
+F 0 "#PWR0142" H 4100 6700 50  0001 C CNN
 F 1 "+15V" H 4115 7023 50  0000 C CNN
 F 2 "" H 4100 6850 50  0001 C CNN
@@
 	4100 5750 4100 5850
 $Comp
-L power:-15V #PWR0104
+L power:-15V #PWR0141
 U 1 1 5DE5ACAE
 P 4100 5750
-F 0 "#PWR0104" H 4100 5850 50  0001 C CNN
+F 0 "#PWR0141" H 4100 5850 50  0001 C CNN
 F 1 "-15V" H 4115 5923 50  0000 C CNN
 F 2 "" H 4100 5750 50  0001 C CNN
@@
 	4000 1850 4250 1850
 $Comp
-L Device:R_US R104
-U 1 1 5DE6107D
+L Device:R_US R129
+U 1 1 5DFFAD17
 P 4100 2350
-F 0 "R104" V 4200 2350 50  0000 C CNN
+F 0 "R129" V 4200 2350 50  0000 C CNN
 F 1 "499" V 4000 2350 50  0000 C CNN
 F 2 "Resistor_SMD:R_1206_3216Metric" V 4140 2340 50  0001 C CNN
@@
 	4350 1400 5450 1400
 $Comp
-L Device:R_US R105
-U 1 1 5DE6EE14
+L Device:R_US R130
+U 1 1 5E19558D
 P 4100 5250
-F 0 "R105" V 4200 5250 50  0000 C CNN
+F 0 "R130" V 4200 5250 50  0000 C CNN
 F 1 "499" V 4000 5250 50  0000 C CNN
 F 2 "Resistor_SMD:R_1206_3216Metric" V 4140 5240 50  0001 C CNN
@@
 $EndComp
 $Comp
-L Device:R_US R101
+L Device:R_US R126
 U 1 1 5DE6EE16
 P 3100 4050
-F 0 "R101" V 3200 4050 50  0000 C CNN
+F 0 "R126" V 3200 4050 50  0000 C CNN
 F 1 "49.9" V 3000 4050 50  0000 C CNN
 F 2 "Resistor_SMD:R_0603_1608Metric" V 3140 4040 50  0001 C CNN
@@
 $EndComp
 $Comp
-L Device:R_US R102
+L Device:R_US R127
 U 1 1 5DE6EE17
 P 3500 4050
-F 0 "R102" V 3600 4050 50  0000 C CNN
+F 0 "R127" V 3600 4050 50  0000 C CNN
 F 1 "143" V 3400 4050 50  0000 C CNN
 F 2 "Resistor_SMD:R_0603_1608Metric" V 3540 4040 50  0001 C CNN
@@
 $EndComp
 $Comp
-L Device:R_US R103
+L Device:R_US R128
 U 1 1 5DE76F92
 P 3900 4050
-F 0 "R103" V 4000 4050 50  0000 C CNN
+F 0 "R128" V 4000 4050 50  0000 C CNN
 F 1 "499" V 3800 4050 50  0000 C CNN
 F 2 "Resistor_SMD:R_1206_3216Metric" V 3940 4040 50  0001 C CNN
@@
 Connection ~ 3400 5250
 $Comp
-L Device:C_Small C105
-U 1 1 5DE8AF02
+L Device:C_Small C135
+U 1 1 5E1955A1
 P 7400 3000
-F 0 "C105" V 7171 3000 50  0000 C CNN
+F 0 "C135" V 7171 3000 50  0000 C CNN
 F 1 "1u" V 7262 3000 50  0000 C CNN
 F 2 "Capacitor_SMD:C_0603_1608Metric" H 7400 3000 50  0001 C CNN
@@
 $EndComp
 $Comp
-L power:GNDA #PWR0112
+L power:GNDA #PWR0149
 U 1 1 5DE8AF08
 P 7650 3000
-F 0 "#PWR0112" H 7650 2750 50  0001 C CNN
+F 0 "#PWR0149" H 7650 2750 50  0001 C CNN
 F 1 "GNDA" V 7655 2872 50  0000 R CNN
 F 2 "" H 7650 3000 50  0001 C CNN
@@
 	7500 3000 7650 3000
 $Comp
-L Device:C_Small C106
+L Device:C_Small C136
 U 1 1 5DE6EE1B
 P 7400 3850
-F 0 "C106" V 7171 3850 50  0000 C CNN
+F 0 "C136" V 7171 3850 50  0000 C CNN
 F 1 "1u" V 7262 3850 50  0000 C CNN
 F 2 "Capacitor_SMD:C_0603_1608Metric" H 7400 3850 50  0001 C CNN
@@
 $EndComp
 $Comp
-L power:GNDA #PWR0113
+L power:GNDA #PWR0150
 U 1 1 5DE6EE1C
 P 7650 3850
-F 0 "#PWR0113" H 7650 3600 50  0001 C CNN
+F 0 "#PWR0150" H 7650 3600 50  0001 C CNN
 F 1 "GNDA" V 7655 3722 50  0000 R CNN
 F 2 "" H 7650 3850 50  0001 C CNN
@@
 	7300 3850 7050 3850
 $Comp
-L ilemt_input:opamp_single U104
-U 1 1 5DE8AF1D
+L ilemt_input:opamp_single U107
+U 1 1 5E1955A3
 P 7000 3400
-F 0 "U104" H 7344 3446 50  0000 L CNN
+F 0 "U107" H 7344 3446 50  0000 L CNN
 F 1 "LT1028" H 7344 3355 50  0000 L CNN
 F 2 "" H 7050 3450 50  0001 C CNN
@@
 $EndComp
 $Comp
-L power:+15V #PWR0111
+L power:+15V #PWR0148
 U 1 1 5DE6EE1E
 P 7050 4000
-F 0 "#PWR0111" H 7050 3850 50  0001 C CNN
+F 0 "#PWR0148" H 7050 3850 50  0001 C CNN
 F 1 "+15V" H 7065 4173 50  0000 C CNN
 F 2 "" H 7050 4000 50  0001 C CNN
@@
 	7050 2900 7050 3000
 $Comp
-L power:-15V #PWR0110
-U 1 1 5DE6EE1F
+L power:-15V #PWR0147
+U 1 1 5E195594
 P 7050 2900
-F 0 "#PWR0110" H 7050 3000 50  0001 C CNN
+F 0 "#PWR0147" H 7050 3000 50  0001 C CNN
 F 1 "-15V" H 7065 3073 50  0000 C CNN
 F 2 "" H 7050 2900 50  0001 C CNN
@@
 	7400 3400 8250 3400
 $Comp
-L Device:R_Pack04 RN101
-U 1 1 5DE6EE20
+L Device:R_Pack04 RN103
+U 1 1 5E195595
 P 6250 3500
-F 0 "RN101" V 5950 3500 50  0000 C CNN
+F 0 "RN103" V 5950 3500 50  0000 C CNN
 F 1 "1K" V 6450 3500 50  0000 C CNN
 F 2 "Resistor_SMD:R_Array_Convex_4x1206" V 6525 3500 50  0001 C CNN
@@
 Connection ~ 5450 2350
 $Comp
-L Device:C_Small C125
-U 1 1 5DF0964A
+L Device:C_Small C129
+U 1 1 5E1955B8
 P 4100 2850
-F 0 "C125" V 3871 2850 50  0000 C CNN
+F 0 "C129" V 3871 2850 50  0000 C CNN
 F 1 "2.2n 1% C0G" V 3962 2850 50  0000 C CNN
 F 2 "Capacitor_SMD:C_0805_2012Metric" H 4100 2850 50  0001 C CNN
@@
 	3400 4350 3500 4350
 $Comp
-L Device:C_Small C126
+L Device:C_Small C130
 U 1 1 5DF1938A
 P 4100 4800
-F 0 "C126" V 3871 4800 50  0000 C CNN
+F 0 "C130" V 3871 4800 50  0000 C CNN
 F 1 "2.2n 1% C0G" V 3962 4800 50  0000 C CNN
 F 2 "Capacitor_SMD:C_0805_2012Metric" H 4100 4800 50  0001 C CNN
@@
 Connection ~ 3450 2850
 Text Notes 5800 5250 0    50   ~ 0
-C125,C126 mainly there to swamp excess capacitance at the \ninverting input due to gain switching network, but also give\nsome band limiting, 144 kHz.  The antialias filter gives plenty\nof rejection, so we are not risking compromising CMR by\ntaking a strong cut here (though to first order, mismatch should\nnot matter).
+C195, C1230 mainly there to swamp excess capacitance at the \ninverting input due to gain switching network, but also give\nsome band limiting, 144 kHz.  The antialias filter gives plenty\nof rejection, so we are not risking compromising CMR by\ntaking a strong cut here (though to first order, mismatch should\nnot matter).
 $EndSCHEMATC

Commit message: Still beating into overall shape.  This is a checkpoint before modifying the analog signal chain to fold the diff amp and antialias into the driver, going to a full differential path.
Overall: Changes to component attributes to reduce duplicates in BOM, and added links to Digikey and datasheets.

board_connector.sch: Added reference input pins, decimation SEL lines.

in_filter.sch:
Fixed BIST feedback to be taken at the top of each injection resistor (4 lines, not 2)

input_board.sch:
Added some missing connections and no-connects.

power_budget.xlsx:
Much more elaborate now, models effect of input levels on load currents, computes currents and total power, for several variants.

reference_buffer.sch:
Updated with booster sink transistor to handle sourcing into reference by ADC clamp diodes.

simetrix/:
Added supply_negative.wxsch and supply_positive.wxsch, which are concepts for low noise lowish dropout regulators for the analog rails.  Other simetrix modifications are cosmetic.
Parts:
- C129, C130: value 2.2n 1% C0G -> 2.2nF; Notes (none) -> 1% C0G
- C131, C132, C133, C134, C135, C136: value 1u -> 1uF
- R128, R129, R130: Description (none) -> RES 499 OHM 0.1% 2/5W 1206; Digikey (none) -> 541-3877-1-ND
- RN103: Description (none) -> RES ARRAY 4 RES 1K OHM 1206 0.1%; Digikey (none) -> 749-1015-1-ND; MPN (none) -> ACASA1001S1001P100
Changed lines of the file:
@@
 U 1 1 5DFFAD16
 P 4000 900
+AR Path="/5DFCF14D/5DA78BF5/5DFFAD16" Ref="#PWR0139"  Part="1"
+AR Path="/5DFCF14D/5E195558/5DFFAD16" Ref="#PWR0139"  Part="1"
 F 0 "#PWR0139" H 4000 750 50  0001 C CNN
 F 1 "+15V" H 4015 1073 50  0000 C CNN
@@
 U 1 1 5DE6EE08
 P 4350 1000
+AR Path="/5DFCF14D/5DA78BF5/5DE6EE08" Ref="C131"  Part="1"
+AR Path="/5DFCF14D/5E195558/5DE6EE08" Ref="C131"  Part="1"
 F 0 "C131" V 4121 1000 50  0000 C CNN
-F 1 "1u" V 4212 1000 50  0000 C CNN
+F 1 "1uF" V 4212 1000 50  0000 C CNN
 F 2 "Capacitor_SMD:C_0603_1608Metric" H 4350 1000 50  0001 C CNN
 F 3 "~" H 4350 1000 50  0001 C CNN
@@
 U 1 1 5DE6EE07
 P 4000 1900
+AR Path="/5DFCF14D/5DA78BF5/5DE6EE07" Ref="#PWR0140"  Part="1"
+AR Path="/5DFCF14D/5E195558/5DE6EE07" Ref="#PWR0140"  Part="1"
 F 0 "#PWR0140" H 4000 2000 50  0001 C CNN
 F 1 "-15V" H 4015 2073 50  0000 C CNN
@@
 U 1 1 5DFFAD1A
 P 4600 1000
+AR Path="/5DFCF14D/5DA78BF5/5DFFAD1A" Ref="#PWR0143"  Part="1"
+AR Path="/5DFCF14D/5E195558/5DFFAD1A" Ref="#PWR0143"  Part="1"
 F 0 "#PWR0143" H 4600 750 50  0001 C CNN
 F 1 "GNDA" V 4605 872 50  0000 R CNN
@@
 U 1 1 5E195589
 P 4350 1850
+AR Path="/5DFCF14D/5DA78BF5/5E195589" Ref="C132"  Part="1"
+AR Path="/5DFCF14D/5E195558/5E195589" Ref="C132"  Part="1"
 F 0 "C132" V 4121 1850 50  0000 C CNN
-F 1 "1u" V 4212 1850 50  0000 C CNN
+F 1 "1uF" V 4212 1850 50  0000 C CNN
 F 2 "Capacitor_SMD:C_0603_1608Metric" H 4350 1850 50  0001 C CNN
 F 3 "~" H 4350 1850 50  0001 C CNN
@@
 U 1 1 5E19558A
 P 4600 1850
+AR Path="/5DFCF14D/5DA78BF5/5E19558A" Ref="#PWR0144"  Part="1"
+AR Path="/5DFCF14D/5E195558/5E19558A" Ref="#PWR0144"  Part="1"
 F 0 "#PWR0144" H 4600 1600 50  0001 C CNN
 F 1 "GNDA" V 4605 1722 50  0000 R CNN
@@
 U 1 1 5DFFAD15
 P 3950 1400
+AR Path="/5DFCF14D/5DA78BF5/5DFFAD15" Ref="U105"  Part="1"
+AR Path="/5DFCF14D/5E195558/5DFFAD15" Ref="U105"  Part="1"
 F 0 "U105" H 4294 1446 50  0000 L CNN
 F 1 "LT1028" H 4294 1355 50  0000 L CNN
@@
 U 1 1 5E19556B
 P 4450 5850
+AR Path="/5DFCF14D/5DA78BF5/5E19556B" Ref="C133"  Part="1"
+AR Path="/5DFCF14D/5E195558/5E19556B" Ref="C133"  Part="1"
 F 0 "C133" V 4221 5850 50  0000 C CNN
-F 1 "1u" V 4312 5850 50  0000 C CNN
+F 1 "1uF" V 4312 5850 50  0000 C CNN
 F 2 "Capacitor_SMD:C_0603_1608Metric" H 4450 5850 50  0001 C CNN
 F 3 "~" H 4450 5850 50  0001 C CNN
@@
 U 1 1 5E19556C
 P 4700 5850
+AR Path="/5DFCF14D/5DA78BF5/5E19556C" Ref="#PWR0145"  Part="1"
+AR Path="/5DFCF14D/5E195558/5E19556C" Ref="#PWR0145"  Part="1"
 F 0 "#PWR0145" H 4700 5600 50  0001 C CNN
 F 1 "GNDA" V 4705 5722 50  0000 R CNN
@@
 U 1 1 5DE57CAD
 P 4450 6700
+AR Path="/5DFCF14D/5DA78BF5/5DE57CAD" Ref="C134"  Part="1"
+AR Path="/5DFCF14D/5E195558/5DE57CAD" Ref="C134"  Part="1"
 F 0 "C134" V 4221 6700 50  0000 C CNN
-F 1 "1u" V 4312 6700 50  0000 C CNN
+F 1 "1uF" V 4312 6700 50  0000 C CNN
 F 2 "Capacitor_SMD:C_0603_1608Metric" H 4450 6700 50  0001 C CNN
 F 3 "~" H 4450 6700 50  0001 C CNN
@@
 U 1 1 5DE57CB3
 P 4700 6700
+AR Path="/5DFCF14D/5DA78BF5/5DE57CB3" Ref="#PWR0146"  Part="1"
+AR Path="/5DFCF14D/5E195558/5DE57CB3" Ref="#PWR0146"  Part="1"
 F 0 "#PWR0146" H 4700 6450 50  0001 C CNN
 F 1 "GNDA" V 4705 6572 50  0000 R CNN
@@
 U 1 1 5DE57CBD
 P 4050 6250
+AR Path="/5DFCF14D/5DA78BF5/5DE57CBD" Ref="U106"  Part="1"
+AR Path="/5DFCF14D/5E195558/5DE57CBD" Ref="U106"  Part="1"
 F 0 "U106" H 4394 6296 50  0000 L CNN
 F 1 "LT1028" H 4394 6205 50  0000 L CNN
@@
 U 1 1 5DE6EE11
 P 4100 6850
+AR Path="/5DFCF14D/5DA78BF5/5DE6EE11" Ref="#PWR0142"  Part="1"
+AR Path="/5DFCF14D/5E195558/5DE6EE11" Ref="#PWR0142"  Part="1"
 F 0 "#PWR0142" H 4100 6700 50  0001 C CNN
 F 1 "+15V" H 4115 7023 50  0000 C CNN
@@
 U 1 1 5DE5ACAE
 P 4100 5750
+AR Path="/5DFCF14D/5DA78BF5/5DE5ACAE" Ref="#PWR0141"  Part="1"
+AR Path="/5DFCF14D/5E195558/5DE5ACAE" Ref="#PWR0141"  Part="1"
 F 0 "#PWR0141" H 4100 5850 50  0001 C CNN
 F 1 "-15V" H 4115 5923 50  0000 C CNN
@@
 U 1 1 5DFFAD17
 P 4100 2350
+AR Path="/5DFCF14D/5DA78BF5/5DFFAD17" Ref="R129"  Part="1"
+AR Path="/5DFCF14D/5E195558/5DFFAD17" Ref="R129"  Part="1"
 F 0 "R129" V 4200 2350 50  0000 C CNN
 F 1 "499" V 4000 2350 50  0000 C CNN
 F 2 "Resistor_SMD:R_1206_3216Metric" V 4140 2340 50  0001 C CNN
-F 3 "~" H 4100 2350 50  0001 C CNN
+F 3 "http://www.vishay.com/docs/28758/tnpw_e3.pdf" H 4100 2350 50  0001 C CNN
+F 4 "RES 499 OHM 0.1% 2/5W 1206" H 4100 2350 50  0001 C CNN "Description"
+F 5 "541-3877-1-ND" H 4100 2350 50  0001 C CNN "Digikey"
 	1    4100 2350
 	0    1    1    0
@@
 U 1 1 5E19558D
 P 4100 5250
+AR Path="/5DFCF14D/5DA78BF5/5E19558D" Ref="R130"  Part="1"
+AR Path="/5DFCF14D/5E195558/5E19558D" Ref="R130"  Part="1"
 F 0 "R130" V 4200 5250 50  0000 C CNN
 F 1 "499" V 4000 5250 50  0000 C CNN
 F 2 "Resistor_SMD:R_1206_3216Metric" V 4140 5240 50  0001 C CNN
-F 3 "~" H 4100 5250 50  0001 C CNN
+F 3 "http://www.vishay.com/docs/28758/tnpw_e3.pdf" H 4100 5250 50  0001 C CNN
+F 4 "RES 499 OHM 0.1% 2/5W 1206" H 4100 5250 50  0001 C CNN "Description"
+F 5 "541-3877-1-ND" H 4100 5250 50  0001 C CNN "Digikey"
 	1    4100 5250
 	0    1    1    0
@@
 U 1 1 5DE6EE15
 P 3100 3550
+AR Path="/5DFCF14D/5DA78BF5/5DE6EE15" Ref="J101"  Part="1"
+AR Path="/5DFCF14D/5E195558/5DE6EE15" Ref="J101"  Part="1"
 F 0 "J101" V 3200 3750 50  0000 C CNN
 F 1 "Conn_02x02_Odd_Even" V 3100 4100 50  0000 C CNN
@@
 U 1 1 5DE6EE16
 P 3100 4050
+AR Path="/5DFCF14D/5DA78BF5/5DE6EE16" Ref="R126"  Part="1"
+AR Path="/5DFCF14D/5E195558/5DE6EE16" Ref="R126"  Part="1"
 F 0 "R126" V 3200 4050 50  0000 C CNN
 F 1 "49.9" V 3000 4050 50  0000 C CNN
@@
 U 1 1 5DE6EE17
 P 3500 4050
+AR Path="/5DFCF14D/5DA78BF5/5DE6EE17" Ref="R127"  Part="1"
+AR Path="/5DFCF14D/5E195558/5DE6EE17" Ref="R127"  Part="1"
 F 0 "R127" V 3600 4050 50  0000 C CNN
 F 1 "143" V 3400 4050 50  0000 C CNN
@@
 U 1 1 5DE76F92
 P 3900 4050
+AR Path="/5DFCF14D/5DA78BF5/5DE76F92" Ref="R128"  Part="1"
+AR Path="/5DFCF14D/5E195558/5DE76F92" Ref="R128"  Part="1"
 F 0 "R128" V 4000 4050 50  0000 C CNN
 F 1 "499" V 3800 4050 50  0000 C CNN
 F 2 "Resistor_SMD:R_1206_3216Metric" V 3940 4040 50  0001 C CNN
-F 3 "~" H 3900 4050 50  0001 C CNN
+F 3 "http://www.vishay.com/docs/28758/tnpw_e3.pdf" H 3900 4050 50  0001 C CNN
+F 4 "RES 499 OHM 0.1% 2/5W 1206" H 3900 4050 50  0001 C CNN "Description"
+F 5 "541-3877-1-ND" H 3900 4050 50  0001 C CNN "Digikey"
 	1    3900 4050
 	1    0    0    -1
@@
 U 1 1 5E1955A1
 P 7400 3000
+AR Path="/5DFCF14D/5DA78BF5/5E1955A1" Ref="C135"  Part="1"
+AR Path="/5DFCF14D/5E195558/5E1955A1" Ref="C135"  Part="1"
 F 0 "C135" V 7171 3000 50  0000 C CNN
-F 1 "1u" V 7262 3000 50  0000 C CNN
+F 1 "1uF" V 7262 3000 50  0000 C CNN
 F 2 "Capacitor_SMD:C_0603_1608Metric" H 7400 3000 50  0001 C CNN
 F 3 "~" H 7400 3000 50  0001 C CNN
@@
 U 1 1 5DE8AF08
 P 7650 3000
+AR Path="/5DFCF14D/5DA78BF5/5DE8AF08" Ref="#PWR0149"  Part="1"
+AR Path="/5DFCF14D/5E195558/5DE8AF08" Ref="#PWR0149"  Part="1"
 F 0 "#PWR0149" H 7650 2750 50  0001 C CNN
 F 1 "GNDA" V 7655 2872 50  0000 R CNN
@@
 U 1 1 5DE6EE1B
 P 7400 3850
+AR Path="/5DFCF14D/5DA78BF5/5DE6EE1B" Ref="C136"  Part="1"
+AR Path="/5DFCF14D/5E195558/5DE6EE1B" Ref="C136"  Part="1"
 F 0 "C136" V 7171 3850 50  0000 C CNN
-F 1 "1u" V 7262 3850 50  0000 C CNN
+F 1 "1uF" V 7262 3850 50  0000 C CNN
 F 2 "Capacitor_SMD:C_0603_1608Metric" H 7400 3850 50  0001 C CNN
 F 3 "~" H 7400 3850 50  0001 C CNN
@@
 U 1 1 5DE6EE1C
 P 7650 3850
+AR Path="/5DFCF14D/5DA78BF5/5DE6EE1C" Ref="#PWR0150"  Part="1"
+AR Path="/5DFCF14D/5E195558/5DE6EE1C" Ref="#PWR0150"  Part="1"
 F 0 "#PWR0150" H 7650 3600 50  0001 C CNN
 F 1 "GNDA" V 7655 3722 50  0000 R CNN
@@
 U 1 1 5E1955A3
 P 7000 3400
+AR Path="/5DFCF14D/5DA78BF5/5E1955A3" Ref="U107"  Part="1"
+AR Path="/5DFCF14D/5E195558/5E1955A3" Ref="U107"  Part="1"
 F 0 "U107" H 7344 3446 50  0000 L CNN
 F 1 "LT1028" H 7344 3355 50  0000 L CNN
@@
 U 1 1 5DE6EE1E
 P 7050 4000
+AR Path="/5DFCF14D/5DA78BF5/5DE6EE1E" Ref="#PWR0148"  Part="1"
+AR Path="/5DFCF14D/5E195558/5DE6EE1E" Ref="#PWR0148"  Part="1"
 F 0 "#PWR0148" H 7050 3850 50  0001 C CNN
 F 1 "+15V" H 7065 4173 50  0000 C CNN
@@
 U 1 1 5E195594
 P 7050 2900
+AR Path="/5DFCF14D/5DA78BF5/5E195594" Ref="#PWR0147"  Part="1"
+AR Path="/5DFCF14D/5E195558/5E195594" Ref="#PWR0147"  Part="1"
 F 0 "#PWR0147" H 7050 3000 50  0001 C CNN
 F 1 "-15V" H 7065 3073 50  0000 C CNN
@@
 U 1 1 5E195595
 P 6250 3500
+AR Path="/5DFCF14D/5DA78BF5/5E195595" Ref="RN103"  Part="1"
+AR Path="/5DFCF14D/5E195558/5E195595" Ref="RN103"  Part="1"
 F 0 "RN103" V 5950 3500 50  0000 C CNN
 F 1 "1K" V 6450 3500 50  0000 C CNN
 F 2 "Resistor_SMD:R_Array_Convex_4x1206" V 6525 3500 50  0001 C CNN
-F 3 "~" H 6250 3500 50  0001 C CNN
+F 3 "http://www.vishay.com/docs/28751/acasprec.pdf" H 6250 3500 50  0001 C CNN
+F 4 "749-1015-1-ND" V 6250 3500 50  0001 C CNN "Digikey"
+F 5 "ACASA1001S1001P100" V 6250 3500 50  0001 C CNN "MPN"
+F 6 "RES ARRAY 4 RES 1K OHM 1206 0.1%" V 6250 3500 50  0001 C CNN "Description"
 	1    6250 3500
 	0    1    1    0
@@
 U 1 1 5E1955B8
 P 4100 2850
+AR Path="/5DFCF14D/5DA78BF5/5E1955B8" Ref="C129"  Part="1"
+AR Path="/5DFCF14D/5E195558/5E1955B8" Ref="C129"  Part="1"
 F 0 "C129" V 3871 2850 50  0000 C CNN
-F 1 "2.2n 1% C0G" V 3962 2850 50  0000 C CNN
+F 1 "2.2nF" V 3962 2850 50  0000 C CNN
 F 2 "Capacitor_SMD:C_0805_2012Metric" H 4100 2850 50  0001 C CNN
 F 3 "~" H 4100 2850 50  0001 C CNN
+F 4 "1% C0G" H 4100 2850 50  0001 C CNN "Notes"
 	1    4100 2850
 	0    1    1    0
@@
 U 1 1 5DF1938A
 P 4100 4800
+AR Path="/5DFCF14D/5DA78BF5/5DF1938A" Ref="C130"  Part="1"
+AR Path="/5DFCF14D/5E195558/5DF1938A" Ref="C130"  Part="1"
 F 0 "C130" V 3871 4800 50  0000 C CNN
-F 1 "2.2n 1% C0G" V 3962 4800 50  0000 C CNN
+F 1 "2.2nF" V 3962 4800 50  0000 C CNN
 F 2 "Capacitor_SMD:C_0805_2012Metric" H 4100 4800 50  0001 C CNN
 F 3 "~" H 4100 4800 50  0001 C CNN
+F 4 "1% C0G" H 4100 4800 50  0001 C CNN "Notes"
 	1    4100 4800
 	0    1    1    0
