File: input/reference_buffer.sch (KiCad schematic (older format))
At the start: 23 parts, among them Q1 NSS1C300ET4G, U1 OP27

Commit message: Cleanup to get ready to start board layout. I had to get rid off all the bus signals, since in Kicad busses don't work that way.  Added a couple testpoints; many more needed.
Work on component placement in PCB.  I changed DGND to plain GND and "protective earth" to
"earth" (for chassis ground).  Chassis ground is now connected on the board only via a capacitor.
I had to fix the connector footprint to match the pin numbers on the symbol (there was a case
difference).
Parts:
- D1, D12, D13, D14, D2, D5, D6, D7: symbol Diode:BAV99 -> ilemt_input:BAS21S
Connections:
- net RAW_V+ renamed FILT_+10V
Changed lines of the file:
@@
 Wire Wire Line
 	4050 3550 4050 3700
-Wire Wire Line
-	4300 2850 4050 2850
 Connection ~ 4050 2850
 Wire Wire Line
@@
 	1    0    0    -1
 $EndComp
-Wire Wire Line
-	4050 3700 4300 3700
 $Comp
 L Device:R_US R4
@@
 Reference buffer
 $Comp
-L Diode:BAV99 D?
+L ilemt_input:BAS21S D?
 U 2 1 5E52A154
 P 5300 3050
@@
 Connection ~ 4050 3700
 Text GLabel 1500 2450 0    50   Input ~ 0
-RAW_V+
+FILT_+10V
 Wire Wire Line
 	4050 2450 4050 2850
 $Comp
-L Diode:BAV99 D?
+L ilemt_input:BAS21S D?
 U 1 1 5E29F9EE
 P 4300 2200
@@
 $EndComp
 $Comp
-L Diode:BAV99 D?
+L ilemt_input:BAS21S D?
 U 1 1 5E291915
 P 3800 4200
@@
 Wire Wire Line
 	3800 4400 3800 4350
-$Comp
-L Diode:BAV99 D?
-U 1 1 5E29190F
-P 4300 4200
-AR Path="/5DFCF14D/5DE42731/5E29190F" Ref="D?"  Part="2"
-AR Path="/5E1D6729/5E1DA2AA/5E29190F" Ref="D?"  Part="2"
-AR Path="/5E2EB92B/5E29190F" Ref="D7"  Part="1"
-F 0 "D7" H 4300 4415 50  0000 C CNN
-F 1 "BAS21S" H 4300 4324 50  0000 C CNN
-F 2 "Package_TO_SOT_SMD:SOT-23" H 4300 4050 50  0001 C CNN
-F 3 "https://assets.nexperia.com/documents/data-sheet/BAV99_SER.pdf" H 4300 4300 50  0001 C CNN
-	1    4300 4200
-	0    -1   -1   0
-$EndComp
 Wire Wire Line
 	4300 4400 4300 4350
@@
 Connection ~ 4050 3950
 Wire Wire Line
-	3800 3950 4050 3950
+	3800 3950 3850 3950
 Connection ~ 4050 2450
 Wire Wire Line
@@
 	5750 2500 6100 2500
 $Comp
-L Diode:BAV99 D?
+L ilemt_input:BAS21S D?
 U 1 1 5E52A153
 P 5750 2700
@@
 $EndComp
 $Comp
-L Diode:BAV99 D?
+L ilemt_input:BAS21S D?
 U 2 1 5E52A152
 P 5750 3050
@@
 $EndComp
 $Comp
-L Diode:BAV99 D?
+L ilemt_input:BAS21S D?
 U 1 1 5E5E3816
 P 1750 2450
@@
 $EndComp
 $Comp
-L Diode:BAV99 D?
+L ilemt_input:BAS21S D?
 U 2 1 5E5E381C
 P 2100 2450
@@
 	1900 2450 1950 2450
 $Comp
-L Diode:BAV99 D?
+L ilemt_input:BAS21S D?
 U 1 1 5E5E5222
 P 2450 2450
@@
 $EndComp
 $Comp
-L Diode:BAV99 D?
+L ilemt_input:BAS21S D?
 U 2 1 5E5E5228
 P 2800 2450
@@
 	1500 2450 1600 2450
 $Comp
-L Diode:BAV99 D?
+L ilemt_input:BAS21S D?
 U 1 1 5E600273
 P 3150 2450
@@
 $EndComp
 $Comp
-L Diode:BAV99 D?
+L ilemt_input:BAS21S D?
 U 2 1 5E600279
 P 3500 2450
@@
 	2950 2450 3000 2450
 Wire Wire Line
-	3650 2450 4050 2450
+	3650 2450 3850 2450
 Text GLabel 1450 3150 0    50   Input ~ 0
 +reference
 Text GLabel 1450 4750 0    50   Input ~ 0
 -reference
+$Comp
+L power:PWR_FLAG #FLG0108
+U 1 1 5E9020E8
+P 3850 2450
+F 0 "#FLG0108" H 3850 2525 50  0001 C CNN
+F 1 "PWR_FLAG" H 3850 2600 50  0000 C CNN
+F 2 "" H 3850 2450 50  0001 C CNN
+F 3 "~" H 3850 2450 50  0001 C CNN
+	1    3850 2450
+	1    0    0    -1
+$EndComp
+$Comp
+L power:PWR_FLAG #FLG0110
+U 1 1 5E902531
+P 3850 3950
+F 0 "#FLG0110" H 3850 4025 50  0001 C CNN
+F 1 "PWR_FLAG" H 3850 4100 50  0000 C CNN
+F 2 "" H 3850 3950 50  0001 C CNN
+F 3 "~" H 3850 3950 50  0001 C CNN
+	1    3850 3950
+	1    0    0    -1
+$EndComp
+Connection ~ 3850 2450
+Wire Wire Line
+	3850 2450 4050 2450
+Connection ~ 3850 3950
+Wire Wire Line
+	3850 3950 4050 3950
+Wire Wire Line
+	4050 3700 4300 3700
+Wire Wire Line
+	4050 2850 4300 2850
+$Comp
+L ilemt_input:BAS21S D?
+U 1 1 5E29190F
+P 4300 4200
+AR Path="/5DFCF14D/5DE42731/5E29190F" Ref="D?"  Part="2"
+AR Path="/5E1D6729/5E1DA2AA/5E29190F" Ref="D?"  Part="2"
+AR Path="/5E2EB92B/5E29190F" Ref="D7"  Part="1"
+F 0 "D7" H 4300 4415 50  0000 C CNN
+F 1 "BAS21S" H 4300 4324 50  0000 C CNN
+F 2 "Package_TO_SOT_SMD:SOT-23" H 4300 4050 50  0001 C CNN
+F 3 "https://assets.nexperia.com/documents/data-sheet/BAV99_SER.pdf" H 4300 4300 50  0001 C CNN
+	1    4300 4200
+	0    -1   -1   0
+$EndComp
 $EndSCHEMATC

Commit message: Changed board connector to PCIe 8x, added test points, cleanup of component values. Add LVDS Rx termination, bypass caps.
Parts:
- R1, R2, R3, R4: footprint Resistor_SMD:R_0805_2012Metric -> Resistor_SMD:R_0603_1608Metric
Changed lines of the file:
@@
 F 0 "R4" V 7250 4750 50  0000 C CNN
 F 1 "2K" V 7050 4750 50  0000 C CNN
-F 2 "Resistor_SMD:R_0805_2012Metric" V 7190 4740 50  0001 C CNN
+F 2 "Resistor_SMD:R_0603_1608Metric" V 7190 4740 50  0001 C CNN
 F 3 "~" H 7150 4750 50  0001 C CNN
 F 4 "0.1%" V 7150 4750 50  0001 C CNN "Notes"
@@
 F 0 "R3" V 2400 3650 50  0000 C CNN
 F 1 "2K" V 2200 3650 50  0000 C CNN
-F 2 "Resistor_SMD:R_0805_2012Metric" V 2340 3640 50  0001 C CNN
+F 2 "Resistor_SMD:R_0603_1608Metric" V 2340 3640 50  0001 C CNN
 F 3 "~" H 2300 3650 50  0001 C CNN
 F 4 "0.1%" V 2300 3650 50  0001 C CNN "Notes"
@@
 F 0 "R2" V 1850 4750 50  0000 C CNN
 F 1 "2K" V 1650 4750 50  0000 C CNN
-F 2 "Resistor_SMD:R_0805_2012Metric" V 1790 4740 50  0001 C CNN
+F 2 "Resistor_SMD:R_0603_1608Metric" V 1790 4740 50  0001 C CNN
 F 3 "~" H 1750 4750 50  0001 C CNN
 F 4 "0.1%" V 1750 4750 50  0001 C CNN "Notes"
@@
 F 0 "R1" V 1900 3150 50  0000 C CNN
 F 1 "2K" V 1700 3150 50  0000 C CNN
-F 2 "Resistor_SMD:R_0805_2012Metric" V 1840 3140 50  0001 C CNN
+F 2 "Resistor_SMD:R_0603_1608Metric" V 1840 3140 50  0001 C CNN
 F 3 "~" H 1800 3150 50  0001 C CNN
 F 4 "0.1%" V 1800 3150 50  0001 C CNN "Notes"

Commit message: Checkpoint before starting routing.  Added power and ground testpoints.
Parts:
- added TP5: VREF, TestPoint:TestPoint_THTPad_D1.5mm_Drill0.7mm, symbol Connector:TestPoint
- C1, C2: DK line (none) -> 14
- C3, C4: DK line (none) -> 27
- C5, C6: DK line (none) -> 28
- D1, D12, D13, D14, D2, D5, D6, D7: DK line (none) -> 43; Description (none) -> DIODE ARRAY GP 250V 225MA SOT23; Digikey (none) -> BAS21SLT1GOSCT-ND; MPN (none) -> BAS21SLT1G
- Q1: DK line (none) -> 23
- R1, R2, R3, R4: DK line (none) -> 17; Description (none) -> RES 2K OHM 0.1% 1/8W 0805; Digikey (none) -> P2.0KDACT-ND
- R5: DK line (none) -> 30
- R5: DK line (none) -> 10; Description (none) -> RES 0.068 OHM 1% 1/4W 1206; Digikey (none) -> 311-.068LWCT-ND
- R6: DK line (none) -> 16; Description (none) -> 2.74 Ohms ±1% 0.25W, 1/4W Chip Resistor 1206 (3216 Metric) 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; Digikey (none) -> 2019-RK73H2BTTD2R74FCT-ND; MPN (none) -> RK73H2BTTD2R74F
- U1: DK line (none) -> 15; Description (none) -> IC OPAMP GP 1 CIRCUIT 8SOIC; Digikey (none) -> 296-31706-1-ND
Connections:
- net VREF: now also TP5.1
- net +reference renamed VREF+
- net -reference renamed VREF-
