File: input/input_board.kicad_pcb (KiCad board)
At the start: 4 copper layers, 191 parts, among them J1 Sensor, J101 Gain, J2 C64AB, J3 Decimate, Q1 NSS1C300ET4G, Q2 2STD1665T4, Q3 NSS1C300ET4G, U1 FIN1048, U101 AD8599, U102 LTC2512-24, U104 THS4131, U2 FIN1047, U3 OP27, U4 OPA830, U5 74LVC541A, U6 OPA830, U7 MCP1755S-3302E/DB, U8 NCP1117STAT3G, U9 OPA1679, X1 channel_dummy, X2 channel_dummy

Commit message: Changed board connector to PCIe 8x, added test points, cleanup of component values. Add LVDS Rx termination, bypass caps.
Parts:
- removed FL1: 100uH, input:L_CommonMode_Wuerth_WE-SL3
- added C134: 1uF, Capacitor_SMD:C_0805_2012Metric, F.Cu at (144.5, 66.9)
- added C135: 1uF, Capacitor_SMD:C_0805_2012Metric, F.Cu at (98.5, 67.0)
- added C33: 100nF, Capacitor_SMD:C_0603_1608Metric, F.Cu at (271.8, 85.2)
- added C34: 100nF, Capacitor_SMD:C_0603_1608Metric, F.Cu at (280.2, 70.2)
- added D15: 10V (standoff), Diode_SMD:D_SMA, F.Cu at (213.2, 99.2)
- added D16: 5V (standoff), Diode_SMD:D_SMA, F.Cu at (225.5, 99.2)
- added J102: +IN, Connector_Coaxial:MMCX_Molex_73415-1471_Vertical, F.Cu at (158.5, 55.0)
- added J103: -IN, Connector_Coaxial:MMCX_Molex_73415-1471_Vertical, F.Cu at (158.5, 68.0)
- added J4: SCKA, Connector_Coaxial:MMCX_Molex_73415-1471_Vertical, F.Cu at (243.8, 87.5)
- added J5: SCKB, Connector_Coaxial:MMCX_Molex_73415-1471_Vertical, F.Cu at (251.0, 87.5)
- added J6: SDOB1, Connector_Coaxial:MMCX_Molex_73415-1471_Vertical, F.Cu at (258.3, 87.5)
- added P1: my_pcie_8x, input:BUS_PCIexpress_x8, B.Cu at (301.5, 59.5)
- added R133: GND lift, Resistor_SMD:R_0603_1608Metric, F.Cu at (157.2, 74.8)
- added R29: 100, Resistor_SMD:R_0603_1608Metric, F.Cu at (292.0, 85.2)
- added R30: 100, Resistor_SMD:R_0603_1608Metric, F.Cu at (294.2, 82.8)
- added R31: 100, Resistor_SMD:R_0603_1608Metric, F.Cu at (292.0, 80.2)
- added R32: 1K, Resistor_SMD:R_0603_1608Metric, F.Cu at (281.2, 86.8)
- added R33: 1K, Resistor_SMD:R_0603_1608Metric, F.Cu at (279.2, 86.8)
- added R34: 1K, Resistor_SMD:R_0603_1608Metric, F.Cu at (281.0, 75.5)
- added R35: 1K, Resistor_SMD:R_0603_1608Metric, F.Cu at (280.0, 68.0)
- added TP1: X+, TestPoint:TestPoint_THTPad_D1.5mm_Drill0.7mm, F.Cu at (37.8, 60.2)
- added TP103: SDOA, TestPoint:TestPoint_THTPad_D1.5mm_Drill0.7mm, F.Cu at (186.5, 68.2)
- added TP104: SDOB, TestPoint:TestPoint_THTPad_D1.5mm_Drill0.7mm, F.Cu at (186.5, 54.5)
- added TP105: +IN2, TestPoint:TestPoint_THTPad_D1.5mm_Drill0.7mm, F.Cu at (145.5, 55.0)
- added TP106: -IN2, TestPoint:TestPoint_THTPad_D1.5mm_Drill0.7mm, F.Cu at (145.5, 79.0)
- added TP107: -IN1, TestPoint:TestPoint_THTPad_D1.5mm_Drill0.7mm, F.Cu at (86.0, 78.0)
- added TP108: +IN1, TestPoint:TestPoint_THTPad_D1.5mm_Drill0.7mm, F.Cu at (86.0, 56.0)
- added TP2: X-, TestPoint:TestPoint_THTPad_D1.5mm_Drill0.7mm, F.Cu at (37.8, 74.0)
- added TP3: SYNC, TestPoint:TestPoint_THTPad_D1.5mm_Drill0.7mm, F.Cu at (258.5, 65.5)
- C111: value 34nF -> 33nF; footprint Capacitor_SMD:C_0603_1608Metric -> Capacitor_SMD:C_0805_2012Metric
- C112, C114: value 2.05nF -> 2.2nF; footprint Capacitor_SMD:C_0603_1608Metric -> Capacitor_SMD:C_0805_2012Metric
- C18, C19: value 1uF -> 100nF; footprint Capacitor_SMD:C_0805_2012Metric -> Capacitor_SMD:C_0603_1608Metric
- J2: value C64AB -> MCLK; footprint Connector_DIN:DIN41612_B_2x32_Horizontal -> Connector_Coaxial:MMCX_Molex_73415-1471_Vertical
- R1, R12, R2, R20, R3, R4: footprint Resistor_SMD:R_0805_2012Metric -> Resistor_SMD:R_0603_1608Metric
- R105, R106, R108, R110: value 1.07K -> 1K
- R107, R109: value 750 -> 698
- R111, R112, R23, R24, R25, R26: value 4.02K -> 3.3K; footprint Resistor_SMD:R_0805_2012Metric -> Resistor_SMD:R_0603_1608Metric
- U5: footprint Package_SO:SSOP-20_5.3x7.2mm_P0.65mm -> Package_SO:SSOP-20_4.4x6.5mm_P0.65mm
- moved TP102 144.8 mm to (179.0, 54.5)
- moved TP101 136.8 mm to (179.2, 68.5)
- moved C26 136.4 mm to (207.1, 58.1), turned to 0 degrees
- moved J2 135.8 mm to (236.5, 87.5), turned to 0 degrees
- moved R21 132.6 mm to (225.6, 55.5), turned to 180 degrees
- moved U8 131.4 mm to (218.3, 58.1), turned to 180 degrees
- moved FB3 129.8 mm to (291.1, 60.1), turned to 180 degrees
- moved C24 129.1 mm to (225.6, 58.1), turned to 0 degrees
- moved C131 128.8 mm to (89.5, 60.0), turned to 270 degrees
- moved C110 127.1 mm to (170.1, 75.3)
- moved D111 127.1 mm to (162.5, 76.2)
- moved R130 126.3 mm to (93.0, 56.8), turned to 0 degrees
- moved FB105 125.6 mm to (177.0, 73.2), turned to 270 degrees
- moved R22 125.6 mm to (225.6, 60.6), turned to 180 degrees
- moved R127 125.5 mm to (103.7, 61.0), turned to 180 degrees
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Connections:
- C16 pad 2: Net-(C16-Pad2) -> FILT_+10V
- C17 pad 1: Net-(C17-Pad1) -> FILT_-6V
- C18 pad 1: GND -> OVDD
- C18 pad 2: FILT_+10V -> GND
- C19 pad 1: FILT_-6V -> OVDD
- D107 pad 1: (no net) -> BIST+-_FB
- D107 pad 2: BIST+- -> (no net)
- D107 pad 3: BIST+-_FB -> BIST+-
- D108 pad 1: (no net) -> BIST--_FB
- D108 pad 2: BIST-- -> (no net)
- D108 pad 3: BIST--_FB -> BIST--
- D4 pad 1: Net-(C16-Pad2) -> FILT_+10V
- D8 pad 2: Net-(C17-Pad1) -> FILT_-6V
- FB1 pad 1: Net-(C17-Pad1) -> RAW_-6V
- FB2 pad 1: Net-(C16-Pad2) -> RAW_+10V
- RN2 pad 4: Net-(RN2-Pad4) -> Net-(R34-Pad1)
- RN2 pad 5: Net-(RN2-Pad5) -> /input_channel/SCKB
- U1 pad 11: /input_channel/SCKB -> Net-(R34-Pad1)
- U5 pad 11: Net-(RN2-Pad4) -> Net-(U5-Pad11)
- U5 pad 9: Net-(U5-Pad9) -> GND
Other:
- board outline added: 271.6 x 100 mm
- board text added: "CHAN_V+ pour"
- board text added: "CHAN_V- pour"
- board text added: "Earth/chassis ground"
- board text added: "Front high speed routing area"
- board text added: "Layer usage: Front: components and high speed digital, random local routing, mostly horizontal L2: ground, with tabs under the channels and an island for "Earth" at the input. L3: mostly horizontal, power busses and islands, misc low speed signals Back: mostly vertical. High speed signals need care about the reference plane, either GND or an L3 pour stitched to GND."
- board text added: "Low speed digital (I2C)"
- board text added: "OVDD BUS"
- board text added: "OVDD power zone"
- board text added: "Remote sense here at tap point"
- board text added: "V+ BUS"
- board text added: "V- BUS"
- board text added: "VDD BUS"
- board text added: "VREF BUS"

Commit message: Checkpoint before starting routing.  Added power and ground testpoints.
Parts:
- added R36: 499, Resistor_SMD:R_0805_2012Metric, F.Cu at (259.9, 112.5)
- added TP109: GND, TestPoint:TestPoint_THTPad_D1.5mm_Drill0.7mm, F.Cu at (158.5, 61.8)
- added TP110: VREF, TestPoint:TestPoint_THTPad_D1.5mm_Drill0.7mm, F.Cu at (166.2, 70.8)
- added TP4: GND, input:TestPoint_THTPad_D5.0mm_Drill2.41mm, F.Cu at (217.0, 119.0)
- added TP5: VREF, TestPoint:TestPoint_THTPad_D1.5mm_Drill0.7mm, F.Cu at (207.2, 95.8)
- added TP6: +3.3V, TestPoint:TestPoint_THTPad_D1.5mm_Drill0.7mm, F.Cu at (257.0, 57.5)
- added TP7: +2.5V, TestPoint:TestPoint_THTPad_D1.5mm_Drill0.7mm, F.Cu at (198.5, 53.5)
- added TP8: +8V, TestPoint:TestPoint_THTPad_D1.5mm_Drill0.7mm, F.Cu at (207.2, 102.4)
- added TP9: -4V, TestPoint:TestPoint_THTPad_D1.5mm_Drill0.7mm, F.Cu at (207.2, 109.0)
- C112, C114, C129, C130: footprint Capacitor_SMD:C_0805_2012Metric -> Capacitor_SMD:C_0603_1608Metric
- C122: footprint Capacitor_SMD:C_0603_1608Metric -> Capacitor_SMD:C_0805_2012Metric
- FB101, FB102, FB5, FB6: value 600 Ohm -> 2K Ohm
- R12, R20: value 399 -> 392
- R14: value 1K -> 499; footprint Resistor_SMD:R_0603_1608Metric -> Resistor_SMD:R_0805_2012Metric
- R23, R24, R25, R26: value 3.3K -> 200
- U1: value FIN1048 -> DS90LV048
- moved R105 16.0 mm to (130.0, 71.8)
- moved R106 16.0 mm to (130.0, 62.2)
- moved R108 16.0 mm to (130.0, 74.0)
- moved R109 16.0 mm to (130.0, 60.0)
- moved TP105 16.0 mm to (129.5, 55.0)
- moved TP106 16.0 mm to (129.5, 79.0)
- moved FB105 6.73 mm to (181.5, 78.2)
- moved R14 5.84 mm to (255.5, 112.5), turned to 0 degrees
- moved C111 5.50 mm to (133.8, 67.0)
- moved C112 5.50 mm to (136.6, 59.4)
- moved C114 5.50 mm to (136.6, 71.8)
- moved C115 5.50 mm to (142.0, 74.3)
- moved C117 5.50 mm to (145.5, 74.3)
- moved C118 5.50 mm to (145.5, 59.7)
- moved C134 5.50 mm to (150.0, 66.9)
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- renumbered E1 to E101
Connections:
- net +reference renamed VREF+
- net -reference renamed VREF-
- D12 pad 3: Net-(D12-Pad3) -> (no net)
- D13 pad 3: Net-(D13-Pad3) -> (no net)
- D14 pad 3: Net-(D14-Pad3) -> (no net)
- D2 pad 3: Net-(D2-Pad3) -> (no net)
- D3 pad 3: Net-(D3-Pad3) -> (no net)
- P1 pad A25: Net-(P1-PadA25) -> (no net)
- P1 pad A27: Net-(P1-PadA27) -> (no net)
- P1 pad A3: CARDSEL -> (no net)
- P1 pad A5: SCL -> (no net)
- P1 pad A8: Net-(P1-PadA8) -> (no net)
- P1 pad B25: Net-(P1-PadB25) -> (no net)
- P1 pad B27: Net-(P1-PadB27) -> (no net)
- P1 pad B5: SDA -> (no net)
- P1 pad B7: Net-(P1-PadB7) -> (no net)
- P1 pad B8: Net-(P1-PadB8) -> (no net)
- R14 pad 1: FILT_+10V -> Net-(C9-Pad2)
- R14 pad 2: Net-(C9-Pad2) -> Net-(R14-Pad2)
- U1 pad 10: Net-(U1-Pad10) -> (no net)
- U1 pad 7: Net-(U1-Pad7) -> (no net)
- U1 pad 8: Net-(U1-Pad8) -> (no net)
- U5 pad 11: Net-(U5-Pad11) -> (no net)
- X1 pad 7: /channel_dummy1/SDOB -> (no net)
- X2 pad 7: /channel_dummy2/SDOB -> (no net)
Other:
- net class Default: via_dia 0.8 -> 0.6; via_drill 0.4 -> 0.3
- net class Fast added: clearance 0.635, trace_width 0.15, via_dia 0.6, via_drill 0.3
- net class Ground added: clearance 0.2, trace_width 0.5, via_dia 0.6, via_drill 0.3
- net class LVDS added: clearance 0.635, trace_width 0.175, via_dia 0.6, via_drill 0.3
- net class Power added: clearance 0.2, trace_width 0.5, via_dia 0.6, via_drill 0.3
- net class Sensitive added: clearance 0.2, trace_width 0.15, via_dia 0.6, via_drill 0.3
- net class Slow added: clearance 0.2, trace_width 0.15, via_dia 0.6, via_drill 0.3
- rule trace_min: 0.2 -> 0.1016
- rule via_min_drill: 0.3 -> 0.2
- rule via_min_size: 0.4 -> 0.5

Commit message: Lots of work on routing input_board.kicad_pcb, not done yet.
Parts:
- removed TP104: SDOB, TestPoint:TestPoint_THTPad_D1.5mm_Drill0.7mm
- J2: value MCLK -> SCKB
- J5: value SCKB -> MCLK
- U1: footprint Package_SO:SOIC-16_3.9x9.9mm_P1.27mm -> Package_SO:TSSOP-16_4.4x5mm_P0.65mm
- moved R24 149.3 mm to (143.3, 171.1)
- moved R26 149.3 mm to (147.5, 171.1)
- moved R23 149.2 mm to (147.5, 168.1)
- moved R25 149.2 mm to (143.3, 168.1)
- moved R21 82.2 mm to (225.5, 137.7)
- moved R22 82.2 mm to (225.5, 142.8)
- moved C24 82.2 mm to (225.5, 140.2)
- moved U8 82.2 mm to (218.2, 140.2)
- moved C26 71.2 mm to (210.2, 129.2), turned to 270 degrees
- moved TP7 68.1 mm to (207.2, 121.0)
- moved C25 51.0 mm to (214.5, 59.2), turned to 270 degrees
- moved TP6 50.5 mm to (206.5, 58.5)
- moved TP4 31.9 mm to (227.8, 89.0)
- moved J6 30.5 mm to (286.5, 75.9)
- moved D16 18.4 mm to (222.2, 117.4), turned to 90 degrees
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Connections:
- net Net-(J102-Pad2) renamed /input_channel/ADC/J102_J103_GND
- net Net-(J2-Pad1) renamed /SCKB_JACK
- net Net-(J4-Pad1) renamed /SCKA_JACK
- net Net-(J5-Pad1) renamed /MCLK_JACK
- net Net-(J6-Pad1) renamed /SDOB1_JACK
- net Net-(TP101-Pad1) renamed /input_channel/ADC/DRL
- net Net-(TP102-Pad1) renamed /input_channel/ADC/BUSY
- R32 pad 1: Net-(R32-Pad1) -> /SCKB_RX
- R33 pad 1: Net-(R33-Pad1) -> /SCKA_RX
- R34 pad 1: Net-(R34-Pad1) -> /MCLK_RX
- RN1 pad 5: /input_channel/SCKA -> /channel_dummy1/SCKA
- RN1 pad 6: /channel_dummy2/MCLK -> /channel_dummy1/MCLK
- RN1 pad 7: /channel_dummy1/MCLK -> /channel_dummy2/SCKA
- RN1 pad 8: /input_channel/MCLK -> /channel_dummy2/MCLK
- RN2 pad 3: Net-(RN2-Pad3) -> /SCKB_RX
- RN2 pad 4: Net-(R34-Pad1) -> Net-(RN2-Pad4)
- RN2 pad 5: /input_channel/SCKB -> SYNC
- RN2 pad 6: SYNC -> /input_channel/SCKB
- RN2 pad 7: /channel_dummy2/SCKA -> /input_channel/SCKA
- RN2 pad 8: /channel_dummy1/SCKA -> /input_channel/MCLK
- U1 pad 11: Net-(R34-Pad1) -> /SCKB_RX
- U1 pad 14: Net-(R33-Pad1) -> /SCKA_RX
- U1 pad 15: Net-(R32-Pad1) -> /MCLK_RX
- U101 pad 2: /input_channel/in_amp/+in -> Net-(C129-Pad2)
- U101 pad 3: Net-(C129-Pad2) -> /input_channel/in_amp/+in
- U5 pad 12: Net-(RN2-Pad3) -> Net-(RN2-Pad4)
- U5 pad 2: Net-(R32-Pad1) -> /MCLK_RX
- U5 pad 3: Net-(R32-Pad1) -> /SCKA_RX
- U5 pad 4: Net-(R32-Pad1) -> /MCLK_RX
- U5 pad 5: Net-(R33-Pad1) -> /SCKA_RX
- U5 pad 6: Net-(R33-Pad1) -> /MCLK_RX
- U5 pad 7: Net-(R33-Pad1) -> /SCKA_RX
Routing:
- net PROBE_CONFIG: track 0.00 -> 299.9 mm, vias 0 -> 2
- net GND: track 0.00 -> 215.7 mm, vias 0 -> 91
- net SEL0: track 0.00 -> 185.2 mm, vias 0 -> 2
- net SEL1: track 0.00 -> 180.6 mm, vias 0 -> 2
- net FILT_+10V: track 0.00 -> 163.9 mm, vias 0 -> 4
- net /channel_dummy2/SDOA: track 0.00 -> 131.4 mm, vias 0 -> 2
- net V+: track 0.00 -> 128.3 mm, vias 0 -> 2
- net Net-(C23-Pad2): track 0.00 -> 122.5 mm, vias 0 -> 2
- net /channel_dummy2/SCKA: track 0.00 -> 122.0 mm
- net /channel_dummy2/MCLK: track 0.00 -> 121.1 mm
- net /channel_dummy1/SDOA: track 0.00 -> 111.2 mm, vias 0 -> 2
- net V-: track 0.00 -> 111.1 mm, vias 0 -> 2
- net /input_channel/SDOA: track 0.00 -> 106.5 mm, vias 0 -> 3
- net /input_channel/SDOB: track 0.00 -> 103.6 mm
- net SYNC: track 0.00 -> 95.6 mm, vias 0 -> 4
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- added copper zone on B.Cu, net /input_channel/ADC/J102_J103_GND
- added copper zone on In2.Cu, net /input_channel/antialias_driver/CHAN_V+
- added copper zone on In2.Cu, net /input_channel/antialias_driver/CHAN_V-
- added copper zone on In1.Cu, net GND
Other:
- net class 50 Ohm added: clearance 0.24, trace_width 0.36, via_dia 0.6, via_drill 0.3
- net class Fast: clearance 0.635 -> 0.2; via_dia 0.6 -> 0.45; via_drill 0.3 -> 0.2
- net class LVDS: clearance 0.635 -> 0.0889; via_dia 0.6 -> 0.45; via_drill 0.3 -> 0.2
- net class Slow: via_dia 0.6 -> 0.45; via_drill 0.3 -> 0.2
- rule via_min_size: 0.5 -> 0.45
- board text added: "Low speed digital"
- board text removed: "Low speed digital (I2C)"

Commit message: Minor tweaks to schematic, and ongoing progress on PCB layout.
Changed BIST buffer to run off of CHAN1_V+, not the global V+.  This caused the CHAN_V+ net name to change.
On power.sch, added bypass caps for the VREF inputs to the V+/V- regulators.  Also, the BIST input lines now
have an RC filter, not just a resistor.
Parts:
- added C35: 10nF, Capacitor_SMD:C_0805_2012Metric, F.Cu at (287.5, 123.2)
- added C36: 10nF, Capacitor_SMD:C_0805_2012Metric, F.Cu at (287.5, 119.1)
- added C37: 10nF, Capacitor_SMD:C_0805_2012Metric, F.Cu at (287.5, 131.2)
- added C38: 10nF, Capacitor_SMD:C_0805_2012Metric, F.Cu at (287.5, 127.2)
- added C39: 1uF, Capacitor_SMD:C_0805_2012Metric, F.Cu at (250.2, 111.2)
- added C40: 1uF, Capacitor_SMD:C_0805_2012Metric, F.Cu at (243.5, 119.8)
- moved R24 154.1 mm to (287.7, 117.1)
- moved R25 149.5 mm to (287.7, 129.2)
- moved R23 147.9 mm to (287.7, 121.1)
- moved R26 147.6 mm to (287.7, 125.2)
- moved R22 51.1 mm to (222.5, 91.7), turned to 0 degrees
- moved U8 49.1 mm to (228.3, 92.2), turned to 90 degrees
- moved C24 46.0 mm to (222.5, 94.3), turned to 180 degrees
- moved R21 41.3 mm to (222.5, 96.5)
- moved C26 36.7 mm to (212.0, 92.5)
- moved TP4 30.9 mm to (232.5, 58.5)
- moved TP7 29.6 mm to (205.5, 91.5)
- moved D15 26.0 mm to (212.5, 119.5), turned to 180 degrees
- moved R16 14.5 mm to (269.2, 130.2), turned to 0 degrees
- moved TP103 9.96 mm to (190.8, 59.8)
- moved C5 8.27 mm to (211.0, 101.2)
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Connections:
- C10 pad 1: GND -> Net-(C10-Pad1)
- C117 pad 2: /input_channel/antialias_driver/CHAN_V+ -> CHAN1_V+
- C118 pad 2: /input_channel/antialias_driver/CHAN_V- -> CHAN1_V-
- C119 pad 1: /input_channel/antialias_driver/CHAN_V+ -> CHAN1_V+
- C123 pad 2: /input_channel/antialias_driver/CHAN_V+ -> CHAN1_V+
- C124 pad 2: /input_channel/antialias_driver/CHAN_V- -> CHAN1_V-
- C125 pad 2: /input_channel/antialias_driver/CHAN_V+ -> CHAN1_V+
- C126 pad 2: /input_channel/antialias_driver/CHAN_V- -> CHAN1_V-
- C131 pad 2: /input_channel/antialias_driver/CHAN_V+ -> CHAN1_V+
- C132 pad 2: /input_channel/antialias_driver/CHAN_V- -> CHAN1_V-
- C133 pad 2: /input_channel/antialias_driver/CHAN_V- -> CHAN1_V-
- C134 pad 1: /input_channel/antialias_driver/CHAN_V- -> CHAN1_V-
- C134 pad 2: /input_channel/antialias_driver/CHAN_V+ -> CHAN1_V+
- C135 pad 1: /input_channel/antialias_driver/CHAN_V- -> CHAN1_V-
- C135 pad 2: /input_channel/antialias_driver/CHAN_V+ -> CHAN1_V+
- C27 pad 2: V+ -> CHAN1_V+
- C28 pad 2: V- -> CHAN1_V-
- D103 pad 1: /input_channel/antialias_driver/CHAN_V- -> CHAN1_V-
- D103 pad 2: /input_channel/antialias_driver/CHAN_V+ -> CHAN1_V+
- D104 pad 1: /input_channel/antialias_driver/CHAN_V- -> CHAN1_V-
- D104 pad 2: /input_channel/antialias_driver/CHAN_V+ -> CHAN1_V+
- D12 pad 3: (no net) -> Net-(D12-Pad3)
- D13 pad 3: (no net) -> Net-(D13-Pad3)
- D14 pad 3: (no net) -> Net-(D14-Pad3)
- D2 pad 3: (no net) -> Net-(D2-Pad3)
- D3 pad 3: (no net) -> Net-(D3-Pad3)
- FB103 pad 2: /input_channel/antialias_driver/CHAN_V+ -> CHAN1_V+
- FB104 pad 2: /input_channel/antialias_driver/CHAN_V- -> CHAN1_V-
- J1 pad 4: /channel_dummy2/+in -> /channel_dummy3/+in
- J1 pad 5: /channel_dummy2/-in -> /channel_dummy3/-in
- J1 pad 7: /channel_dummy1/-in -> /channel_dummy2/-in
- J1 pad 8: /channel_dummy1/+in -> /channel_dummy2/+in
- P1 pad A25: (no net) -> Net-(P1-PadA25)
- P1 pad A27: (no net) -> Net-(P1-PadA27)
- P1 pad A3: (no net) -> CARDSEL
- P1 pad A5: (no net) -> SCL
- P1 pad A8: (no net) -> Net-(P1-PadA8)
- P1 pad B25: (no net) -> Net-(P1-PadB25)
- P1 pad B27: (no net) -> Net-(P1-PadB27)
- P1 pad B5: (no net) -> SDA
- P1 pad B7: (no net) -> Net-(P1-PadB7)
- P1 pad B8: (no net) -> Net-(P1-PadB8)
- RN1 pad 5: /channel_dummy1/SCKA -> /channel_dummy2/SCKA
- RN1 pad 6: /channel_dummy1/MCLK -> /channel_dummy2/MCLK
- RN1 pad 7: /channel_dummy2/SCKA -> /channel_dummy3/SCKA
- RN1 pad 8: /channel_dummy2/MCLK -> /channel_dummy3/MCLK
- U1 pad 10: (no net) -> Net-(U1-Pad10)
- U1 pad 7: (no net) -> Net-(U1-Pad7)
- U1 pad 8: (no net) -> Net-(U1-Pad8)
- U101 pad 4: /input_channel/antialias_driver/CHAN_V- -> CHAN1_V-
- U101 pad 8: /input_channel/antialias_driver/CHAN_V+ -> CHAN1_V+
- U104 pad 3: /input_channel/antialias_driver/CHAN_V+ -> CHAN1_V+
- U104 pad 6: /input_channel/antialias_driver/CHAN_V- -> CHAN1_V-
- U2 pad 6: /channel_dummy1/SDOA -> /channel_dummy2/SDOA
- U2 pad 7: /channel_dummy2/SDOA -> /channel_dummy3/SDOA
- U5 pad 11: (no net) -> Net-(U5-Pad11)
- U9 pad 11: V- -> CHAN1_V-
- U9 pad 4: V+ -> CHAN1_V+
- X1 pad 1: /channel_dummy1/MCLK -> /channel_dummy2/MCLK
- X1 pad 2: /channel_dummy1/SCKA -> /channel_dummy2/SCKA
- X1 pad 4: /channel_dummy1/+in -> /channel_dummy2/+in
- X1 pad 5: /channel_dummy1/-in -> /channel_dummy2/-in
- X1 pad 6: /channel_dummy1/SDOA -> /channel_dummy2/SDOA
- X1 pad 7: (no net) -> /channel_dummy2/SDOB
- X2 pad 1: /channel_dummy2/MCLK -> /channel_dummy3/MCLK
- X2 pad 2: /channel_dummy2/SCKA -> /channel_dummy3/SCKA
- X2 pad 4: /channel_dummy2/+in -> /channel_dummy3/+in
- X2 pad 5: /channel_dummy2/-in -> /channel_dummy3/-in
- X2 pad 6: /channel_dummy2/SDOA -> /channel_dummy3/SDOA
- X2 pad 7: (no net) -> /channel_dummy3/SDOB
Routing:
- net V+: track 128.3 -> 391.6 mm, vias 2 -> 12
- net /channel_dummy3/SDOA: track 0.00 -> 261.2 mm, vias 0 -> 2
- net /channel_dummy3/SCKA: track 0.00 -> 255.4 mm
- net /channel_dummy3/MCLK: track 0.00 -> 250.0 mm
- net V-: track 111.1 -> 348.1 mm, vias 2 -> 12
- net VREF: track 80.5 -> 210.0 mm, vias 3 -> 18
- net GND: track 215.7 -> 333.8 mm, vias 91 -> 150
- net /channel_dummy1/SDOA: track 111.2 -> 0.00 mm, vias 2 -> 0
- net /channel_dummy2/MCLK: track 121.1 -> 217.0 mm
- net CHAN1_V+: track 0.00 -> 94.4 mm, vias 0 -> 17
- net /channel_dummy2/SDOA: track 131.4 -> 225.6 mm
- net CHAN1_V-: track 0.00 -> 94.2 mm, vias 0 -> 14
- net /channel_dummy2/SCKA: track 122.0 -> 214.1 mm
- net /channel_dummy1/SCKA: track 87.0 -> 0.00 mm
- net VDD: track 26.1 -> 107.0 mm, vias 0 -> 7
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- added copper zone on In2.Cu, net CHAN1_V+
- added copper zone on In2.Cu, net CHAN1_V-
- added copper zone on In1.Cu, net Earth
- added copper zone on In2.Cu, net OVDD
- added copper zone on In2.Cu, net V+
- added copper zone on In2.Cu, net V-
- added copper zone on In2.Cu, net VDD
- added copper zone on In2.Cu, net VREF
- removed copper zone on In2.Cu, net /input_channel/antialias_driver/CHAN_V+
- removed copper zone on In2.Cu, net /input_channel/antialias_driver/CHAN_V-
Other:
- board text removed: "Remote sense here at tap point"

Commit message: Snapshot before replicating input channels
Parts:
- moved C32 159.2 mm to (200.8, 143.8), turned to 90 degrees
- moved TP4 77.5 mm to (210.2, 132.8)
- moved C120 1.75 mm to (39.5, 65.8)
- moved C121 1.75 mm to (39.5, 68.3)
- moved D101 1.75 mm to (51.0, 63.0)
- moved D102 1.75 mm to (51.0, 71.0)
- moved E101 1.75 mm to (32.1, 67.0)
- moved FB101 1.75 mm to (39.5, 63.5)
- moved FB102 1.75 mm to (39.5, 70.5)
- moved FL101 1.75 mm to (48.2, 67.0)
- moved TP1 1.75 mm to (36.0, 60.2)
- moved TP2 1.75 mm to (36.0, 74.0)
- moved J102 1.50 mm to (158.5, 56.5)
- moved TP109 1.06 mm to (159.2, 62.2)
- moved TP106 1.00 mm to (129.5, 78.0)
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Routing:
- net Earth: track 11.8 -> 318.1 mm, vias 3 -> 12
- net Net-(C36-Pad2): track 2.17 -> 289.3 mm, vias 0 -> 5
- net Net-(C38-Pad2): track 2.17 -> 285.4 mm, vias 0 -> 5
- net Net-(C35-Pad2): track 2.17 -> 283.5 mm, vias 0 -> 4
- net Net-(C37-Pad2): track 2.17 -> 280.2 mm, vias 0 -> 4
- net GND: track 333.8 -> 521.8 mm, vias 150 -> 186
- net /input_channel/ADC/CHAN_VREF: track 43.9 -> 106.8 mm, vias 0 -> 27
- net /input_channel/+in: track 37.7 -> 13.0 mm, vias 1 -> 0
- net /input_channel/-in: track 32.0 -> 12.6 mm
- net V-: track 348.1 -> 361.2 mm
- net /input_channel/antialias_driver/-in: track 46.2 -> 53.3 mm
- net /input_channel/antialias_driver/+in: track 46.3 -> 53.2 mm
- net RAW_+10V: track 17.1 -> 23.8 mm, vias 0 -> 1
- net RAW_-6V: track 18.3 -> 24.2 mm, vias 0 -> 1
- net VREF: track 210.0 -> 212.2 mm
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- added copper zone on F.Cu, net /input_channel/ADC/CHAN_VREF
- added copper zone on In2.Cu, net /input_channel/ADC/CHAN_VREF
- added copper zone on B.Cu, net GND
- added copper zone on F.Cu, net GND
- added copper zone on In2.Cu, net GND
- added copper zone on F.Cu, net OVDD
- added copper zone on F.Cu, net VDD
