File: input/probe_connector.sch (KiCad schematic (older format))
At the start: 5 parts, among them J1 Sensor

Commit message: Cleanup to get ready to start board layout. I had to get rid off all the bus signals, since in Kicad busses don't work that way.  Added a couple testpoints; many more needed.
Work on component placement in PCB.  I changed DGND to plain GND and "protective earth" to
"earth" (for chassis ground).  Chassis ground is now connected on the board only via a capacitor.
I had to fix the connector footprint to match the pin numbers on the symbol (there was a case
difference).
Parts:
- FB5, FB6: footprint digikey-footprints:0805 -> Inductor_SMD:L_0805_2012Metric
Connections:
- net labels added: Earth
- net labels removed: Earth_Protective, Inputs
Other:
- moved on the sheet: D9
Changed lines of the file:
@@
 	2650 3250 2650 3300
-$Comp
-L power:Earth_Protective #PWR?
-U 1 1 5E75AFB4
-P 2650 3400
-AR Path="/5E75AFB4" Ref="#PWR?"  Part="1"
-AR Path="/5E756356/5E75AFB4" Ref="#PWR04"  Part="1"
-F 0 "#PWR04" H 2900 3150 50  0001 C CNN
-F 1 "Earth_Protective" H 3100 3250 50  0001 C CNN
-F 2 "" H 2650 3300 50  0001 C CNN
-F 3 "~" H 2650 3300 50  0001 C CNN
-	1    2650 3400
-	1    0    0    -1
-$EndComp
 $Comp
 L Connector:RJ45_Shielded J?
@@
 Wire Wire Line
 	2650 3300 2650 3400
-Wire Bus Line
-	4600 3100 4800 3100
-Text HLabel 4800 3100 2    50   Output ~ 0
-Inputs
-Entry Wire Line
-	4500 2350 4600 2450
-Entry Wire Line
-	4500 2450 4600 2550
-Entry Wire Line
-	4500 2550 4600 2650
-Entry Wire Line
-	4500 2650 4600 2750
-Entry Wire Line
-	4500 2750 4600 2850
-Entry Wire Line
-	4500 2850 4600 2950
 Wire Wire Line
 	3050 2350 4500 2350
@@
 F 0 "FB5" H 4000 4337 60  0000 C CNN
 F 1 "600 Ohm" H 4000 4231 60  0000 C CNN
-F 2 "digikey-footprints:0805" H 4200 4250 60  0001 L CNN
+F 2 "Inductor_SMD:L_0805_2012Metric" H 4200 4250 60  0001 L CNN
 F 3 "" H 4200 4350 60  0001 L CNN
 F 4 " 240-2396-1-ND" H 4200 4450 60  0001 L CNN "Digi-Key_PN"
@@
 L Device:D_Zener D?
 U 1 1 5E7695B8
-P 5550 4450
+P 5550 4400
 AR Path="/5E51E83D/5E7695B8" Ref="D?"  Part="1"
 AR Path="/5E756356/5E7695B8" Ref="D9"  Part="1"
-F 0 "D9" H 5550 4550 50  0000 C CNN
-F 1 "5V (standoff)" H 5650 4250 50  0000 C CNN
-F 2 "Diode_SMD:D_SMA" H 5550 4450 50  0001 C CNN
-F 3 "https://katalog.we-online.de/pbs/datasheet/824500500.pdf" H 5550 4450 50  0001 C CNN
-F 4 "824500500" H 5550 4450 50  0001 C CNN "MPN"
-F 5 "TVS DIODE 5V 9.2V DO214AC" H 5550 4450 50  0001 C CNN "Description"
-F 6 "732-9974-1-ND" H 5550 4450 50  0001 C CNN "Digikey"
-	1    5550 4450
+F 0 "D9" H 5550 4500 50  0000 C CNN
+F 1 "5V (standoff)" H 5650 4200 50  0000 C CNN
+F 2 "Diode_SMD:D_SMA" H 5550 4400 50  0001 C CNN
+F 3 "https://katalog.we-online.de/pbs/datasheet/824500500.pdf" H 5550 4400 50  0001 C CNN
+F 4 "824500500" H 5550 4400 50  0001 C CNN "MPN"
+F 5 "TVS DIODE 5V 9.2V DO214AC" H 5550 4400 50  0001 C CNN "Description"
+F 6 "732-9974-1-ND" H 5550 4400 50  0001 C CNN "Digikey"
+	1    5550 4400
 	0    1    1    0
 $EndComp
 Wire Wire Line
-	5550 4050 5550 4300
-$Comp
-L power:Earth_Protective #PWR?
-U 1 1 5E75F219
-P 5550 4700
-AR Path="/5DFCF14D/5DE42731/5E75F219" Ref="#PWR?"  Part="1"
-AR Path="/5E756356/5E75F219" Ref="#PWR049"  Part="1"
-F 0 "#PWR049" H 5800 4450 50  0001 C CNN
-F 1 "Earth_Protective" H 6000 4550 50  0001 C CNN
-F 2 "" H 5550 4600 50  0001 C CNN
-F 3 "~" H 5550 4600 50  0001 C CNN
-	1    5550 4700
-	1    0    0    -1
-$EndComp
+	5550 4050 5550 4250
 Wire Wire Line
-	5550 4600 5550 4700
+	5550 4550 5550 4650
 $Comp
 L dk_Ferrite-Beads-and-Chips:MPZ2012S601AT000 FB?
@@
 F 0 "FB6" H 5000 4337 60  0000 C CNN
 F 1 "600 Ohm" H 5000 4231 60  0000 C CNN
-F 2 "digikey-footprints:0805" H 5200 4250 60  0001 L CNN
+F 2 "Inductor_SMD:L_0805_2012Metric" H 5200 4250 60  0001 L CNN
 F 3 "" H 5200 4350 60  0001 L CNN
 F 4 " 240-2396-1-ND" H 5200 4450 60  0001 L CNN "Digi-Key_PN"
@@
 Wire Wire Line
 	4450 4050 4800 4050
-$Comp
-L power:Earth_Protective #PWR?
-U 1 1 5E76FD86
-P 4450 4650
-AR Path="/5DFCF14D/5DE42731/5E76FD86" Ref="#PWR?"  Part="1"
-AR Path="/5E756356/5E76FD86" Ref="#PWR048"  Part="1"
-F 0 "#PWR048" H 4700 4400 50  0001 C CNN
-F 1 "Earth_Protective" H 4900 4500 50  0001 C CNN
-F 2 "" H 4450 4550 50  0001 C CNN
-F 3 "~" H 4450 4550 50  0001 C CNN
-	1    4450 4650
-	1    0    0    -1
-$EndComp
 Wire Wire Line
 	4450 4450 4450 4650
@@
 	5800 4050 5550 4050
 Connection ~ 5550 4050
-Wire Bus Line
-	4600 2400 4600 3100
 Text Notes 3250 2150 0    50   ~ 0
 This pinout uses the pairs in \n T-568B RJ45 ethernet cable
+Text HLabel 4500 2350 2    50   Output ~ 0
+Y+
+Text HLabel 4500 2450 2    50   Output ~ 0
+Y-
+Text HLabel 4500 2550 2    50   Output ~ 0
+X+
+Text HLabel 4500 2650 2    50   Output ~ 0
+Z-
+Text HLabel 4500 2750 2    50   Output ~ 0
+Z+
+Text HLabel 4500 2850 2    50   Output ~ 0
+X-
+$Comp
+L power:Earth #PWR0155
+U 1 1 5E36FAA0
+P 2650 3400
+F 0 "#PWR0155" H 2650 3150 50  0001 C CNN
+F 1 "Earth" H 2650 3250 50  0001 C CNN
+F 2 "" H 2650 3400 50  0001 C CNN
+F 3 "~" H 2650 3400 50  0001 C CNN
+	1    2650 3400
+	1    0    0    -1
+$EndComp
+$Comp
+L power:Earth #PWR0156
+U 1 1 5E36FFC7
+P 4450 4650
+F 0 "#PWR0156" H 4450 4400 50  0001 C CNN
+F 1 "Earth" H 4450 4500 50  0001 C CNN
+F 2 "" H 4450 4650 50  0001 C CNN
+F 3 "~" H 4450 4650 50  0001 C CNN
+	1    4450 4650
+	1    0    0    -1
+$EndComp
+$Comp
+L power:Earth #PWR0157
+U 1 1 5E370459
+P 5550 4650
+F 0 "#PWR0157" H 5550 4400 50  0001 C CNN
+F 1 "Earth" H 5550 4500 50  0001 C CNN
+F 2 "" H 5550 4650 50  0001 C CNN
+F 3 "~" H 5550 4650 50  0001 C CNN
+	1    5550 4650
+	1    0    0    -1
+$EndComp
 $EndSCHEMATC

Commit message: Changed board connector to PCIe 8x, added test points, cleanup of component values. Add LVDS Rx termination, bypass caps.
Parts:
- added TP1: X+, TestPoint:TestPoint_THTPad_D1.5mm_Drill0.7mm, symbol Connector:TestPoint
- added TP2: X-, TestPoint:TestPoint_THTPad_D1.5mm_Drill0.7mm, symbol Connector:TestPoint
Connections:
- net X+: now also TP1.1
- net X-: now also TP2.1
Changed lines of the file:
@@
 	3050 2450 4500 2450
 Wire Wire Line
-	3050 2550 4500 2550
-Wire Wire Line
-	3050 2650 4500 2650
+	3050 2550 4200 2550
 Wire Wire Line
 	3050 2750 4500 2750
 Wire Wire Line
-	3050 2850 4500 2850
+	3050 2850 4400 2850
 Text Label 4100 2850 2    50   ~ 0
 X-
@@
 	1    0    0    -1
 $EndComp
+$Comp
+L Connector:TestPoint TP?
+U 1 1 5E5ADFFD
+P 4200 2950
+AR Path="/5DFCF14D/5DA78AA2/5E5ADFFD" Ref="TP?"  Part="1"
+AR Path="/5DFCF14D/5E295469/5E5ADFFD" Ref="TP?"  Part="1"
+AR Path="/5DFCF14D/5E195558/5E5ADFFD" Ref="TP?"  Part="1"
+AR Path="/5E756356/5E5ADFFD" Ref="TP1"  Part="1"
+F 0 "TP1" H 4200 3200 50  0000 C CNN
+F 1 "X+" H 4200 3300 50  0000 C CNN
+F 2 "TestPoint:TestPoint_THTPad_D1.5mm_Drill0.7mm" H 4400 2950 50  0001 C CNN
+F 3 "~" H 4400 2950 50  0001 C CNN
+	1    4200 2950
+	-1   0    0    1
+$EndComp
+$Comp
+L Connector:TestPoint TP?
+U 1 1 5E5AE003
+P 4400 2950
+AR Path="/5DFCF14D/5DA78AA2/5E5AE003" Ref="TP?"  Part="1"
+AR Path="/5DFCF14D/5E295469/5E5AE003" Ref="TP?"  Part="1"
+AR Path="/5DFCF14D/5E195558/5E5AE003" Ref="TP?"  Part="1"
+AR Path="/5E756356/5E5AE003" Ref="TP2"  Part="1"
+F 0 "TP2" H 4400 3200 50  0000 C CNN
+F 1 "X-" H 4400 3300 50  0000 C CNN
+F 2 "TestPoint:TestPoint_THTPad_D1.5mm_Drill0.7mm" H 4600 2950 50  0001 C CNN
+F 3 "~" H 4600 2950 50  0001 C CNN
+	1    4400 2950
+	-1   0    0    1
+$EndComp
+Wire Wire Line
+	4200 2950 4200 2550
+Connection ~ 4200 2550
+Wire Wire Line
+	4200 2550 4500 2550
+Wire Wire Line
+	3050 2650 4500 2650
+Wire Wire Line
+	4400 2950 4400 2850
+Connection ~ 4400 2850
+Wire Wire Line
+	4400 2850 4500 2850
 $EndSCHEMATC

Commit message: Checkpoint before starting routing.  Added power and ground testpoints.
Parts:
- C31: DK line (none) -> 1; Description (none) -> CAP CER 1000PF 100V NPO 0805
- D9: DK line (none) -> 40
- FB5, FB6: value 600 Ohm -> 2K Ohm; DK line (none) -> 5; Description FERRITE BEAD 600 OHM 0805 1LN -> FERRITE BEAD 2 KOHM 0805 1LN; Digikey (none) -> 240-2396-1-ND
- J1: DK line (none) -> 18
Changed lines of the file:
@@
 EESchema Schematic File Version 4
-LIBS:input_board-cache
-EELAYER 29 0
+EELAYER 30 0
 EELAYER END
 $Descr A4 11693 8268
@@
 F 5 "RJHSE5387" H 2650 2750 50  0001 C CNN "MPN"
 F 6 "CONN MOD JACK 8P8C R/A SHIELDED" H 2650 2750 50  0001 C CNN "Description"
+F 7 "18" H 2650 2750 50  0001 C CNN "DK line"
 	1    2650 2750
 	1    0    0    -1
@@
 AR Path="/5E756356/5E75F20B" Ref="FB5"  Part="1"
 F 0 "FB5" H 4000 4337 60  0000 C CNN
-F 1 "600 Ohm" H 4000 4231 60  0000 C CNN
+F 1 "2K Ohm" H 4000 4231 60  0000 C CNN
 F 2 "Inductor_SMD:L_0805_2012Metric" H 4200 4250 60  0001 L CNN
-F 3 "" H 4200 4350 60  0001 L CNN
+F 3 "https://assets.lairdtech.com/home/brandworld/files/Catalog_EMI%20FILTERING%20RF%200717.pdf" H 4200 4350 60  0001 L CNN
 F 4 " 240-2396-1-ND" H 4200 4450 60  0001 L CNN "Digi-Key_PN"
 F 5 "HZ0805C202R-10" H 4200 4550 60  0001 L CNN "MPN"
@@
 F 8 "https://product.tdk.com/info/en/catalog/datasheets/beads_commercial_power_mpz2012_en.pdf" H 4200 4850 60  0001 L CNN "DK_Datasheet_Link"
 F 9 "/product-detail/en/tdk-corporation/MPZ2012S601AT000/445-2206-1-ND/765104" H 4200 4950 60  0001 L CNN "DK_Detail_Page"
-F 10 "FERRITE BEAD 600 OHM 0805 1LN" H 4200 5050 60  0001 L CNN "Description"
+F 10 "FERRITE BEAD 2 KOHM 0805 1LN" H 4200 5050 60  0001 L CNN "Description"
 F 11 "TDK Corporation" H 4200 5150 60  0001 L CNN "Manufacturer"
 F 12 "Active" H 4200 5250 60  0001 L CNN "Status"
+F 13 "5" H 4000 4050 50  0001 C CNN "DK line"
+F 14 "240-2396-1-ND" H 4000 4050 50  0001 C CNN "Digikey"
 	1    4000 4050
 	1    0    0    -1
@@
 F 5 "TVS DIODE 5V 9.2V DO214AC" H 5550 4400 50  0001 C CNN "Description"
 F 6 "732-9974-1-ND" H 5550 4400 50  0001 C CNN "Digikey"
+F 7 "40" H 5550 4400 50  0001 C CNN "DK line"
 	1    5550 4400
 	0    1    1    0
@@
 AR Path="/5E756356/5E76B461" Ref="FB6"  Part="1"
 F 0 "FB6" H 5000 4337 60  0000 C CNN
-F 1 "600 Ohm" H 5000 4231 60  0000 C CNN
+F 1 "2K Ohm" H 5000 4231 60  0000 C CNN
 F 2 "Inductor_SMD:L_0805_2012Metric" H 5200 4250 60  0001 L CNN
-F 3 "" H 5200 4350 60  0001 L CNN
+F 3 "https://assets.lairdtech.com/home/brandworld/files/Catalog_EMI%20FILTERING%20RF%200717.pdf" H 5200 4350 60  0001 L CNN
 F 4 " 240-2396-1-ND" H 5200 4450 60  0001 L CNN "Digi-Key_PN"
 F 5 "HZ0805C202R-10" H 5200 4550 60  0001 L CNN "MPN"
@@
 F 8 "https://product.tdk.com/info/en/catalog/datasheets/beads_commercial_power_mpz2012_en.pdf" H 5200 4850 60  0001 L CNN "DK_Datasheet_Link"
 F 9 "/product-detail/en/tdk-corporation/MPZ2012S601AT000/445-2206-1-ND/765104" H 5200 4950 60  0001 L CNN "DK_Detail_Page"
-F 10 "FERRITE BEAD 600 OHM 0805 1LN" H 5200 5050 60  0001 L CNN "Description"
+F 10 "FERRITE BEAD 2 KOHM 0805 1LN" H 5200 5050 60  0001 L CNN "Description"
 F 11 "TDK Corporation" H 5200 5150 60  0001 L CNN "Manufacturer"
 F 12 "Active" H 5200 5250 60  0001 L CNN "Status"
+F 13 "5" H 5000 4050 50  0001 C CNN "DK line"
+F 14 "240-2396-1-ND" H 5000 4050 50  0001 C CNN "Digikey"
 	1    5000 4050
 	1    0    0    -1
@@
 F 4 "311-3585-1-ND" H 4450 4350 50  0001 C CNN "Digikey"
 F 5 "CC0805FRNPO0BN102" H 4450 4350 50  0001 C CNN "MPN"
+F 6 "CAP CER 1000PF 100V NPO 0805" H 4450 4350 50  0001 C CNN "Description"
+F 7 "1" H 4450 4350 50  0001 C CNN "DK line"
 	1    4450 4350
 	1    0    0    -1

Commit message: Work on main board.
Changed lines of the file:
@@
 $Descr A4 11693 8268
 encoding utf-8
-Sheet 6 21
+Sheet 6 33
 Title ""
 Date ""
@@
 AR Path="/5E75AFBD" Ref="J?"  Part="1"
 AR Path="/5E756356/5E75AFBD" Ref="J1"  Part="1"
-F 0 "J1" H 2450 3300 50  0000 R CNN
+AR Path="/5E624B3C/5E756356/5E75AFBD" Ref="J1"  Part="1"
+F 0 "J?" H 2450 3300 50  0000 R CNN
 F 1 "Sensor" H 2550 3300 50  0000 L CNN
 F 2 "Connector_RJ:RJ45_Amphenol_RJHSE538X" V 2650 2775 50  0001 C CNN
@@
 AR Path="/5DFCF14D/5DE42731/5E75F20B" Ref="FB?"  Part="1"
 AR Path="/5E756356/5E75F20B" Ref="FB5"  Part="1"
-F 0 "FB5" H 4000 4337 60  0000 C CNN
+AR Path="/5E624B3C/5E756356/5E75F20B" Ref="FB5"  Part="1"
+F 0 "FB?" H 4000 4337 60  0000 C CNN
 F 1 "2K Ohm" H 4000 4231 60  0000 C CNN
 F 2 "Inductor_SMD:L_0805_2012Metric" H 4200 4250 60  0001 L CNN
@@
 AR Path="/5E51E83D/5E7695B8" Ref="D?"  Part="1"
 AR Path="/5E756356/5E7695B8" Ref="D9"  Part="1"
-F 0 "D9" H 5550 4500 50  0000 C CNN
+AR Path="/5E624B3C/5E756356/5E7695B8" Ref="D9"  Part="1"
+F 0 "D?" H 5550 4500 50  0000 C CNN
 F 1 "5V (standoff)" H 5650 4200 50  0000 C CNN
 F 2 "Diode_SMD:D_SMA" H 5550 4400 50  0001 C CNN
@@
 AR Path="/5DFCF14D/5DE42731/5E76B461" Ref="FB?"  Part="1"
 AR Path="/5E756356/5E76B461" Ref="FB6"  Part="1"
-F 0 "FB6" H 5000 4337 60  0000 C CNN
+AR Path="/5E624B3C/5E756356/5E76B461" Ref="FB6"  Part="1"
+F 0 "FB?" H 5000 4337 60  0000 C CNN
 F 1 "2K Ohm" H 5000 4231 60  0000 C CNN
 F 2 "Inductor_SMD:L_0805_2012Metric" H 5200 4250 60  0001 L CNN
@@
 AR Path="/5DFCF14D/5DE42731/5E76E2C4" Ref="C?"  Part="1"
 AR Path="/5E756356/5E76E2C4" Ref="C31"  Part="1"
-F 0 "C31" H 4542 4396 50  0000 L CNN
+AR Path="/5E624B3C/5E756356/5E76E2C4" Ref="C31"  Part="1"
+F 0 "C?" H 4542 4396 50  0000 L CNN
 F 1 "1nF" H 4542 4305 50  0000 L CNN
 F 2 "Capacitor_SMD:C_0805_2012Metric" H 4450 4350 50  0001 C CNN
@@
 X-
 $Comp
-L power:Earth #PWR0155
+L power:Earth #PWR?
 U 1 1 5E36FAA0
 P 2650 3400
-F 0 "#PWR0155" H 2650 3150 50  0001 C CNN
+F 0 "#PWR?" H 2650 3150 50  0001 C CNN
 F 1 "Earth" H 2650 3250 50  0001 C CNN
 F 2 "" H 2650 3400 50  0001 C CNN
@@
 $EndComp
 $Comp
-L power:Earth #PWR0156
+L power:Earth #PWR?
 U 1 1 5E36FFC7
 P 4450 4650
-F 0 "#PWR0156" H 4450 4400 50  0001 C CNN
+F 0 "#PWR?" H 4450 4400 50  0001 C CNN
 F 1 "Earth" H 4450 4500 50  0001 C CNN
 F 2 "" H 4450 4650 50  0001 C CNN
@@
 $EndComp
 $Comp
-L power:Earth #PWR0157
+L power:Earth #PWR?
 U 1 1 5E370459
 P 5550 4650
-F 0 "#PWR0157" H 5550 4400 50  0001 C CNN
+F 0 "#PWR?" H 5550 4400 50  0001 C CNN
 F 1 "Earth" H 5550 4500 50  0001 C CNN
 F 2 "" H 5550 4650 50  0001 C CNN
@@
 AR Path="/5DFCF14D/5E195558/5E5ADFFD" Ref="TP?"  Part="1"
 AR Path="/5E756356/5E5ADFFD" Ref="TP1"  Part="1"
-F 0 "TP1" H 4200 3200 50  0000 C CNN
+AR Path="/5E624B3C/5E756356/5E5ADFFD" Ref="TP1"  Part="1"
+F 0 "TP?" H 4200 3200 50  0000 C CNN
 F 1 "X+" H 4200 3300 50  0000 C CNN
 F 2 "TestPoint:TestPoint_THTPad_D1.5mm_Drill0.7mm" H 4400 2950 50  0001 C CNN
@@
 AR Path="/5DFCF14D/5E195558/5E5AE003" Ref="TP?"  Part="1"
 AR Path="/5E756356/5E5AE003" Ref="TP2"  Part="1"
-F 0 "TP2" H 4400 3200 50  0000 C CNN
+AR Path="/5E624B3C/5E756356/5E5AE003" Ref="TP2"  Part="1"
+F 0 "TP?" H 4400 3200 50  0000 C CNN
 F 1 "X-" H 4400 3300 50  0000 C CNN
 F 2 "TestPoint:TestPoint_THTPad_D1.5mm_Drill0.7mm" H 4600 2950 50  0001 C CNN

Commit message: Checkpoint of state before I start schematic revisions for the next version of the input board. There are not any substantive modifications to the input board, but some broad changes in component attributes related enabling a fabrication quote.
Parts:
- C31: Manufacturer (none) -> Yageo
- D9: Manufacturer (none) -> Würth Elektronik
- FB5, FB6: Manufacturer TDK Corporation -> Laird-Signal Integrity Products
- J1: Manufacturer (none) -> Amphenol ICC (Commercial Products)
- TP1, TP2: Description (none) -> Do Not Populate; MPN (none) -> DNP
Changed lines of the file:
@@
 $Descr A4 11693 8268
 encoding utf-8
-Sheet 6 33
+Sheet 6 21
 Title ""
 Date ""
@@
 AR Path="/5E756356/5E75AFBD" Ref="J1"  Part="1"
 AR Path="/5E624B3C/5E756356/5E75AFBD" Ref="J1"  Part="1"
-F 0 "J?" H 2450 3300 50  0000 R CNN
+F 0 "J1" H 2450 3300 50  0000 R CNN
 F 1 "Sensor" H 2550 3300 50  0000 L CNN
 F 2 "Connector_RJ:RJ45_Amphenol_RJHSE538X" V 2650 2775 50  0001 C CNN
@@
 F 6 "CONN MOD JACK 8P8C R/A SHIELDED" H 2650 2750 50  0001 C CNN "Description"
 F 7 "18" H 2650 2750 50  0001 C CNN "DK line"
+F 8 "Amphenol ICC (Commercial Products)" H 2650 2750 50  0001 C CNN "Manufacturer"
 	1    2650 2750
 	1    0    0    -1
@@
 AR Path="/5E756356/5E75F20B" Ref="FB5"  Part="1"
 AR Path="/5E624B3C/5E756356/5E75F20B" Ref="FB5"  Part="1"
-F 0 "FB?" H 4000 4337 60  0000 C CNN
+F 0 "FB5" H 4000 4337 60  0000 C CNN
 F 1 "2K Ohm" H 4000 4231 60  0000 C CNN
 F 2 "Inductor_SMD:L_0805_2012Metric" H 4200 4250 60  0001 L CNN
@@
 F 9 "/product-detail/en/tdk-corporation/MPZ2012S601AT000/445-2206-1-ND/765104" H 4200 4950 60  0001 L CNN "DK_Detail_Page"
 F 10 "FERRITE BEAD 2 KOHM 0805 1LN" H 4200 5050 60  0001 L CNN "Description"
-F 11 "TDK Corporation" H 4200 5150 60  0001 L CNN "Manufacturer"
+F 11 "Laird-Signal Integrity Products" H 4200 5150 60  0001 L CNN "Manufacturer"
 F 12 "Active" H 4200 5250 60  0001 L CNN "Status"
 F 13 "5" H 4000 4050 50  0001 C CNN "DK line"
@@
 AR Path="/5E756356/5E7695B8" Ref="D9"  Part="1"
 AR Path="/5E624B3C/5E756356/5E7695B8" Ref="D9"  Part="1"
-F 0 "D?" H 5550 4500 50  0000 C CNN
+F 0 "D9" H 5550 4500 50  0000 C CNN
 F 1 "5V (standoff)" H 5650 4200 50  0000 C CNN
 F 2 "Diode_SMD:D_SMA" H 5550 4400 50  0001 C CNN
@@
 F 6 "732-9974-1-ND" H 5550 4400 50  0001 C CNN "Digikey"
 F 7 "40" H 5550 4400 50  0001 C CNN "DK line"
+F 8 "Würth Elektronik" H 5550 4400 50  0001 C CNN "Manufacturer"
 	1    5550 4400
 	0    1    1    0
@@
 AR Path="/5E756356/5E76B461" Ref="FB6"  Part="1"
 AR Path="/5E624B3C/5E756356/5E76B461" Ref="FB6"  Part="1"
-F 0 "FB?" H 5000 4337 60  0000 C CNN
+F 0 "FB6" H 5000 4337 60  0000 C CNN
 F 1 "2K Ohm" H 5000 4231 60  0000 C CNN
 F 2 "Inductor_SMD:L_0805_2012Metric" H 5200 4250 60  0001 L CNN
@@
 F 9 "/product-detail/en/tdk-corporation/MPZ2012S601AT000/445-2206-1-ND/765104" H 5200 4950 60  0001 L CNN "DK_Detail_Page"
 F 10 "FERRITE BEAD 2 KOHM 0805 1LN" H 5200 5050 60  0001 L CNN "Description"
-F 11 "TDK Corporation" H 5200 5150 60  0001 L CNN "Manufacturer"
+F 11 "Laird-Signal Integrity Products" H 5200 5150 60  0001 L CNN "Manufacturer"
 F 12 "Active" H 5200 5250 60  0001 L CNN "Status"
 F 13 "5" H 5000 4050 50  0001 C CNN "DK line"
@@
 AR Path="/5E756356/5E76E2C4" Ref="C31"  Part="1"
 AR Path="/5E624B3C/5E756356/5E76E2C4" Ref="C31"  Part="1"
-F 0 "C?" H 4542 4396 50  0000 L CNN
+F 0 "C31" H 4542 4396 50  0000 L CNN
 F 1 "1nF" H 4542 4305 50  0000 L CNN
 F 2 "Capacitor_SMD:C_0805_2012Metric" H 4450 4350 50  0001 C CNN
@@
 F 6 "CAP CER 1000PF 100V NPO 0805" H 4450 4350 50  0001 C CNN "Description"
 F 7 "1" H 4450 4350 50  0001 C CNN "DK line"
+F 8 "Yageo" H 4450 4350 50  0001 C CNN "Manufacturer"
 	1    4450 4350
 	1    0    0    -1
@@
 X-
 $Comp
-L power:Earth #PWR?
+L power:Earth #PWR059
 U 1 1 5E36FAA0
 P 2650 3400
-F 0 "#PWR?" H 2650 3150 50  0001 C CNN
+F 0 "#PWR059" H 2650 3150 50  0001 C CNN
 F 1 "Earth" H 2650 3250 50  0001 C CNN
 F 2 "" H 2650 3400 50  0001 C CNN
@@
 $EndComp
 $Comp
-L power:Earth #PWR?
+L power:Earth #PWR060
 U 1 1 5E36FFC7
 P 4450 4650
-F 0 "#PWR?" H 4450 4400 50  0001 C CNN
+F 0 "#PWR060" H 4450 4400 50  0001 C CNN
 F 1 "Earth" H 4450 4500 50  0001 C CNN
 F 2 "" H 4450 4650 50  0001 C CNN
@@
 $EndComp
 $Comp
-L power:Earth #PWR?
+L power:Earth #PWR061
 U 1 1 5E370459
 P 5550 4650
-F 0 "#PWR?" H 5550 4400 50  0001 C CNN
+F 0 "#PWR061" H 5550 4400 50  0001 C CNN
 F 1 "Earth" H 5550 4500 50  0001 C CNN
 F 2 "" H 5550 4650 50  0001 C CNN
@@
 AR Path="/5E756356/5E5ADFFD" Ref="TP1"  Part="1"
 AR Path="/5E624B3C/5E756356/5E5ADFFD" Ref="TP1"  Part="1"
-F 0 "TP?" H 4200 3200 50  0000 C CNN
+F 0 "TP1" H 4200 3200 50  0000 C CNN
 F 1 "X+" H 4200 3300 50  0000 C CNN
 F 2 "TestPoint:TestPoint_THTPad_D1.5mm_Drill0.7mm" H 4400 2950 50  0001 C CNN
 F 3 "~" H 4400 2950 50  0001 C CNN
+F 4 "Do Not Populate" H 4200 2950 50  0001 C CNN "Description"
+F 5 "DNP" H 4200 2950 50  0001 C CNN "MPN"
 	1    4200 2950
 	-1   0    0    1
@@
 AR Path="/5E756356/5E5AE003" Ref="TP2"  Part="1"
 AR Path="/5E624B3C/5E756356/5E5AE003" Ref="TP2"  Part="1"
-F 0 "TP?" H 4400 3200 50  0000 C CNN
+F 0 "TP2" H 4400 3200 50  0000 C CNN
 F 1 "X-" H 4400 3300 50  0000 C CNN
 F 2 "TestPoint:TestPoint_THTPad_D1.5mm_Drill0.7mm" H 4600 2950 50  0001 C CNN
 F 3 "~" H 4600 2950 50  0001 C CNN
+F 4 "Do Not Populate" H 4400 2950 50  0001 C CNN "Description"
+F 5 "DNP" H 4400 2950 50  0001 C CNN "MPN"
 	1    4400 2950
 	-1   0    0    1
