File: input/input_channel.sch (KiCad schematic (older format))
At the start: 4 parts

Commit message: Minor tweaks to schematic, and ongoing progress on PCB layout.
Changed BIST buffer to run off of CHAN1_V+, not the global V+.  This caused the CHAN_V+ net name to change.
On power.sch, added bypass caps for the VREF inputs to the V+/V- regulators.  Also, the BIST input lines now
have an RC filter, not just a resistor.
Connections:
- net antialias_driver/CHAN_V+ renamed CHAN_V+
- net antialias_driver/CHAN_V- renamed CHAN_V-
Changed lines of the file:
@@
 	3250 4100 3800 4100
 Wire Wire Line
-	2400 4100 2800 4100
+	2400 4100 2625 4100
 Wire Wire Line
-	2350 5250 2800 5250
+	2350 5250 2625 5250
 Connection ~ 2800 5250
 Wire Wire Line
@@
 	1    0    0    -1
 $EndComp
+Text HLabel 2700 3800 2    50   Output ~ 0
+CHAN_V+
+Text HLabel 2700 5550 2    50   Output ~ 0
+CHAN_V-
+Wire Wire Line
+	2700 3800 2625 3800
+Wire Wire Line
+	2625 3800 2625 4100
+Connection ~ 2625 4100
+Wire Wire Line
+	2625 4100 2800 4100
+Wire Wire Line
+	2700 5550 2625 5550
+Wire Wire Line
+	2625 5550 2625 5250
+Connection ~ 2625 5250
+Wire Wire Line
+	2625 5250 2800 5250
 $EndSCHEMATC

Commit message: Snapshot before replicating input channels
Changed lines of the file:
@@
 $Descr A4 11693 8268
 encoding utf-8
-Sheet 2 13
+Sheet 13 21
 Title ""
 Date ""
@@
 AR Path="/5DFCF14D/5DE42731/5E23902C" Ref="FB?"  Part="1"
 AR Path="/5DFCF14D/5E23902C" Ref="FB103"  Part="1"
-F 0 "FB103" H 2200 4387 60  0000 C CNN
+AR Path="/5E448095/5E23902C" Ref="FB202"  Part="1"
+AR Path="/5E45936E/5E23902C" Ref="FB302"  Part="1"
+F 0 "FB?" H 2200 4387 60  0000 C CNN
 F 1 "21 Ohm" H 2200 4281 60  0000 C CNN
 F 2 "Inductor_SMD:L_0805_2012Metric" H 2400 4300 60  0001 L CNN
@@
 U 1 1 5E23AF8A
 P 1750 4000
-F 0 "#PWR0119" H 1750 3850 50  0001 C CNN
+AR Path="/5DFCF14D/5E23AF8A" Ref="#PWR0119"  Part="1"
+AR Path="/5E448095/5E23AF8A" Ref="#PWR0201"  Part="1"
+AR Path="/5E45936E/5E23AF8A" Ref="#PWR0301"  Part="1"
+F 0 "#PWR?" H 1750 3850 50  0001 C CNN
 F 1 "V+" H 1750 4140 50  0000 C CNN
 F 2 "" H 1750 4000 50  0001 C CNN
@@
 U 1 1 5E23B186
 P 1750 5400
-F 0 "#PWR0121" H 1750 5250 50  0001 C CNN
+AR Path="/5DFCF14D/5E23B186" Ref="#PWR0121"  Part="1"
+AR Path="/5E448095/5E23B186" Ref="#PWR0202"  Part="1"
+AR Path="/5E45936E/5E23B186" Ref="#PWR0302"  Part="1"
+F 0 "#PWR?" H 1750 5250 50  0001 C CNN
 F 1 "V-" H 1750 5360 50  0000 C CNN
 F 2 "" H 1750 5500 50  0001 C CNN
@@
 AR Path="/5E51E83D/5E23EF6F" Ref="C?"  Part="1"
 AR Path="/5DFCF14D/5E23EF6F" Ref="C119"  Part="1"
-F 0 "C119" V 2950 4350 50  0000 C CNN
+AR Path="/5E448095/5E23EF6F" Ref="C201"  Part="1"
+AR Path="/5E45936E/5E23EF6F" Ref="C301"  Part="1"
+F 0 "C?" V 2950 4350 50  0000 C CNN
 F 1 "330uF" V 2662 4350 50  0000 C CNN
 F 2 "Capacitor_SMD:CP_Elec_8x6.7" H 2800 4350 50  0001 C CNN
@@
 U 1 1 5E23FC8E
 P 2650 4650
-F 0 "#PWR0122" H 2650 4400 50  0001 C CNN
+AR Path="/5DFCF14D/5E23FC8E" Ref="#PWR0122"  Part="1"
+AR Path="/5E448095/5E23FC8E" Ref="#PWR0203"  Part="1"
+AR Path="/5E45936E/5E23FC8E" Ref="#PWR0303"  Part="1"
+F 0 "#PWR?" H 2650 4400 50  0001 C CNN
 F 1 "GNDA" H 2650 4500 50  0000 C CNN
 F 2 "" H 2650 4650 50  0001 C CNN
@@
 AR Path="/5DFCF14D/5DE42731/5E24179B" Ref="FB?"  Part="1"
 AR Path="/5DFCF14D/5E24179B" Ref="FB104"  Part="1"
-F 0 "FB104" H 2150 5537 60  0000 C CNN
+AR Path="/5E448095/5E24179B" Ref="FB201"  Part="1"
+AR Path="/5E45936E/5E24179B" Ref="FB301"  Part="1"
+F 0 "FB?" H 2150 5537 60  0000 C CNN
 F 1 "21 Ohm" H 2150 5431 60  0000 C CNN
 F 2 "Inductor_SMD:L_0805_2012Metric" H 2350 5450 60  0001 L CNN
@@
 AR Path="/5E51E83D/5E2417A1" Ref="C?"  Part="1"
 AR Path="/5DFCF14D/5E2417A1" Ref="C133"  Part="1"
-F 0 "C133" V 2950 4950 50  0000 C CNN
+AR Path="/5E448095/5E2417A1" Ref="C202"  Part="1"
+AR Path="/5E45936E/5E2417A1" Ref="C302"  Part="1"
+F 0 "C?" V 2950 4950 50  0000 C CNN
 F 1 "330uF" V 2662 4950 50  0000 C CNN
 F 2 "Capacitor_SMD:CP_Elec_8x6.7" H 2800 4950 50  0001 C CNN
@@
 U 1 1 5E8B0766
 P 3250 4100
-F 0 "#FLG0103" H 3250 4175 50  0001 C CNN
+AR Path="/5DFCF14D/5E8B0766" Ref="#FLG0103"  Part="1"
+AR Path="/5E448095/5E8B0766" Ref="#FLG0201"  Part="1"
+AR Path="/5E45936E/5E8B0766" Ref="#FLG0301"  Part="1"
+F 0 "#FLG?" H 3250 4175 50  0001 C CNN
 F 1 "PWR_FLAG" H 3250 4250 50  0000 C CNN
 F 2 "" H 3250 4100 50  0001 C CNN
@@
 U 1 1 5E8B104C
 P 3250 5250
-F 0 "#FLG0104" H 3250 5325 50  0001 C CNN
+AR Path="/5DFCF14D/5E8B104C" Ref="#FLG0104"  Part="1"
+AR Path="/5E448095/5E8B104C" Ref="#FLG0202"  Part="1"
+AR Path="/5E45936E/5E8B104C" Ref="#FLG0302"  Part="1"
+F 0 "#FLG?" H 3250 5325 50  0001 C CNN
 F 1 "PWR_FLAG" H 3250 5400 50  0000 C CNN
 F 2 "" H 3250 5250 50  0001 C CNN

Commit message: Input board is nearly ready to send off for the first spin.
Changed lines of the file:
@@
 $Descr A4 11693 8268
 encoding utf-8
-Sheet 13 21
+Sheet 7 21
 Title ""
 Date ""
@@
 One input channel, from filter and protection, all the way through to the ADC.
 $Sheet
-S 4150 2950 1200 750
+S 4150 2350 1200 1100
 U 5DE42731
 F0 "in_filter" 50
@@
 F2 "+out" O R 5350 3050 50
 F3 "-out" O R 5350 3200 50
-F4 "-in" I L 4150 3200 50
-F5 "+in" I L 4150 3050 50
-F6 "CHAN_V+" I L 4150 3350 50
-F7 "CHAN_V-" I L 4150 3450 50
-F8 "CHAN_VREF" I L 4150 3600 50
+F4 "-in" I L 4150 2600 50
+F5 "+in" I L 4150 2450 50
+F6 "CHAN_V+" I L 4150 2750 50
+F7 "CHAN_V-" I L 4150 2850 50
+F8 "CHAN_VREF" I L 4150 3000 50
+F9 "BIST-+_FB" O R 5350 2650 50
+F10 "BIST--_FB" O R 5350 2750 50
+F11 "BIST++_FB" O R 5350 2450 50
+F12 "BIST+-_FB" O R 5350 2550 50
 $EndSheet
 $Sheet
@@
 F7 "CHAN_V-" I L 6000 3450 50
 $EndSheet
-Text HLabel 3800 3050 0    50   Input ~ 0
+Text HLabel 3800 2450 0    50   Input ~ 0
 +in
-Text HLabel 3800 3200 0    50   Input ~ 0
+Text HLabel 3800 2600 0    50   Input ~ 0
 -in
 Wire Wire Line
-	3800 3050 4150 3050
-Wire Wire Line
-	3800 3200 4150 3200
+	3800 2450 4150 2450
+Wire Wire Line
+	3800 2600 4150 2600
 Wire Wire Line
 	7100 3050 7700 3050
@@
 AR Path="/5E448095/5E23902C" Ref="FB202"  Part="1"
 AR Path="/5E45936E/5E23902C" Ref="FB302"  Part="1"
-F 0 "FB?" H 2200 4387 60  0000 C CNN
+F 0 "FB103" H 2200 4387 60  0000 C CNN
 F 1 "21 Ohm" H 2200 4281 60  0000 C CNN
 F 2 "Inductor_SMD:L_0805_2012Metric" H 2400 4300 60  0001 L CNN
@@
 AR Path="/5E448095/5E23AF8A" Ref="#PWR0201"  Part="1"
 AR Path="/5E45936E/5E23AF8A" Ref="#PWR0301"  Part="1"
-F 0 "#PWR?" H 1750 3850 50  0001 C CNN
+F 0 "#PWR0119" H 1750 3850 50  0001 C CNN
 F 1 "V+" H 1750 4140 50  0000 C CNN
 F 2 "" H 1750 4000 50  0001 C CNN
@@
 AR Path="/5E448095/5E23B186" Ref="#PWR0202"  Part="1"
 AR Path="/5E45936E/5E23B186" Ref="#PWR0302"  Part="1"
-F 0 "#PWR?" H 1750 5250 50  0001 C CNN
+F 0 "#PWR0121" H 1750 5250 50  0001 C CNN
 F 1 "V-" H 1750 5360 50  0000 C CNN
 F 2 "" H 1750 5500 50  0001 C CNN
@@
 AR Path="/5E448095/5E23EF6F" Ref="C201"  Part="1"
 AR Path="/5E45936E/5E23EF6F" Ref="C301"  Part="1"
-F 0 "C?" V 2950 4350 50  0000 C CNN
+F 0 "C119" V 2950 4350 50  0000 C CNN
 F 1 "330uF" V 2662 4350 50  0000 C CNN
 F 2 "Capacitor_SMD:CP_Elec_8x6.7" H 2800 4350 50  0001 C CNN
@@
 AR Path="/5E448095/5E23FC8E" Ref="#PWR0203"  Part="1"
 AR Path="/5E45936E/5E23FC8E" Ref="#PWR0303"  Part="1"
-F 0 "#PWR?" H 2650 4400 50  0001 C CNN
+F 0 "#PWR0122" H 2650 4400 50  0001 C CNN
 F 1 "GNDA" H 2650 4500 50  0000 C CNN
 F 2 "" H 2650 4650 50  0001 C CNN
@@
 AR Path="/5E448095/5E24179B" Ref="FB201"  Part="1"
 AR Path="/5E45936E/5E24179B" Ref="FB301"  Part="1"
-F 0 "FB?" H 2150 5537 60  0000 C CNN
+F 0 "FB104" H 2150 5537 60  0000 C CNN
 F 1 "21 Ohm" H 2150 5431 60  0000 C CNN
 F 2 "Inductor_SMD:L_0805_2012Metric" H 2350 5450 60  0001 L CNN
@@
 AR Path="/5E448095/5E2417A1" Ref="C202"  Part="1"
 AR Path="/5E45936E/5E2417A1" Ref="C302"  Part="1"
-F 0 "C?" V 2950 4950 50  0000 C CNN
+F 0 "C133" V 2950 4950 50  0000 C CNN
 F 1 "330uF" V 2662 4950 50  0000 C CNN
 F 2 "Capacitor_SMD:CP_Elec_8x6.7" H 2800 4950 50  0001 C CNN
@@
 Wire Wire Line
 	5850 3450 5850 4200
-Wire Wire Line
-	4150 3350 3800 3350
-Wire Wire Line
-	3800 3350 3800 4100
-Wire Wire Line
-	4150 3450 3900 3450
-Wire Wire Line
-	3900 3450 3900 4200
 Connection ~ 3800 4100
 Connection ~ 3900 4200
@@
 $EndSheet
 Wire Wire Line
-	5350 3050 6000 3050
-Wire Wire Line
-	5350 3200 6000 3200
-Wire Wire Line
 	5750 3350 6000 3350
 Wire Wire Line
@@
 	4050 4500 7600 4500
 Connection ~ 7600 4500
-Wire Wire Line
-	4150 3600 4050 3600
-Wire Wire Line
-	4050 3600 4050 4500
 $Comp
 L power:PWR_FLAG #FLG0103
@@
 AR Path="/5E448095/5E8B0766" Ref="#FLG0201"  Part="1"
 AR Path="/5E45936E/5E8B0766" Ref="#FLG0301"  Part="1"
-F 0 "#FLG?" H 3250 4175 50  0001 C CNN
+F 0 "#FLG0103" H 3250 4175 50  0001 C CNN
 F 1 "PWR_FLAG" H 3250 4250 50  0000 C CNN
 F 2 "" H 3250 4100 50  0001 C CNN
@@
 AR Path="/5E448095/5E8B104C" Ref="#FLG0202"  Part="1"
 AR Path="/5E45936E/5E8B104C" Ref="#FLG0302"  Part="1"
-F 0 "#FLG?" H 3250 5325 50  0001 C CNN
+F 0 "#FLG0104" H 3250 5325 50  0001 C CNN
 F 1 "PWR_FLAG" H 3250 5400 50  0000 C CNN
 F 2 "" H 3250 5250 50  0001 C CNN
@@
 Wire Wire Line
 	2625 5250 2800 5250
+Wire Wire Line
+	5350 3050 6000 3050
+Wire Wire Line
+	5350 3200 6000 3200
+Wire Wire Line
+	4150 3000 4050 3000
+Wire Wire Line
+	4050 3000 4050 4500
+Wire Wire Line
+	4150 2850 3900 2850
+Wire Wire Line
+	3900 2850 3900 4200
+Wire Wire Line
+	4150 2750 3800 2750
+Wire Wire Line
+	3800 2750 3800 4100
+Text HLabel 5500 2650 2    50   Output ~ 0
+BIST-+_FB
+Text HLabel 5500 2750 2    50   Output ~ 0
+BIST--_FB
+Text HLabel 5500 2450 2    50   Output ~ 0
+BIST++_FB
+Text HLabel 5500 2550 2    50   Output ~ 0
+BIST+-_FB
+Wire Wire Line
+	5350 2450 5500 2450
+Wire Wire Line
+	5350 2550 5500 2550
+Wire Wire Line
+	5350 2650 5500 2650
+Wire Wire Line
+	5350 2750 5500 2750
 $EndSCHEMATC

Commit message: Various tweaks to schematic which help in the PCB view, mainly getting informative net names. Also unscrambled the + and - paths in the input channel.  This avoided a cross-over before the first stage, and an unintended inversion, but mostly just made net naming less confusing.
Getting better net names made it easier to review the PCB to see if it made sense.  I checked
the ICs on the PCB against the datasheet pinout, and while doing this fixed an actual bug where
I had BIST-+ and BIST+-swapped.

I made some tweaks on the PCB to try to equalize the copper area on the input nets so as to
match the capacitance.  I tweaked the top-side ground pours somewhat, adding in the regulator
area, removing around the high speed traces.

Some changes from gerber viewing.  I reduced the solder mask clearances so that we get mask
web between the SOIC and DFN pads.  I reduced the pad size of the big via from 1.2 to 1.0 mm.
Changed lines of the file:
@@
 F2 "-out" I R 8750 3200 50
 F3 "+out" I R 8750 3050 50
-F4 "-in" I L 7700 3200 50
-F5 "+in" I L 7700 3050 50
+F4 "-IN2" I L 7700 3200 50
+F5 "+IN2" I L 7700 3050 50
 F6 "CHAN_V+" I L 7700 3350 50
 F7 "CHAN_V-" I L 7700 3450 50
@@
 F0 "in_amp" 50
 F1 "in_amp.sch" 50
-F2 "-in" I L 6000 3200 50
-F3 "+in" I L 6000 3050 50
+F2 "-IN1" I L 6000 3200 50
+F3 "+IN1" I L 6000 3050 50
 F4 "+out" I R 7100 3050 50
 F5 "-out" I R 7100 3200 50
@@
 F0 "ADC" 50
 F1 "adc.sch" 50
-F2 "+in" I L 9350 3050 50
-F3 "-in" I L 9350 3200 50
+F2 "+IN_ADC" I L 9350 3050 50
+F3 "-IN_ADC" I L 9350 3200 50
 F4 "CHAN_VREF" O R 10450 3350 50
 F5 "SDOA" O R 10450 3050 50

Commit message: Work on main board.
Changed lines of the file:
@@
 $Descr A4 11693 8268
 encoding utf-8
-Sheet 7 21
+Sheet 17 33
 Title ""
 Date ""
@@
 AR Path="/5E448095/5E23902C" Ref="FB202"  Part="1"
 AR Path="/5E45936E/5E23902C" Ref="FB302"  Part="1"
-F 0 "FB103" H 2200 4387 60  0000 C CNN
+AR Path="/5E525F2C/5E6427A0/5E23902C" Ref="FB?"  Part="1"
+AR Path="/5E624B3C/5DFCF14D/5E23902C" Ref="FB103"  Part="1"
+AR Path="/5E624B3C/5E448095/5E23902C" Ref="FB103"  Part="1"
+AR Path="/5E624B3C/5E45936E/5E23902C" Ref="FB103"  Part="1"
+AR Path="/5E62FD57/5DFCF14D/5E23902C" Ref="FB?"  Part="1"
+AR Path="/5E62FD57/5E448095/5E23902C" Ref="FB?"  Part="1"
+AR Path="/5E62FD57/5E45936E/5E23902C" Ref="FB?"  Part="1"
+F 0 "FB?" H 2200 4387 60  0000 C CNN
 F 1 "21 Ohm" H 2200 4281 60  0000 C CNN
 F 2 "Inductor_SMD:L_0805_2012Metric" H 2400 4300 60  0001 L CNN
@@
 AR Path="/5E448095/5E23AF8A" Ref="#PWR0201"  Part="1"
 AR Path="/5E45936E/5E23AF8A" Ref="#PWR0301"  Part="1"
-F 0 "#PWR0119" H 1750 3850 50  0001 C CNN
+AR Path="/5E525F2C/5E6427A0/5E23AF8A" Ref="#PWR?"  Part="1"
+AR Path="/5E624B3C/5DFCF14D/5E23AF8A" Ref="#PWR0119"  Part="1"
+AR Path="/5E624B3C/5E448095/5E23AF8A" Ref="#PWR0119"  Part="1"
+AR Path="/5E624B3C/5E45936E/5E23AF8A" Ref="#PWR0119"  Part="1"
+AR Path="/5E62FD57/5DFCF14D/5E23AF8A" Ref="#PWR?"  Part="1"
+AR Path="/5E62FD57/5E448095/5E23AF8A" Ref="#PWR?"  Part="1"
+AR Path="/5E62FD57/5E45936E/5E23AF8A" Ref="#PWR?"  Part="1"
+F 0 "#PWR?" H 1750 3850 50  0001 C CNN
 F 1 "V+" H 1750 4140 50  0000 C CNN
 F 2 "" H 1750 4000 50  0001 C CNN
@@
 AR Path="/5E448095/5E23B186" Ref="#PWR0202"  Part="1"
 AR Path="/5E45936E/5E23B186" Ref="#PWR0302"  Part="1"
-F 0 "#PWR0121" H 1750 5250 50  0001 C CNN
+AR Path="/5E525F2C/5E6427A0/5E23B186" Ref="#PWR?"  Part="1"
+AR Path="/5E624B3C/5DFCF14D/5E23B186" Ref="#PWR0121"  Part="1"
+AR Path="/5E624B3C/5E448095/5E23B186" Ref="#PWR0121"  Part="1"
+AR Path="/5E624B3C/5E45936E/5E23B186" Ref="#PWR0121"  Part="1"
+AR Path="/5E62FD57/5DFCF14D/5E23B186" Ref="#PWR?"  Part="1"
+AR Path="/5E62FD57/5E448095/5E23B186" Ref="#PWR?"  Part="1"
+AR Path="/5E62FD57/5E45936E/5E23B186" Ref="#PWR?"  Part="1"
+F 0 "#PWR?" H 1750 5250 50  0001 C CNN
 F 1 "V-" H 1750 5360 50  0000 C CNN
 F 2 "" H 1750 5500 50  0001 C CNN
@@
 AR Path="/5E448095/5E23EF6F" Ref="C201"  Part="1"
 AR Path="/5E45936E/5E23EF6F" Ref="C301"  Part="1"
-F 0 "C119" V 2950 4350 50  0000 C CNN
+AR Path="/5E525F2C/5E6427A0/5E23EF6F" Ref="C?"  Part="1"
+AR Path="/5E624B3C/5DFCF14D/5E23EF6F" Ref="C119"  Part="1"
+AR Path="/5E624B3C/5E448095/5E23EF6F" Ref="C119"  Part="1"
+AR Path="/5E624B3C/5E45936E/5E23EF6F" Ref="C119"  Part="1"
+AR Path="/5E62FD57/5DFCF14D/5E23EF6F" Ref="C?"  Part="1"
+AR Path="/5E62FD57/5E448095/5E23EF6F" Ref="C?"  Part="1"
+AR Path="/5E62FD57/5E45936E/5E23EF6F" Ref="C?"  Part="1"
+F 0 "C?" V 2950 4350 50  0000 C CNN
 F 1 "330uF" V 2662 4350 50  0000 C CNN
 F 2 "Capacitor_SMD:CP_Elec_8x6.7" H 2800 4350 50  0001 C CNN
@@
 AR Path="/5E448095/5E23FC8E" Ref="#PWR0203"  Part="1"
 AR Path="/5E45936E/5E23FC8E" Ref="#PWR0303"  Part="1"
-F 0 "#PWR0122" H 2650 4400 50  0001 C CNN
+AR Path="/5E525F2C/5E6427A0/5E23FC8E" Ref="#PWR?"  Part="1"
+AR Path="/5E624B3C/5DFCF14D/5E23FC8E" Ref="#PWR0122"  Part="1"
+AR Path="/5E624B3C/5E448095/5E23FC8E" Ref="#PWR0122"  Part="1"
+AR Path="/5E624B3C/5E45936E/5E23FC8E" Ref="#PWR0122"  Part="1"
+AR Path="/5E62FD57/5DFCF14D/5E23FC8E" Ref="#PWR?"  Part="1"
+AR Path="/5E62FD57/5E448095/5E23FC8E" Ref="#PWR?"  Part="1"
+AR Path="/5E62FD57/5E45936E/5E23FC8E" Ref="#PWR?"  Part="1"
+F 0 "#PWR?" H 2650 4400 50  0001 C CNN
 F 1 "GNDA" H 2650 4500 50  0000 C CNN
 F 2 "" H 2650 4650 50  0001 C CNN
@@
 AR Path="/5E448095/5E24179B" Ref="FB201"  Part="1"
 AR Path="/5E45936E/5E24179B" Ref="FB301"  Part="1"
-F 0 "FB104" H 2150 5537 60  0000 C CNN
+AR Path="/5E525F2C/5E6427A0/5E24179B" Ref="FB?"  Part="1"
+AR Path="/5E624B3C/5DFCF14D/5E24179B" Ref="FB104"  Part="1"
+AR Path="/5E624B3C/5E448095/5E24179B" Ref="FB104"  Part="1"
+AR Path="/5E624B3C/5E45936E/5E24179B" Ref="FB104"  Part="1"
+AR Path="/5E62FD57/5DFCF14D/5E24179B" Ref="FB?"  Part="1"
+AR Path="/5E62FD57/5E448095/5E24179B" Ref="FB?"  Part="1"
+AR Path="/5E62FD57/5E45936E/5E24179B" Ref="FB?"  Part="1"
+F 0 "FB?" H 2150 5537 60  0000 C CNN
 F 1 "21 Ohm" H 2150 5431 60  0000 C CNN
 F 2 "Inductor_SMD:L_0805_2012Metric" H 2350 5450 60  0001 L CNN
@@
 AR Path="/5E448095/5E2417A1" Ref="C202"  Part="1"
 AR Path="/5E45936E/5E2417A1" Ref="C302"  Part="1"
-F 0 "C133" V 2950 4950 50  0000 C CNN
+AR Path="/5E525F2C/5E6427A0/5E2417A1" Ref="C?"  Part="1"
+AR Path="/5E624B3C/5DFCF14D/5E2417A1" Ref="C133"  Part="1"
+AR Path="/5E624B3C/5E448095/5E2417A1" Ref="C133"  Part="1"
+AR Path="/5E624B3C/5E45936E/5E2417A1" Ref="C133"  Part="1"
+AR Path="/5E62FD57/5DFCF14D/5E2417A1" Ref="C?"  Part="1"
+AR Path="/5E62FD57/5E448095/5E2417A1" Ref="C?"  Part="1"
+AR Path="/5E62FD57/5E45936E/5E2417A1" Ref="C?"  Part="1"
+F 0 "C?" V 2950 4950 50  0000 C CNN
 F 1 "330uF" V 2662 4950 50  0000 C CNN
 F 2 "Capacitor_SMD:CP_Elec_8x6.7" H 2800 4950 50  0001 C CNN
@@
 AR Path="/5E448095/5E8B0766" Ref="#FLG0201"  Part="1"
 AR Path="/5E45936E/5E8B0766" Ref="#FLG0301"  Part="1"
-F 0 "#FLG0103" H 3250 4175 50  0001 C CNN
+AR Path="/5E525F2C/5E6427A0/5E8B0766" Ref="#FLG?"  Part="1"
+AR Path="/5E624B3C/5DFCF14D/5E8B0766" Ref="#FLG0103"  Part="1"
+AR Path="/5E624B3C/5E448095/5E8B0766" Ref="#FLG0103"  Part="1"
+AR Path="/5E624B3C/5E45936E/5E8B0766" Ref="#FLG0103"  Part="1"
+AR Path="/5E62FD57/5DFCF14D/5E8B0766" Ref="#FLG?"  Part="1"
+AR Path="/5E62FD57/5E448095/5E8B0766" Ref="#FLG?"  Part="1"
+AR Path="/5E62FD57/5E45936E/5E8B0766" Ref="#FLG?"  Part="1"
+F 0 "#FLG?" H 3250 4175 50  0001 C CNN
 F 1 "PWR_FLAG" H 3250 4250 50  0000 C CNN
 F 2 "" H 3250 4100 50  0001 C CNN
@@
 AR Path="/5E448095/5E8B104C" Ref="#FLG0202"  Part="1"
 AR Path="/5E45936E/5E8B104C" Ref="#FLG0302"  Part="1"
-F 0 "#FLG0104" H 3250 5325 50  0001 C CNN
+AR Path="/5E525F2C/5E6427A0/5E8B104C" Ref="#FLG?"  Part="1"
+AR Path="/5E624B3C/5DFCF14D/5E8B104C" Ref="#FLG0104"  Part="1"
+AR Path="/5E624B3C/5E448095/5E8B104C" Ref="#FLG0104"  Part="1"
+AR Path="/5E624B3C/5E45936E/5E8B104C" Ref="#FLG0104"  Part="1"
+AR Path="/5E62FD57/5DFCF14D/5E8B104C" Ref="#FLG?"  Part="1"
+AR Path="/5E62FD57/5E448095/5E8B104C" Ref="#FLG?"  Part="1"
+AR Path="/5E62FD57/5E45936E/5E8B104C" Ref="#FLG?"  Part="1"
+F 0 "#FLG?" H 3250 5325 50  0001 C CNN
 F 1 "PWR_FLAG" H 3250 5400 50  0000 C CNN
 F 2 "" H 3250 5250 50  0001 C CNN

Commit message: Checkpoint of state before I start schematic revisions for the next version of the input board. There are not any substantive modifications to the input board, but some broad changes in component attributes related enabling a fabrication quote.
Parts:
- C119, C133: Manufacturer (none) -> United Chemi-Con
- FB103, FB104: MPN HZ0805C202R-10 -> FBMJ2125HM210NT; Manufacturer (none) -> Taiyo Yuden
Changed lines of the file:
@@
 $Descr A4 11693 8268
 encoding utf-8
-Sheet 17 33
+Sheet 7 21
 Title ""
 Date ""
@@
 AR Path="/5E62FD57/5E448095/5E23902C" Ref="FB?"  Part="1"
 AR Path="/5E62FD57/5E45936E/5E23902C" Ref="FB?"  Part="1"
-F 0 "FB?" H 2200 4387 60  0000 C CNN
+F 0 "FB103" H 2200 4387 60  0000 C CNN
 F 1 "21 Ohm" H 2200 4281 60  0000 C CNN
 F 2 "Inductor_SMD:L_0805_2012Metric" H 2400 4300 60  0001 L CNN
 F 3 "https://www.yuden.co.jp/productdata/catalog/chipbeads01_e.pdf" H 2400 4400 60  0001 L CNN
-F 4 "HZ0805C202R-10" H 2400 4600 60  0001 L CNN "MPN"
+F 4 "FBMJ2125HM210NT" H 2400 4600 60  0001 L CNN "MPN"
 F 5 "Ferrite Beads and Chips" H 2400 4800 60  0001 L CNN "Family"
 F 6 "FERRITE BEAD 21 OHM 0805, 100 nH, 5 mOhm" H 2400 5100 60  0001 L CNN "Description"
 F 7 "587-1765-1-ND" H 2200 4100 50  0001 C CNN "Digikey"
 F 8 "24" H 2200 4100 50  0001 C CNN "DK line"
+F 9 "Taiyo Yuden" H 2200 4100 50  0001 C CNN "Manufacturer"
 	1    2200 4100
 	1    0    0    -1
@@
 AR Path="/5E62FD57/5E448095/5E23AF8A" Ref="#PWR?"  Part="1"
 AR Path="/5E62FD57/5E45936E/5E23AF8A" Ref="#PWR?"  Part="1"
-F 0 "#PWR?" H 1750 3850 50  0001 C CNN
+F 0 "#PWR0301" H 1750 3850 50  0001 C CNN
 F 1 "V+" H 1750 4140 50  0000 C CNN
 F 2 "" H 1750 4000 50  0001 C CNN
@@
 AR Path="/5E62FD57/5E448095/5E23B186" Ref="#PWR?"  Part="1"
 AR Path="/5E62FD57/5E45936E/5E23B186" Ref="#PWR?"  Part="1"
-F 0 "#PWR?" H 1750 5250 50  0001 C CNN
+F 0 "#PWR0302" H 1750 5250 50  0001 C CNN
 F 1 "V-" H 1750 5360 50  0000 C CNN
 F 2 "" H 1750 5500 50  0001 C CNN
@@
 AR Path="/5E62FD57/5E448095/5E23EF6F" Ref="C?"  Part="1"
 AR Path="/5E62FD57/5E45936E/5E23EF6F" Ref="C?"  Part="1"
-F 0 "C?" V 2950 4350 50  0000 C CNN
+F 0 "C119" V 2950 4350 50  0000 C CNN
 F 1 "330uF" V 2662 4350 50  0000 C CNN
 F 2 "Capacitor_SMD:CP_Elec_8x6.7" H 2800 4350 50  0001 C CNN
@@
 F 6 "APXG160ARA331MH70G" H 2800 4350 50  0001 C CNN "MPN"
 F 7 "19" H 2800 4350 50  0001 C CNN "DK line"
+F 8 "United Chemi-Con" H 2800 4350 50  0001 C CNN "Manufacturer"
 	1    2800 4350
 	1    0    0    -1
@@
 AR Path="/5E62FD57/5E448095/5E23FC8E" Ref="#PWR?"  Part="1"
 AR Path="/5E62FD57/5E45936E/5E23FC8E" Ref="#PWR?"  Part="1"
-F 0 "#PWR?" H 2650 4400 50  0001 C CNN
+F 0 "#PWR0303" H 2650 4400 50  0001 C CNN
 F 1 "GNDA" H 2650 4500 50  0000 C CNN
 F 2 "" H 2650 4650 50  0001 C CNN
@@
 AR Path="/5E62FD57/5E448095/5E24179B" Ref="FB?"  Part="1"
 AR Path="/5E62FD57/5E45936E/5E24179B" Ref="FB?"  Part="1"
-F 0 "FB?" H 2150 5537 60  0000 C CNN
+F 0 "FB104" H 2150 5537 60  0000 C CNN
 F 1 "21 Ohm" H 2150 5431 60  0000 C CNN
 F 2 "Inductor_SMD:L_0805_2012Metric" H 2350 5450 60  0001 L CNN
 F 3 "https://www.yuden.co.jp/productdata/catalog/chipbeads01_e.pdf" H 2350 5550 60  0001 L CNN
-F 4 "HZ0805C202R-10" H 2350 5750 60  0001 L CNN "MPN"
+F 4 "FBMJ2125HM210NT" H 2350 5750 60  0001 L CNN "MPN"
 F 5 "Ferrite Beads and Chips" H 2350 5950 60  0001 L CNN "Family"
 F 6 "FERRITE BEAD 21 OHM 0805, 100 nH, 5 mOhm" H 2350 6250 60  0001 L CNN "Description"
 F 7 "587-1765-1-ND" H 2150 5250 50  0001 C CNN "Digikey"
 F 8 "24" H 2150 5250 50  0001 C CNN "DK line"
+F 9 "Taiyo Yuden" H 2150 5250 50  0001 C CNN "Manufacturer"
 	1    2150 5250
 	1    0    0    -1
@@
 AR Path="/5E62FD57/5E448095/5E2417A1" Ref="C?"  Part="1"
 AR Path="/5E62FD57/5E45936E/5E2417A1" Ref="C?"  Part="1"
-F 0 "C?" V 2950 4950 50  0000 C CNN
+F 0 "C133" V 2950 4950 50  0000 C CNN
 F 1 "330uF" V 2662 4950 50  0000 C CNN
 F 2 "Capacitor_SMD:CP_Elec_8x6.7" H 2800 4950 50  0001 C CNN
@@
 F 6 "APXG160ARA331MH70G" H 2800 4950 50  0001 C CNN "MPN"
 F 7 "19" H 2800 4950 50  0001 C CNN "DK line"
+F 8 "United Chemi-Con" H 2800 4950 50  0001 C CNN "Manufacturer"
 	1    2800 4950
 	1    0    0    -1
@@
 AR Path="/5E62FD57/5E448095/5E8B0766" Ref="#FLG?"  Part="1"
 AR Path="/5E62FD57/5E45936E/5E8B0766" Ref="#FLG?"  Part="1"
-F 0 "#FLG?" H 3250 4175 50  0001 C CNN
+F 0 "#FLG0301" H 3250 4175 50  0001 C CNN
 F 1 "PWR_FLAG" H 3250 4250 50  0000 C CNN
 F 2 "" H 3250 4100 50  0001 C CNN
@@
 AR Path="/5E62FD57/5E448095/5E8B104C" Ref="#FLG?"  Part="1"
 AR Path="/5E62FD57/5E45936E/5E8B104C" Ref="#FLG?"  Part="1"
-F 0 "#FLG?" H 3250 5325 50  0001 C CNN
+F 0 "#FLG0302" H 3250 5325 50  0001 C CNN
 F 1 "PWR_FLAG" H 3250 5400 50  0000 C CNN
 F 2 "" H 3250 5250 50  0001 C CNN
