File: input/input_channel.sch (KiCad schematic (older format))
At the start: 4 parts

Commit message: Input board revisions, mostly related to reference buffer.
power.sch: changed +3.3V to use the NCP1117 adjustable regulator, the MCP1577 was so noisy it was injecting noise into the ground plane, disturbing the VREF distribution.  Fixed fuse footprint, was too small.

reference_buffer.sch: added series resistor R40 on VREF buffer feedback cap C2, this adds damping to the response, avoiding noise peaking and overshoot.  Changed VREF bias R5/R14 to be taken from V+, rather than FILT_+10V.  V+ is a much lower noise regulated output, but this does reintroduce a bootstrapping issue between VREF and V+.  We don't get any startup problems here, though, because U3B can source current into VREF (from LPF_+10V) until the V+ supply comes up.  Because of 8V rather than 10V, the bias resistors are changed to 301 Ohm to maintain 20 mA bias. Change the VREF bus capacitor from  2x 47 uF ceramic to 330 uF aluminum poly.  This improves damping and disturbance rejection between 10 kHz and 100 kHz.

input_board.kicad_pcb: update for these schematic changes.

reference_buffer_lpf.wxsch: update to match current design.
Changed lines of the file:
@@
 AR Path="/5E62FD57/5E448095/5E23902C" Ref="FB?"  Part="1"
 AR Path="/5E62FD57/5E45936E/5E23902C" Ref="FB?"  Part="1"
-F 0 "FB103" H 2200 4387 60  0000 C CNN
+F 0 "FB302" H 2200 4387 60  0000 C CNN
 F 1 "21 Ohm" H 2200 4281 60  0000 C CNN
 F 2 "Inductor_SMD:L_0805_2012Metric" H 2400 4300 60  0001 L CNN
@@
 AR Path="/5E62FD57/5E448095/5E23AF8A" Ref="#PWR?"  Part="1"
 AR Path="/5E62FD57/5E45936E/5E23AF8A" Ref="#PWR?"  Part="1"
-F 0 "#PWR0119" H 1750 3850 50  0001 C CNN
+F 0 "#PWR0301" H 1750 3850 50  0001 C CNN
 F 1 "V+" H 1750 4140 50  0000 C CNN
 F 2 "" H 1750 4000 50  0001 C CNN
@@
 AR Path="/5E62FD57/5E448095/5E23B186" Ref="#PWR?"  Part="1"
 AR Path="/5E62FD57/5E45936E/5E23B186" Ref="#PWR?"  Part="1"
-F 0 "#PWR0121" H 1750 5250 50  0001 C CNN
+F 0 "#PWR0302" H 1750 5250 50  0001 C CNN
 F 1 "V-" H 1750 5360 50  0000 C CNN
 F 2 "" H 1750 5500 50  0001 C CNN
@@
 AR Path="/5E62FD57/5E448095/5E23EF6F" Ref="C?"  Part="1"
 AR Path="/5E62FD57/5E45936E/5E23EF6F" Ref="C?"  Part="1"
-F 0 "C119" V 2950 4350 50  0000 C CNN
+F 0 "C301" V 2950 4350 50  0000 C CNN
 F 1 "330uF" V 2662 4350 50  0000 C CNN
 F 2 "Capacitor_SMD:CP_Elec_8x6.7" H 2800 4350 50  0001 C CNN
@@
 AR Path="/5E62FD57/5E448095/5E23FC8E" Ref="#PWR?"  Part="1"
 AR Path="/5E62FD57/5E45936E/5E23FC8E" Ref="#PWR?"  Part="1"
-F 0 "#PWR0122" H 2650 4400 50  0001 C CNN
+F 0 "#PWR0303" H 2650 4400 50  0001 C CNN
 F 1 "GNDA" H 2650 4500 50  0000 C CNN
 F 2 "" H 2650 4650 50  0001 C CNN
@@
 AR Path="/5E62FD57/5E448095/5E24179B" Ref="FB?"  Part="1"
 AR Path="/5E62FD57/5E45936E/5E24179B" Ref="FB?"  Part="1"
-F 0 "FB104" H 2150 5537 60  0000 C CNN
+F 0 "FB301" H 2150 5537 60  0000 C CNN
 F 1 "21 Ohm" H 2150 5431 60  0000 C CNN
 F 2 "Inductor_SMD:L_0805_2012Metric" H 2350 5450 60  0001 L CNN
@@
 AR Path="/5E62FD57/5E448095/5E2417A1" Ref="C?"  Part="1"
 AR Path="/5E62FD57/5E45936E/5E2417A1" Ref="C?"  Part="1"
-F 0 "C133" V 2950 4950 50  0000 C CNN
+F 0 "C302" V 2950 4950 50  0000 C CNN
 F 1 "330uF" V 2662 4950 50  0000 C CNN
 F 2 "Capacitor_SMD:CP_Elec_8x6.7" H 2800 4950 50  0001 C CNN
@@
 AR Path="/5E62FD57/5E448095/5E8B0766" Ref="#FLG?"  Part="1"
 AR Path="/5E62FD57/5E45936E/5E8B0766" Ref="#FLG?"  Part="1"
-F 0 "#FLG0103" H 3250 4175 50  0001 C CNN
+F 0 "#FLG0301" H 3250 4175 50  0001 C CNN
 F 1 "PWR_FLAG" H 3250 4250 50  0000 C CNN
 F 2 "" H 3250 4100 50  0001 C CNN
@@
 AR Path="/5E62FD57/5E448095/5E8B104C" Ref="#FLG?"  Part="1"
 AR Path="/5E62FD57/5E45936E/5E8B104C" Ref="#FLG?"  Part="1"
-F 0 "#FLG0104" H 3250 5325 50  0001 C CNN
+F 0 "#FLG0302" H 3250 5325 50  0001 C CNN
 F 1 "PWR_FLAG" H 3250 5400 50  0000 C CNN
 F 2 "" H 3250 5250 50  0001 C CNN
