File: main/main_board/clock.sch (KiCad schematic (older format))
At the start: 0 parts

Commit message: Work on main board.
Parts:
- added C41, C42, C44, C46: 100nF, Capacitor_SMD:C_0603_1608Metric, symbol Device:C_Small
- added C43: 1uF, Capacitor_SMD:C_0805_2012Metric, symbol Device:C_Small
- added C45: 10uF, Capacitor_SMD:C_0603_1608Metric, symbol Device:C_Small
- added FB7, FB8: 21 Ohm, Inductor_SMD:L_0805_2012Metric, symbol dk_Ferrite-Beads-and-Chips:MPZ2012S601AT000
- added U10: 74AUP1G74, Package_SO:VSSOP-8_2.3x2mm_P0.5mm, symbol 74xGxx:74AUC1G74
- added U11: MCP1755S-3302E/DB, Package_TO_SOT_SMD:SOT-223-3_TabPin2, symbol Regulator_Linear:MCP1703A-1202_SOT223
- added U12: FIN1047, Package_SO:TSSOP-16_4.4x5mm_P0.65mm, symbol Interface:SN65LVDS047PW
- added X1: Si570, input:QFN-8_5x7_Pitch2.54mm, symbol ilemt_input:Si570
Connections:
- net labels added: FILT_+5VDIG, FPGA_CLK+, FPGA_CLK-, GND, MCLK, MCLK_ENA, OUT_CLK+, OUT_CLK-, OVDD, SCL, SDA
- wire segments 0 -> 64
Other:
- note added: "Clock oscillator and distribution"
- note added: "To FPGA"
- note added: "To minimize MCLK jitter, we derive it directly from our clean clock, \nrather than running it rhough the FPGA. When MCLK_ENA is asserted\nthe next clock edge causes MCLK to go high."
- note added: "To output slot"
