File: main/main_board/clock.sch (KiCad schematic (older format))
At the start: 11 parts, among them J2 MCLK, U10 74AUP1G74, U12 FIN1047, X2 Si570

Commit message: Various preparations for routing the main board. Cleaned up the BOM and reconciled it with the Digikey BOM, so lots of component attributes have changed. This involved pinning down some components which had been vague, especially ferrite beads and chip capacitors. 1uF capacitors have all been changed to 10uF. Changed CARDSEL lines to be buffered rather than filtered, since we had the unused buffers sitting there. Another pass on the Microzed pin mapping.  Brought out the DEBUG LVDS line, and tweaked orderings. Added RC filter and pullups on I2C and PROBE_CONFIG.  We might need level translators here to get >=3.3V Added mount holes for the low volt regulator daughtercard, and dimensioned the connector location.
Parts:
- C41, C42, C44, C46: DK line 2 -> 18; MPN (none) -> CC0603KRX7R8BB104; Manufacturer (none) -> Yageo
- FB7: value 21 Ohm -> 300 Ohm; footprint Inductor_SMD:L_0805_2012Metric -> Capacitor_SMD:C_2220_5650Metric; DK line 24 -> 13; Description FERRITE BEAD 21 OHM 0805, 100 nH, 5 mOhm -> FERRITE BEAD 300 OHM 2220 1LN; Digikey 587-1765-1-ND -> 240-2430-1-ND; Family Ferrite Beads and Chips -> (none); MPN HZ0805C202R-10 -> HI2220R301R-10; Manufacturer (none) -> Laird-Signal Integrity Products
- J2: DK line 35 -> (none); Description (none) -> CONN MMCX JACK STR 50 OHM PCB; Digikey (none) -> WM5557-ND; MPN (none) -> 0734151471; Manufacturer (none) -> Molex
- R7: DK line 48 -> 31; Description RES SMD 1K OHM 0.1% 1/10W 0603 -> RES 1K OHM 1% 1/8W 0603; Digikey P1.0KDBCT-ND -> RNCP0603FTD1K00CT-ND; MPN (none) -> RNCP0603FTD1K00; Manufacturer (none) -> Stackpole Electronics Inc
- R8: DK line (none) -> 33; Description (none) -> RES 33.2 OHM 1% 1/8W 0603; Digikey (none) -> RNCP0603FTD33R2CT-ND; MPN (none) -> RNCP0603FTD33R2; Manufacturer (none) -> Stackpole Electronics Inc
- U10: DK line (none) -> 3; MFG Nexperia USA Inc. -> (none); Manufacturer (none) -> Nexperia USA Inc.
- U12: DK line 38 -> 27; MPN (none) -> FIN1047MTCX; Manufacturer (none) -> ON Semiconductor
- X2: value Si570 -> 570CAC000121DG; DK line (none) -> 19; Description (none) -> XTAL OSC XO 100.0000MHZ CMOS SMD; Digikey (none) -> 336-2519-ND; MPN (none) -> 570CAC000121DG; Manufacturer (none) -> Silicon Labs
Connections:
- wire segments 61 -> 59
- no-connect marks 6 -> 8
Changed lines of the file:
@@
 P 2900 3750
 F 0 "X2" H 2400 3300 50  0000 C CNN
-F 1 "Si570" H 2350 3400 50  0000 C CNN
+F 1 "570CAC000121DG" H 2350 3400 50  0000 C CNN
 F 2 "input:QFN-8_5x7_Pitch2.54mm" H 2900 3750 50  0001 C CNN
 F 3 "https://www.silabs.com/documents/public/data-sheets/si570.pdf" H 2900 3750 50  0001 C CNN
+F 4 "XTAL OSC XO 100.0000MHZ CMOS SMD" H 2900 3750 50  0001 C CNN "Description"
+F 5 "336-2519-ND" H 2900 3750 50  0001 C CNN "Digikey"
+F 6 "570CAC000121DG" H 2900 3750 50  0001 C CNN "MPN"
+F 7 "Silicon Labs" H 2900 3750 50  0001 C CNN "Manufacturer"
+F 8 "19" H 2900 3750 50  0001 C CNN "DK line"
 	1    2900 3750
 	1    0    0    -1
@@
 F 1 "100nF" V 2525 2850 50  0000 L CNN
 F 2 "Capacitor_SMD:C_0603_1608Metric" H 2650 2950 50  0001 C CNN
-F 3 "~" H 2650 2950 50  0001 C CNN
+F 3 "https://www.yageo.com/upload/media/product/productsearch/datasheet/mlcc/UPY-GPHC_X7R_6.3V-to-50V_18.pdf" H 2650 2950 50  0001 C CNN
 F 4 "CAP CER 0.1UF 25V X7R 0603" H 2650 2950 50  0001 C CNN "Description"
 F 5 "311-1341-1-ND" H 2650 2950 50  0001 C CNN "Digikey"
-F 6 "2" H 2650 2950 50  0001 C CNN "DK line"
+F 6 "18" H 2650 2950 50  0001 C CNN "DK line"
+F 7 "" H 2650 2950 50  0001 C CNN "MFG"
+F 8 "CC0603KRX7R8BB104" H 2650 2950 50  0001 C CNN "MPN"
+F 9 "Yageo" H 2650 2950 50  0001 C CNN "Manufacturer"
 	1    2650 2950
 	0    1    1    0
@@
 F 1 "100nF" V 4875 3875 50  0000 L CNN
 F 2 "Capacitor_SMD:C_0603_1608Metric" H 4750 4000 50  0001 C CNN
-F 3 "~" H 4750 4000 50  0001 C CNN
+F 3 "https://www.yageo.com/upload/media/product/productsearch/datasheet/mlcc/UPY-GPHC_X7R_6.3V-to-50V_18.pdf" H 4750 4000 50  0001 C CNN
 F 4 "CAP CER 0.1UF 25V X7R 0603" H 4750 4000 50  0001 C CNN "Description"
 F 5 "311-1341-1-ND" H 4750 4000 50  0001 C CNN "Digikey"
-F 6 "2" H 4750 4000 50  0001 C CNN "DK line"
+F 6 "18" H 4750 4000 50  0001 C CNN "DK line"
+F 7 "" H 4750 4000 50  0001 C CNN "MFG"
+F 8 "CC0603KRX7R8BB104" H 4750 4000 50  0001 C CNN "MPN"
+F 9 "Yageo" H 4750 4000 50  0001 C CNN "Manufacturer"
 	1    4750 4000
 	0    -1   -1   0
@@
 F 4 "1727-6029-1-ND" H 4450 4450 50  0001 C CNN "Digikey"
 F 5 "74AUP1G74DC,125" H 4450 4450 50  0001 C CNN "MPN"
-F 6 "Nexperia USA Inc." H 4450 4450 50  0001 C CNN "MFG"
+F 6 "" H 4450 4450 50  0001 C CNN "MFG"
 F 7 "IC FF D-TYPE SNGL 1BIT 8VSSOP" H 4450 4450 50  0001 C CNN "Description"
+F 8 "Nexperia USA Inc." H 4450 4450 50  0001 C CNN "Manufacturer"
+F 9 "3" H 4450 4450 50  0001 C CNN "DK line"
 	1    4450 4450
 	1    0    0    -1
@@
 F 1 "100nF" V 3275 2825 50  0000 L CNN
 F 2 "Capacitor_SMD:C_0603_1608Metric" H 3150 2950 50  0001 C CNN
-F 3 "~" H 3150 2950 50  0001 C CNN
+F 3 "https://www.yageo.com/upload/media/product/productsearch/datasheet/mlcc/UPY-GPHC_X7R_6.3V-to-50V_18.pdf" H 3150 2950 50  0001 C CNN
 F 4 "CAP CER 0.1UF 25V X7R 0603" H 3150 2950 50  0001 C CNN "Description"
 F 5 "311-1341-1-ND" H 3150 2950 50  0001 C CNN "Digikey"
-F 6 "2" H 3150 2950 50  0001 C CNN "DK line"
+F 6 "18" H 3150 2950 50  0001 C CNN "DK line"
+F 7 "" H 3150 2950 50  0001 C CNN "MFG"
+F 8 "CC0603KRX7R8BB104" H 3150 2950 50  0001 C CNN "MPN"
+F 9 "Yageo" H 3150 2950 50  0001 C CNN "Manufacturer"
 	1    3150 2950
 	0    -1   -1   0
@@
 F 4 "IC DRIVER 4/0 16TSSOP" H 7400 3600 50  0001 C CNN "Description"
 F 5 "FIN1047MTCXFSCT-ND" H 7400 3600 50  0001 C CNN "Digikey"
-F 6 "38" H 7400 3600 50  0001 C CNN "DK line"
+F 6 "27" H 7400 3600 50  0001 C CNN "DK line"
+F 7 "FIN1047MTCX" H 7400 3600 50  0001 C CNN "MPN"
+F 8 "ON Semiconductor" H 7400 3600 50  0001 C CNN "Manufacturer"
 	1    7400 3600
 	1    0    0    -1
@@
 F 1 "100nF" V 7525 2425 50  0000 L CNN
 F 2 "Capacitor_SMD:C_0603_1608Metric" H 7650 2550 50  0001 C CNN
-F 3 "~" H 7650 2550 50  0001 C CNN
+F 3 "https://www.yageo.com/upload/media/product/productsearch/datasheet/mlcc/UPY-GPHC_X7R_6.3V-to-50V_18.pdf" H 7650 2550 50  0001 C CNN
 F 4 "CAP CER 0.1UF 25V X7R 0603" H 7650 2550 50  0001 C CNN "Description"
 F 5 "311-1341-1-ND" H 7650 2550 50  0001 C CNN "Digikey"
-F 6 "2" H 7650 2550 50  0001 C CNN "DK line"
+F 6 "18" H 7650 2550 50  0001 C CNN "DK line"
+F 7 "" H 7650 2550 50  0001 C CNN "MFG"
+F 8 "CC0603KRX7R8BB104" H 7650 2550 50  0001 C CNN "MPN"
+F 9 "Yageo" H 7650 2550 50  0001 C CNN "Manufacturer"
 	1    7650 2550
 	0    -1   -1   0
@@
 Wire Wire Line
 	7400 2550 7400 2700
-Wire Wire Line
-	6800 3300 6750 3300
-Wire Wire Line
-	6800 3000 6750 3000
 Connection ~ 3550 3600
 Wire Wire Line
@@
 AR Path="/5E525F2C/5EC43544" Ref="FB7"  Part="1"
 F 0 "FB7" V 2750 2750 60  0000 C CNN
-F 1 "21 Ohm" V 2850 2850 60  0000 C CNN
-F 2 "Inductor_SMD:L_0805_2012Metric" H 3100 2700 60  0001 L CNN
-F 3 "https://www.yuden.co.jp/productdata/catalog/chipbeads01_e.pdf" H 3100 2800 60  0001 L CNN
-F 4 "HZ0805C202R-10" H 3100 3000 60  0001 L CNN "MPN"
-F 5 "Ferrite Beads and Chips" H 3100 3200 60  0001 L CNN "Family"
-F 6 "FERRITE BEAD 21 OHM 0805, 100 nH, 5 mOhm" H 3100 3500 60  0001 L CNN "Description"
-F 7 "587-1765-1-ND" H 2900 2500 50  0001 C CNN "Digikey"
-F 8 "24" H 2900 2500 50  0001 C CNN "DK line"
+F 1 "300 Ohm" V 2850 2850 60  0000 C CNN
+F 2 "Capacitor_SMD:C_2220_5650Metric" H 3100 2700 60  0001 L CNN
+F 3 "https://media.digikey.com/pdf/Data%20Sheets/Laird%20Technologies/Ferrite_EMI_Catalog.pdf" H 3100 2800 60  0001 L CNN
+F 4 "HI2220R301R-10" H 3100 3000 60  0001 L CNN "MPN"
+F 5 "" H 3100 3200 60  0001 L CNN "Family"
+F 6 "FERRITE BEAD 300 OHM 2220 1LN" H 3100 3500 60  0001 L CNN "Description"
+F 7 "240-2430-1-ND" H 2900 2500 50  0001 C CNN "Digikey"
+F 8 "13" H 2900 2500 50  0001 C CNN "DK line"
+F 9 "Laird-Signal Integrity Products" H 2900 2500 50  0001 C CNN "Manufacturer"
 	1    2900 2500
 	0    1    1    0
@@
 F 1 "33" V 6100 5075 50  0000 C CNN
 F 2 "Resistor_SMD:R_0603_1608Metric" V 6040 4990 50  0001 C CNN
-F 3 "~" H 6000 5000 50  0001 C CNN
+F 3 "https://www.seielect.com/catalog/sei-rncp.pdf" H 6000 5000 50  0001 C CNN
+F 4 "RES 33.2 OHM 1% 1/8W 0603" H 6000 5000 50  0001 C CNN "Description"
+F 5 "RNCP0603FTD33R2CT-ND" H 6000 5000 50  0001 C CNN "Digikey"
+F 6 "RNCP0603FTD33R2" H 6000 5000 50  0001 C CNN "MPN"
+F 7 "Stackpole Electronics Inc" H 6000 5000 50  0001 C CNN "Manufacturer"
+F 8 "33" H 6000 5000 50  0001 C CNN "DK line"
 	1    6000 5000
 	0    -1   -1   0
@@
 F 1 "MCLK" V 5715 5800 50  0000 C CNN
 F 2 "Connector_Coaxial:MMCX_Molex_73415-1471_Vertical" H 5600 5800 50  0001 C CNN
-F 3 " ~" H 5600 5800 50  0001 C CNN
-F 4 "35" H 5600 5800 50  0001 C CNN "DK line"
+F 3 "https://www.molex.com/pdm_docs/sd/734151471_sd.pdf" H 5600 5800 50  0001 C CNN
+F 4 "" H 5600 5800 50  0001 C CNN "DK line"
+F 5 "CONN MMCX JACK STR 50 OHM PCB" H 5600 5800 50  0001 C CNN "Description"
+F 6 "WM5557-ND" H 5600 5800 50  0001 C CNN "Digikey"
+F 7 "0734151471" H 5600 5800 50  0001 C CNN "MPN"
+F 8 "Molex" H 5600 5800 50  0001 C CNN "Manufacturer"
 	1    5600 5800
 	0    1    1    0
@@
 F 1 "1K" V 5700 5375 50  0000 C CNN
 F 2 "Resistor_SMD:R_0603_1608Metric" V 5640 5290 50  0001 C CNN
-F 3 "~" H 5600 5300 50  0001 C CNN
-F 4 "48" H 5600 5300 50  0001 C CNN "DK line"
-F 5 "RES SMD 1K OHM 0.1% 1/10W 0603" H 5600 5300 50  0001 C CNN "Description"
-F 6 "P1.0KDBCT-ND" H 5600 5300 50  0001 C CNN "Digikey"
+F 3 "https://www.seielect.com/catalog/sei-rncp.pdf" H 5600 5300 50  0001 C CNN
+F 4 "31" H 5600 5300 50  0001 C CNN "DK line"
+F 5 "RES 1K OHM 1% 1/8W 0603" H 5600 5300 50  0001 C CNN "Description"
+F 6 "RNCP0603FTD1K00CT-ND" H 5600 5300 50  0001 C CNN "Digikey"
+F 7 "RNCP0603FTD1K00" H 5600 5300 50  0001 C CNN "MPN"
+F 8 "Stackpole Electronics Inc" H 5600 5300 50  0001 C CNN "Manufacturer"
 	1    5600 5300
 	1    0    0    -1
@@
 Wire Wire Line
 	6350 2200 4450 2200
+NoConn ~ 6800 3000
+NoConn ~ 6800 3300
 $EndSCHEMATC

Commit message: Main board is now fully routed and passing DRC. Minor changes related to pin remapping. I2C and one-wire pullups are to OVDD 3.3V, not VCCIO 2.5V. Changes to supply decoupling and VREF- net in reference.sch, suggested by routing.
Parts:
- FB7: value 300 Ohm -> 180 Ohm; footprint Capacitor_SMD:C_2220_5650Metric -> Inductor_SMD:L_0805_2012Metric; DK line 13 -> 36; Description FERRITE BEAD 300 OHM 2220 1LN -> FERRITE BEAD 180 OHM 0805 1LN; Digikey 240-2430-1-ND -> 732-6123-1-ND; MPN HI2220R301R-10 -> 74279220181; Manufacturer Laird-Signal Integrity Products -> Würth Elektronik
Changed lines of the file:
@@
 AR Path="/5E525F2C/5EC43544" Ref="FB7"  Part="1"
 F 0 "FB7" V 2750 2750 60  0000 C CNN
-F 1 "300 Ohm" V 2850 2850 60  0000 C CNN
-F 2 "Capacitor_SMD:C_2220_5650Metric" H 3100 2700 60  0001 L CNN
-F 3 "https://media.digikey.com/pdf/Data%20Sheets/Laird%20Technologies/Ferrite_EMI_Catalog.pdf" H 3100 2800 60  0001 L CNN
-F 4 "HI2220R301R-10" H 3100 3000 60  0001 L CNN "MPN"
+F 1 "180 Ohm" V 2850 2850 60  0000 C CNN
+F 2 "Inductor_SMD:L_0805_2012Metric" H 3100 2700 60  0001 L CNN
+F 3 "https://katalog.we-online.de/pbs/datasheet/74279220181.pdf" H 3100 2800 60  0001 L CNN
+F 4 "74279220181" H 3100 3000 60  0001 L CNN "MPN"
 F 5 "" H 3100 3200 60  0001 L CNN "Family"
-F 6 "FERRITE BEAD 300 OHM 2220 1LN" H 3100 3500 60  0001 L CNN "Description"
-F 7 "240-2430-1-ND" H 2900 2500 50  0001 C CNN "Digikey"
-F 8 "13" H 2900 2500 50  0001 C CNN "DK line"
-F 9 "Laird-Signal Integrity Products" H 2900 2500 50  0001 C CNN "Manufacturer"
+F 6 "FERRITE BEAD 180 OHM 0805 1LN" H 3100 3500 60  0001 L CNN "Description"
+F 7 "732-6123-1-ND" H 2900 2500 50  0001 C CNN "Digikey"
+F 8 "36" H 2900 2500 50  0001 C CNN "DK line"
+F 9 "Würth Elektronik" H 2900 2500 50  0001 C CNN "Manufacturer"
 	1    2900 2500
 	0    1    1    0
