File: main/main_board/clock.sch (KiCad schematic (older format))
At the start: 15 parts, among them J2 MCLK, J4 CLOCK, U10 74AUP1G74, U12 FIN1047, X2 570CAC000121DG

Commit message: Finishing up main/main_board/main_board.kicad_pcb.  Test points, stiching vias, ground pours.
Parts:
- R8: Description RES 33.2 OHM 1% 1/8W 0603 -> RES 33 OHM 1% 1/10W 0603
Changed lines of the file:
@@
 F 1 "33" V 6100 5075 50  0000 C CNN
 F 2 "Resistor_SMD:R_0603_1608Metric" V 6040 4990 50  0001 C CNN
-F 3 "https://www.seielect.com/catalog/sei-rncp.pdf" H 6000 5000 50  0001 C CNN
-F 4 "RES 33.2 OHM 1% 1/8W 0603" H 6000 5000 50  0001 C CNN "Description"
+F 3 "https://www.seielect.com/catalog/sei-rmcf_rmcp.pdf" H 6000 5000 50  0001 C CNN
+F 4 "RES 33 OHM 1% 1/10W 0603" H 6000 5000 50  0001 C CNN "Description"
 F 5 "RNCP0603FTD33R2CT-ND" H 6000 5000 50  0001 C CNN "Digikey"
 F 6 "RNCP0603FTD33R2" H 6000 5000 50  0001 C CNN "MPN"
