File: main/main_board/microzed.sch (KiCad schematic (older format))
At the start: 0 parts

Commit message: Work on main board.
Parts:
- added C47: 100nF, Capacitor_SMD:C_0603_1608Metric, symbol Device:C_Small
- added R37, R38, R39: 100, Resistor_SMD:R_0603_1608Metric, symbol Device:R_US
- added RN3: 33, Resistor_SMD:R_Array_Convex_4x0603, symbol Device:R_Pack04
- added U13: DS90LV048, Package_SO:TSSOP-16_4.4x5mm_P0.65mm, symbol ilemt_input:FIN1048
Connections:
- new net: RN3.4 (R4.1), U13.10 (RO4)
- new net: RN3.3 (R3.1), U13.11 (RO3)
- new net: RN3.2 (R2.1), U13.14 (RO2)
- new net: RN3.1 (R1.1), U13.15 (RO1)
- new net FPGA_MCLK_ENA+: R37.1, U13.3 (RI2+)
- new net FPGA_MCLK_ENA-: R37.2, U13.4 (RI2-)
- new net FPGA_SCKA+: R38.1, U13.6 (RI3+)
- new net FPGA_SCKA-: R38.2, U13.5 (RI3-)
- new net FPGA_SCKB+: R39.1, U13.7 (RI4+)
- new net FPGA_SCKB-: R39.2, U13.8 (RI4-)
- new net GND: C47.2, U13.12 (GND), U13.9 (~EN)
- new net MCLK_ENA: RN3.7 (R2.2)
- new net OVDD: C47.1, U13.13 (VCC), U13.16 (EN)
- new net SCKA: RN3.6 (R3.2)
- new net SCKB: RN3.5 (R4.2)
