File: main/main_board/reference.sch (KiCad schematic (older format))
At the start: 0 parts

Commit message: Work on main board.
Parts:
- added C?: 1uF, Capacitor_SMD:C_0805_2012Metric, symbol Device:C_Small
- added C?: 10uF, Capacitor_SMD:C_0603_1608Metric, symbol Device:C_Small
- added C?: 330uF, Capacitor_SMD:CP_Elec_8x6.7, symbol Device:CP1_Small
- added C?: 22 uF, Capacitor_THT:C_Rect_L26.5mm_W11.5mm_P22.50mm_MKS4, symbol Device:C_Small
- added FB?: 21 Ohm, Inductor_SMD:L_0805_2012Metric, symbol dk_Ferrite-Beads-and-Chips:MPZ2012S601AT000
- added R?: 200, Resistor_SMD:R_0603_1608Metric, symbol Device:R_US
- added R?: 1K, Resistor_SMD:R_0603_1608Metric, symbol Device:R_US
- added U?: NCP1117STAT3G, Package_TO_SOT_SMD:SOT-223, symbol dk_PMIC-Voltage-Regulators-Linear:NCP1117ST33T3G
Connections:
- net labels added: +10V, GNDA, VREF+, VREF-
- wire segments 0 -> 25
Other:
- note added: "+7.5V"
