File: main/main_board/input_slots.sch (KiCad schematic (older format))
At the start: 22 parts, among them J7 SCKB, J8 SCKA, U14 74LVC541A, U15 FIN1047, U16 FIN1047, U17 FIN1047, U5 DS90LV048, X1 microzed

Commit message: Changes related to pin mapping. There's a new BIST unit in the Microzed symbol, and the unit ordering has changed. I also added SDI lines to the input slots which could be used to configure the ADC in a future version of the input board. Added some wire labels for easier routing.
Parts:
- removed unit 1 of X1
- added M1: microzed, main_board:Microzed, symbol microzed:microzed
Connections:
- net labels added: ICLK_SDI, MCLK_ENA+, MCLK_ENA-, SCKA+, SCKA-, SCKA_DIST, SCKB+, SCKB-, SCKB_DIST
- net labels removed: BIST_MOSI, BIST_MOSI_DIST, BIST_SCLK, BIST_SCLK_DIST, BIST_SYNC, BIST_SYNC_DIST
- wire segments 319 -> 328
- no-connect marks 3 -> 2
Changed lines of the file:
@@
 F16 "SCKA+" I L 15850 2050 50
 F17 "SCKA-" I L 15850 2150 50
+F18 "SDI" I L 15850 2900 50
 $EndSheet
 Wire Wire Line
@@
 F16 "SCKA-" I L 15850 3800 50
 F17 "SCKA+" I L 15850 3700 50
+F18 "SDI" I L 15850 4550 50
 $EndSheet
 $Sheet
@@
 F16 "SCKA+" I L 15850 5400 50
 F17 "SCKA-" I L 15850 5500 50
+F18 "SDI" I L 15850 6250 50
 $EndSheet
 $Sheet
@@
 F16 "SCKA+" I L 15850 7150 50
 F17 "SCKA-" I L 15850 7250 50
+F18 "SDI" I L 15850 8000 50
 $EndSheet
 $Comp
@@
 $Comp
 L microzed:microzed X1
-U 2 1 5F0A97DA
+U 3 1 5F0A97DA
 P 17800 1950
 AR Path="/5F0A97DA" Ref="X1"  Part="2"
-AR Path="/5E525FFE/5F0A97DA" Ref="M1"  Part="2"
+AR Path="/5E525FFE/5F0A97DA" Ref="M1"  Part="3"
 F 0 "M1" H 18000 2200 60  0000 L CNN
 F 1 "microzed" H 18000 2100 60  0000 L CNN
 F 2 "main_board:Microzed" H 18000 2000 60  0001 L CNN
 F 3 "" H 18000 1800 60  0001 L CNN
-	2    17800 1950
+	3    17800 1950
 	1    0    0    -1
 $EndComp
@@
 $Comp
 L microzed:microzed X1
-U 1 1 5F1431B2
-P 2700 11150
-AR Path="/5F1431B2" Ref="X1"  Part="1"
-AR Path="/5E525FFE/5F1431B2" Ref="M1"  Part="1"
-F 0 "M1" H 2900 11400 60  0000 L CNN
-F 1 "microzed" H 2900 11300 60  0000 L CNN
-F 2 "main_board:Microzed" H 2900 11200 60  0001 L CNN
-F 3 "" H 2900 11000 60  0001 L CNN
-	1    2700 11150
-	1    0    0    -1
-$EndComp
-$Comp
-L microzed:microzed X1
-U 3 1 5F159E9E
+U 4 1 5F159E9E
 P 17800 3600
 AR Path="/5F159E9E" Ref="X1"  Part="3"
-AR Path="/5E525FFE/5F159E9E" Ref="M1"  Part="3"
+AR Path="/5E525FFE/5F159E9E" Ref="M1"  Part="4"
 F 0 "M1" H 18000 3850 60  0000 L CNN
 F 1 "microzed" H 18000 3750 60  0000 L CNN
 F 2 "main_board:Microzed" H 18000 3650 60  0001 L CNN
 F 3 "" H 18000 3450 60  0001 L CNN
-	3    17800 3600
+	4    17800 3600
 	1    0    0    -1
 $EndComp
@@
 $Comp
 L microzed:microzed X1
-U 4 1 5F1854CB
+U 5 1 5F1854CB
 P 17800 5300
 AR Path="/5F1854CB" Ref="X1"  Part="4"
-AR Path="/5E525FFE/5F1854CB" Ref="M1"  Part="4"
+AR Path="/5E525FFE/5F1854CB" Ref="M1"  Part="5"
 F 0 "M1" H 18000 5550 60  0000 L CNN
 F 1 "microzed" H 18000 5450 60  0000 L CNN
 F 2 "main_board:Microzed" H 18000 5350 60  0001 L CNN
 F 3 "" H 18000 5150 60  0001 L CNN
-	4    17800 5300
+	5    17800 5300
 	1    0    0    -1
 $EndComp
@@
 $Comp
 L microzed:microzed X1
-U 5 1 5F209C7E
+U 6 1 5F209C7E
 P 17800 7050
 AR Path="/5F209C7E" Ref="X1"  Part="5"
-AR Path="/5E525FFE/5F209C7E" Ref="M1"  Part="5"
+AR Path="/5E525FFE/5F209C7E" Ref="M1"  Part="6"
 F 0 "M1" H 18000 7300 60  0000 L CNN
 F 1 "microzed" H 18000 7200 60  0000 L CNN
 F 2 "main_board:Microzed" H 18000 7100 60  0001 L CNN
 F 3 "" H 18000 6900 60  0001 L CNN
-	5    17800 7050
+	6    17800 7050
 	1    0    0    -1
 $EndComp
@@
 Wire Wire Line
 	15750 3200 15750 3550
-Text GLabel 2600 11550 0    50   Input ~ 0
+Text GLabel 2600 11650 0    50   Input ~ 0
 FPGA_SYSCLK+
-Text GLabel 2600 11650 0    50   Input ~ 0
+Text GLabel 2600 11750 0    50   Input ~ 0
 FPGA_SYSCLK-
 Wire Wire Line
+	2600 11750 2700 11750
+Wire Wire Line
 	2600 11650 2700 11650
-Wire Wire Line
-	2600 11550 2700 11550
 NoConn ~ 9000 11850
 NoConn ~ 6650 6300
@@
 Wire Wire Line
 	8500 2800 8500 8200
-Wire Wire Line
-	6350 8500 4600 8500
-Wire Wire Line
-	4600 11350 4400 11350
-Wire Wire Line
-	4700 11450 4400 11450
 $Comp
 L Device:R_Pack04 RN?
@@
 Wire Wire Line
 	7450 8600 7350 8600
-NoConn ~ 7850 8600
-Wire Wire Line
-	6350 8600 6300 8600
-Wire Wire Line
-	6300 8600 6300 8800
-Connection ~ 6300 8800
-Text GLabel 8000 8300 2    50   Output ~ 0
-BIST_SYNC
-Text GLabel 8000 8400 2    50   Output ~ 0
-BIST_MOSI
-Text GLabel 8000 8500 2    50   Output ~ 0
-BIST_SCLK
-Wire Wire Line
-	8000 8300 7850 8300
-Wire Wire Line
-	8000 8400 7850 8400
-Wire Wire Line
-	8000 8500 7850 8500
-Wire Wire Line
-	4400 8300 4400 11150
-Wire Wire Line
-	4600 8500 4600 11350
-Wire Wire Line
-	4700 8200 4700 11450
-Wire Wire Line
-	4700 8200 6250 8200
+Wire Wire Line
+	4550 8200 6250 8200
 Wire Wire Line
 	6250 8100 6250 8200
@@
 Wire Wire Line
 	6250 8200 6350 8200
-Wire Wire Line
-	4400 8300 6350 8300
-Wire Wire Line
-	4500 8400 6350 8400
+Text Label 4550 10900 1    50   ~ 0
+ICLK_SYNC
+Wire Wire Line
+	7850 8300 8600 8300
+Wire Wire Line
+	8600 8300 8600 2900
+Wire Wire Line
+	8600 2900 15850 2900
+Wire Wire Line
+	7850 8400 8700 8400
+Wire Wire Line
+	8700 8400 8700 4550
+Wire Wire Line
+	8700 4550 15850 4550
+Wire Wire Line
+	7850 8500 8800 8500
+Wire Wire Line
+	8800 8500 8800 6250
+Wire Wire Line
+	8800 6250 15850 6250
+Wire Wire Line
+	7850 8600 8900 8600
+Wire Wire Line
+	8900 8600 8900 8000
+Wire Wire Line
+	8900 8000 15850 8000
+Text Label 5850 11550 0    50   ~ 0
+MCLK_ENA+
+Text Label 5900 11750 0    50   ~ 0
+MCLK_ENA-
+Text Label 6000 11950 0    50   ~ 0
+SCKA+
+Text Label 6000 12150 0    50   ~ 0
+SCKA-
+Text Label 6000 12350 0    50   ~ 0
+SCKB+
+Text Label 6000 12550 0    50   ~ 0
+SCKB-
+Text Label 9750 12050 0    50   ~ 0
+SCKA_DIST
+Text Label 9750 12150 0    50   ~ 0
+SCKB_DIST
+$Comp
+L microzed:microzed M1
+U 2 1 5F079106
+P 2700 11350
+F 0 "M1" H 2900 11600 60  0000 L CNN
+F 1 "microzed" H 2900 11500 60  0000 L CNN
+F 2 "main_board:Microzed" H 2900 11400 60  0001 L CNN
+F 3 "" H 2900 11200 60  0001 L CNN
+	2    2700 11350
+	1    0    0    -1
+$EndComp
+Wire Wire Line
+	4400 11350 4550 11350
+Wire Wire Line
+	4550 8200 4550 11350
+Wire Wire Line
+	4400 11450 4700 11450
+Wire Wire Line
+	4700 11450 4700 8600
+Wire Wire Line
+	4700 8600 6250 8600
 Text Label 4700 10900 1    50   ~ 0
-ICLK_SYNC
-Text Label 4600 10900 1    50   ~ 0
-BIST_SCLK_DIST
-Text Label 4400 10900 1    50   ~ 0
-BIST_SYNC_DIST
-Wire Wire Line
-	4500 11250 4400 11250
-Text Label 4500 10900 1    50   ~ 0
-BIST_MOSI_DIST
-Wire Wire Line
-	4500 8400 4500 11250
+ICLK_SDI
+Wire Wire Line
+	6350 8300 6250 8300
+Wire Wire Line
+	6250 8300 6250 8400
+Connection ~ 6250 8600
+Wire Wire Line
+	6250 8600 6350 8600
+Wire Wire Line
+	6350 8400 6250 8400
+Connection ~ 6250 8400
+Wire Wire Line
+	6250 8400 6250 8500
+Wire Wire Line
+	6350 8500 6250 8500
+Connection ~ 6250 8500
+Wire Wire Line
+	6250 8500 6250 8600
 $EndSCHEMATC

Commit message: Various preparations for routing the main board. Cleaned up the BOM and reconciled it with the Digikey BOM, so lots of component attributes have changed. This involved pinning down some components which had been vague, especially ferrite beads and chip capacitors. 1uF capacitors have all been changed to 10uF. Changed CARDSEL lines to be buffered rather than filtered, since we had the unused buffers sitting there. Another pass on the Microzed pin mapping.  Brought out the DEBUG LVDS line, and tweaked orderings. Added RC filter and pullups on I2C and PROBE_CONFIG.  We might need level translators here to get >=3.3V Added mount holes for the low volt regulator daughtercard, and dimensioned the connector location.
Parts:
- added J3: DEBUG, Connector_Coaxial:MMCX_Molex_73415-1471_Vertical, symbol Connector:Conn_Coaxial
- added R22: 100, Resistor_SMD:R_0603_1608Metric, symbol Device:R_US
- added R27: 1K, Resistor_SMD:R_0603_1608Metric, symbol Device:R_US
- C48, C49, C50, C51, C52, C54: DK line 2 -> 18; MPN (none) -> CC0603KRX7R8BB104; Manufacturer (none) -> Yageo
- J7, J8: DK line 35 -> (none); Description (none) -> CONN MMCX JACK STR 50 OHM PCB; Digikey (none) -> WM5557-ND; MPN (none) -> 0734151471; Manufacturer (none) -> Molex
- R10, R11, R9: DK line 51 -> 29; Description 100 Ohms ±0.1% 0.1W, 1/10W Chip Resistor 0603 (1608 Metric)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 -> RES 100 OHM 1% 1/8W 0603; Digikey P100DBCT-ND -> RNCP0603FTD100RCT-ND; MPN (none) -> RNCP0603FTD100R; Manufacturer (none) -> Stackpole Electronics Inc
- R40, R41: DK line 48 -> 31; Description RES SMD 1K OHM 0.1% 1/10W 0603 -> RES 1K OHM 1% 1/8W 0603; Digikey P1.0KDBCT-ND -> RNCP0603FTD1K00CT-ND; MPN (none) -> RNCP0603FTD1K00; Manufacturer (none) -> Stackpole Electronics Inc
- RN1, RN2, RN4: value 33 -> 33x4; DK line 13 -> 25; MPN (none) -> CAY16-330J4LF; Manufacturer (none) -> Bourns Inc.
- U14: DK line 11 -> 17; MPN (none) -> SN74LVC541ADBR; Manufacturer (none) -> Texas Instruments
- U15, U16, U17: DK line 38 -> 27; MPN (none) -> FIN1047MTCX; Manufacturer (none) -> ON Semiconductor
- U5: DK line 39 -> 26; MPN (none) -> DS90LV048ATMTC/NOPB; Manufacturer (none) -> Texas Instruments
Connections:
- net FPGA_SYSCLK+: now also M1.A048 (SYSCLK+)
- net FPGA_SYSCLK-: now also M1.A050 (SYSCLK-); no longer M1.A048 (SYSCLK+)
- net GND: now also J3.2 (Ext)
- net MCLK_ENA+: now also M1.B081 (ICLK_MCLK_ENA+); no longer M1.B074 (ICLK_DEBUG+)
- net MCLK_ENA-: now also M1.B083 (ICLK_MCLK_ENA-); no longer M1.B076 (ICLK_DEBUG-)
- net SCKA+: now also M1.B082 (SCKA+); no longer M1.B081 (ICLK_MCLK_ENA+)
- net SCKA-: now also M1.B084 (SCKA-); no longer M1.B083 (ICLK_MCLK_ENA-)
- net SCKB+: now also M1.B087 (SCKB+); no longer M1.B082 (SCKA+)
- net SCKB-: now also M1.B089 (SCKB-); no longer M1.B084 (SCKA-)
- net card_slot0/SDI: now also RN2.5 (R4.2); no longer RN2.8 (R1.2)
- net card_slot1/SDI: now also RN2.6 (R3.2); no longer RN2.7 (R2.2)
- net card_slot2/SDI: now also RN2.7 (R2.2); no longer RN2.6 (R3.2)
- net card_slot3/SDI: now also RN2.8 (R1.2); no longer RN2.5 (R4.2)
- net SYNC3: now reaches RN4.1 (R1.1), U14.18 (Y0)
- net SYNC2: now reaches RN4.2 (R2.1), U14.17 (Y1)
- net SYNC1: now reaches RN4.3 (R3.1), U14.16 (Y2)
- net SYNC0: now reaches RN4.4 (R4.1), U14.15 (Y3)
- net SDI0: now reaches RN2.4 (R4.1), U14.11 (Y7)
- net SDI1: now reaches RN2.3 (R3.1), U14.12 (Y6)
- net SDI2: now reaches RN2.2 (R2.1), U14.13 (Y5)
- net SDI3: now reaches RN2.1 (R1.1), U14.14 (Y4)
- net SCKA_RX: now reaches R41.1, RN1.3 (R3.1), U5.11 (RO3)
- net SCKB_RX: now reaches R40.1, RN1.4 (R4.1), U5.10 (RO4)
- net DEBUG-: now reaches U5.1 (RI1-)
- net DEBUG-: now also M1.B076 (ICLK_DEBUG-), R22.2
- net MCLK_ENA_RX: now reaches RN1.2 (R2.1), U5.14 (RO2)
- net DEBUG_RX: now reaches RN1.1 (R1.1), U5.15 (RO1)
- net DEBUG_RX: now also R27.1
- net DEBUG+: now reaches U5.2 (RI1+)
- net DEBUG+: now also M1.B074 (ICLK_DEBUG+), R22.1
- new net DEBUG_JACK: J3.1 (In), R27.2
Other:
- moved on the sheet: C48, C49, J7, J8, M1B, R10, R11, R40, R41, R9, RN1, U14
