File: main/main_board/main_board.kicad_pcb (KiCad board)
At the start: 4 copper layers, 208.3 x 261.9 mm, 162 parts, among them J1 Conn_02x08_Odd_Even, J2 MCLK, J7 SCKB, J8 SCKA, J9 MCLK, M1 microzed, P2 my_pcie_8x, P3 my_pcie_8x, P4 my_pcie_8x, P5 my_pcie_8x, P6 my_pcie_8x, U1 MAX6220ASA-5.0+, U10 74AUP1G74, U12 FIN1047, U14 74LVC541A, U15 FIN1047, U16 FIN1047, U17 FIN1047, U2 OPA209, U3 MCP1755S-3302E/DB, U4 MCP1755S-3302E/DB, U5 DS90LV048, U6 AP3761C-25SP, U7 MCP1755S-5002E/DB, U8 DAC80004IPW, X2 Si570

Commit message: Mostly work on main board layout. Aligned things on mm grid for easier routing, moved things around to create routing area. Neatened up component groups onto the grid. Parts of the routing plan are now drawn on the PCB.  See also notebook.txt. Reduced pad size of the PCIE connector, tweaked design rule clearances. Minor schematic tweaks.
Parts:
- removed J9: MCLK, Connector_Coaxial:MMCX_Molex_73415-1471_Vertical
- removed R42: 1K, Resistor_SMD:R_0603_1608Metric
- added C67: 10uF, Capacitor_SMD:C_0603_1608Metric, F.Cu at (145.8, 108.0)
- added C68: 10uF, Capacitor_SMD:C_0603_1608Metric, F.Cu at (138.6, 108.0)
- added C69: 10uF, Capacitor_SMD:C_0603_1608Metric, F.Cu at (146.6, 51.6)
- C14: value 1uF -> 10uF; footprint Capacitor_SMD:C_0805_2012Metric -> Capacitor_SMD:C_0603_1608Metric
- moved C50 121.0 mm to (225.6, 122.6)
- moved C12 110.9 mm to (38.0, 235.9), turned to 180 degrees
- moved U15 110.7 mm to (220.0, 122.6), turned to 180 degrees
- moved C21 99.4 mm to (38.0, 213.9), turned to 180 degrees
- moved C13 94.5 mm to (38.0, 224.9), turned to 180 degrees
- moved C51 87.2 mm to (225.6, 131.4), turned to 0 degrees
- moved U16 85.8 mm to (220.0, 131.3), turned to 180 degrees
- moved C54 82.4 mm to (225.6, 114.0), turned to 0 degrees
- moved RN1 81.4 mm to (229.6, 114.0), turned to 0 degrees
- moved C42 79.3 mm to (197.8, 60.8), turned to 180 degrees
- moved C41 78.6 mm to (201.2, 60.8)
- moved C14 78.4 mm to (137.8, 51.6)
- moved J2 75.1 mm to (216.1, 57.7)
- moved U17 74.1 mm to (220.0, 140.0), turned to 180 degrees
- moved C52 73.2 mm to (225.6, 140.0), turned to 0 degrees
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Connections:
- net Net-(C41-Pad1) renamed /clock/VDD_CLK
- net Net-(C56-Pad1) renamed /microzed/VCCO
- net Net-(M1-PadB010) renamed /microzed/VCCIO_EN
- net Net-(M1-PadB067) renamed /input_slots/BIST_SYNC_DIST
- net Net-(M1-PadB068) renamed /input_slots/BIST_SCLK_DIST
- net Net-(M1-PadB069) renamed /input_slots/BIST_MOSI_DIST
- net Net-(M1-PadB070) renamed /input_slots/ICLK_SYNC
- net Net-(R7-Pad1) renamed /clock/MCLK_DIST
- net Net-(U10-Pad1) renamed /clock/CLK_DIST
- C14 pad 1: GND -> +5_Zedboard
- C14 pad 2: +5_Zedboard -> GND
- P6 pad A40: GND -> +5VANA
- P6 pad A42: +10V -> -6V
- P6 pad B41: +5VANA -> GND
- P6 pad B43: -6V -> +10V
- U12 pad 1: OVDD -> +3V3_CLOCK
Other:
- net class Default: clearance 0.2 -> 0.15
- net class Ground: clearance 0.2 -> 0.15
- net class LVDS: clearance 0.0889 -> 0.15
- net class Power: clearance 0.2 -> 0.15
- net class Slow: clearance 0.2 -> 0.15
- rule trace_clearance: 0.2 -> 0.15
- board text added: "Input routing area (bottom)"
- board text added: "OVDD pour L2"
- board text added: "Output routing area (bottom)"
- board text added: "X coordinates of mechanical features for eurocard subrack (card locations and backplane mounting holes) are aligned on an inch grid because the Horizontal Pitch (HP) is 0.2 Inches. Both the plugin and Zedboard connectors are metric, so we align objects vertically on a metric grid aligned with the plugin connectors. The Zedboard is then placed on this grid. When possible, route on a 0.2mm grid."

Commit message: Changes related to pin mapping. There's a new BIST unit in the Microzed symbol, and the unit ordering has changed. I also added SDI lines to the input slots which could be used to configure the ADC in a future version of the input board. Added some wire labels for easier routing.
Parts:
- removed the REF** at (0.00, 286.8)
- removed the REF** at (0.00, 164.3)
- removed the REF** at (0.00, 153.5)
- removed the REF** at (0.00, 31.0)
- added C70: 100nF, Capacitor_SMD:C_0603_1608Metric, F.Cu at (91.8, 101.3)
- added C71: 100nF, Capacitor_SMD:C_0603_1608Metric, F.Cu at (91.8, 103.8)
- added RN3: 33, Resistor_SMD:R_Array_Convex_4x0603, F.Cu at (87.7, 102.4)
- added RN5: 33, Resistor_SMD:R_Array_Convex_4x0603, F.Cu at (87.7, 107.2)
- added U9: 74LVC541A, input:my-SSOP-20_5.3x7.2mm_P0.65mm, F.Cu at (80.4, 104.4)
- moved C12 86.6 mm to (122.6, 254.4), turned to 270 degrees
- moved C13 85.9 mm to (122.6, 239.6), turned to 270 degrees
- moved C21 29.0 mm to (39.0, 242.9)
- moved J8 28.3 mm to (227.0, 53.0)
- moved C41 25.2 mm to (218.9, 78.8)
- moved FB7 25.2 mm to (215.3, 76.6)
- moved C42 25.2 mm to (215.5, 78.8)
- moved C44 25.2 mm to (222.5, 85.8)
- moved C46 25.2 mm to (212.7, 93.4)
- moved R7 25.2 mm to (226.5, 89.4)
- moved R8 25.2 mm to (226.5, 91.2)
- moved U10 25.2 mm to (221.7, 88.2)
- moved U12 25.2 mm to (218.5, 93.4)
- moved X2 25.2 mm to (214.9, 85.0)
- moved C22 25.2 mm to (215.5, 74.6)
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Connections:
- net Net-(RN1-Pad5) renamed /input_slots/SCKB_DIST
- net Net-(RN1-Pad6) renamed /input_slots/SCKA_DIST
- M1 pad A009: /input_slots/card_slot2/CARDSEL -> /input_slots/card_slot0/CARDSEL
- M1 pad A010: /input_slots/card_slot3/CARDSEL -> /input_slots/card_slot1/CARDSEL
- M1 pad A011: (no net) -> DOUT8+
- M1 pad A012: (no net) -> DOUT6+
- M1 pad A013: (no net) -> DOUT8-
- M1 pad A014: (no net) -> DOUT6-
- M1 pad A018: (no net) -> DOUT3+
- M1 pad A020: (no net) -> DOUT3-
- M1 pad A023: (no net) -> DOUT1+
- M1 pad A024: (no net) -> DFB4+
- M1 pad A025: (no net) -> DOUT1-
- M1 pad A026: (no net) -> DFB4-
- M1 pad A029: DOUTL1 -> DFB2+
- M1 pad A030: DOUTL3 -> DOUTL6
- M1 pad A031: DOUTL2 -> DFB2-
- M1 pad A035: DOUTL5 -> DOUTL2
- M1 pad A036: DFB1+ -> DOUTL3
- M1 pad A037: DOUTL6 -> DOUTL1
- M1 pad A038: DFB1- -> DOUTL5
- M1 pad A041: DFB2+ -> DFB1+
- M1 pad A043: DFB2- -> DFB1-
- M1 pad A047: DFB4+ -> DOUT2+
- M1 pad A048: DOUT1+ -> FPGA_SYSCLK+
- M1 pad A049: DFB4- -> DOUT2-
- M1 pad A050: DOUT1- -> FPGA_SYSCLK-
- M1 pad A053: DOUT2+ -> DOUT4+
- M1 pad A054: DOUT3+ -> DOUT5+
- M1 pad A055: DOUT2- -> DOUT4-
- M1 pad A056: DOUT3- -> DOUT5-
- M1 pad A061: DOUT4+ -> DOUT7+
- M1 pad A062: DOUT5+ -> (no net)
- M1 pad A063: DOUT4- -> DOUT7-
- M1 pad A064: DOUT5- -> (no net)
- M1 pad A067: DOUT6+ -> (no net)
- M1 pad A068: DOUT7+ -> (no net)
- M1 pad A069: DOUT6- -> (no net)
- M1 pad A070: DOUT7- -> (no net)
- M1 pad A073: DOUT8+ -> (no net)
- M1 pad A075: DOUT8- -> (no net)
- M1 pad B013: /input_slots/card_slot0/CARDSEL -> /input_slots/card_slot2/CARDSEL
- M1 pad B014: /input_slots/card_slot1/CARDSEL -> /input_slots/card_slot3/CARDSEL
- M1 pad B017: /input_slots/card_slot0/SDOA1+ -> Net-(M1-PadB017)
- M1 pad B018: /input_slots/card_slot0/SDOB1+ -> Net-(M1-PadB018)
- M1 pad B019: /input_slots/card_slot0/SDOA1- -> Net-(M1-PadB019)
- M1 pad B020: /input_slots/card_slot0/SDOB1- -> /input_slots/ICLK_SYNC
- M1 pad B023: /input_slots/card_slot0/SDOA2+ -> /input_slots/ICLK_SDI
- M1 pad B025: /input_slots/card_slot0/SDOA2- -> (no net)
- M1 pad B029: /input_slots/card_slot1/SDOA1+ -> /input_slots/card_slot0/SDOB1+
- M1 pad B030: /input_slots/card_slot1/SDOB1+ -> /input_slots/card_slot0/SDOA1+
- M1 pad B031: /input_slots/card_slot1/SDOA1- -> /input_slots/card_slot0/SDOB1-
- M1 pad B032: /input_slots/card_slot1/SDOB1- -> /input_slots/card_slot0/SDOA1-
- M1 pad B035: /input_slots/card_slot1/SDOA2+ -> /input_slots/card_slot0/SDOA2+
- M1 pad B037: /input_slots/card_slot1/SDOA2- -> /input_slots/card_slot0/SDOA2-
- M1 pad B041: /input_slots/card_slot2/SDOA1+ -> /input_slots/card_slot1/SDOB1+
- M1 pad B042: /input_slots/card_slot2/SDOB1+ -> /input_slots/card_slot1/SDOA1+
- M1 pad B043: /input_slots/card_slot2/SDOA1- -> /input_slots/card_slot1/SDOB1-
- M1 pad B044: /input_slots/card_slot2/SDOB1- -> /input_slots/card_slot1/SDOA1-
- M1 pad B047: /input_slots/card_slot2/SDOA2+ -> /input_slots/card_slot1/SDOA2+
- M1 pad B049: /input_slots/card_slot2/SDOA2- -> /input_slots/card_slot1/SDOA2-
- M1 pad B053: /input_slots/card_slot3/SDOA1+ -> /input_slots/card_slot2/SDOB1+
- M1 pad B054: /input_slots/card_slot3/SDOB1+ -> /input_slots/card_slot2/SDOA1+
- M1 pad B055: /input_slots/card_slot3/SDOA1- -> /input_slots/card_slot2/SDOB1-
- M1 pad B056: /input_slots/card_slot3/SDOB1- -> /input_slots/card_slot2/SDOA1-
- M1 pad B061: /input_slots/card_slot3/SDOA2+ -> /input_slots/card_slot2/SDOA2+
- M1 pad B063: /input_slots/card_slot3/SDOA2- -> /input_slots/card_slot2/SDOA2-
- M1 pad B067: /input_slots/BIST_SYNC_DIST -> /input_slots/card_slot3/SDOB1+
- M1 pad B068: /input_slots/BIST_SCLK_DIST -> /input_slots/card_slot3/SDOA1+
- M1 pad B069: /input_slots/BIST_MOSI_DIST -> /input_slots/card_slot3/SDOB1-
- M1 pad B070: /input_slots/ICLK_SYNC -> /input_slots/card_slot3/SDOA1-
- M1 pad B073: Net-(M1-PadB073) -> /input_slots/card_slot3/SDOA2+
- M1 pad B074: Net-(M1-PadB074) -> (no net)
- M1 pad B075: Net-(M1-PadB075) -> /input_slots/card_slot3/SDOA2-
- M1 pad B076: Net-(M1-PadB076) -> (no net)
- M1 pad B081: Net-(M1-PadB081) -> /input_slots/MCLK_ENA+
- M1 pad B082: FPGA_SYSCLK+ -> /input_slots/SCKA+
- M1 pad B083: Net-(M1-PadB083) -> /input_slots/MCLK_ENA-
- M1 pad B084: FPGA_SYSCLK- -> /input_slots/SCKA-
- M1 pad B087: (no net) -> /input_slots/SCKB+
- M1 pad B089: (no net) -> /input_slots/SCKB-
- P2 pad A8: Net-(P2-PadA8) -> /input_slots/card_slot0/SDI
- P3 pad A8: Net-(P3-PadA8) -> /input_slots/card_slot1/SDI
- P4 pad A8: Net-(P4-PadA8) -> /input_slots/card_slot2/SDI
- P5 pad A8: Net-(P5-PadA8) -> /input_slots/card_slot3/SDI
- R10 pad 1: Net-(M1-PadB074) -> /input_slots/SCKA+
- R10 pad 2: Net-(M1-PadB076) -> /input_slots/SCKA-
- R11 pad 1: Net-(M1-PadB081) -> /input_slots/SCKB+
- R11 pad 2: Net-(M1-PadB083) -> /input_slots/SCKB-
- R9 pad 1: Net-(M1-PadB073) -> /input_slots/MCLK_ENA+
- R9 pad 2: Net-(M1-PadB075) -> /input_slots/MCLK_ENA-
- RN2 pad 5: Net-(RN2-Pad5) -> /input_slots/card_slot3/SDI
- RN2 pad 6: BIST_SCLK -> /input_slots/card_slot2/SDI
- RN2 pad 7: BIST_MOSI -> /input_slots/card_slot1/SDI
- RN2 pad 8: BIST_SYNC -> /input_slots/card_slot0/SDI
- U14 pad 6: /input_slots/BIST_SYNC_DIST -> /input_slots/ICLK_SDI
- U14 pad 7: /input_slots/BIST_MOSI_DIST -> /input_slots/ICLK_SDI
- U14 pad 8: /input_slots/BIST_SCLK_DIST -> /input_slots/ICLK_SDI
- U14 pad 9: GND -> /input_slots/ICLK_SDI
- U5 pad 3: Net-(M1-PadB073) -> /input_slots/MCLK_ENA+
- U5 pad 4: Net-(M1-PadB075) -> /input_slots/MCLK_ENA-
- U5 pad 5: Net-(M1-PadB076) -> /input_slots/SCKA-
- U5 pad 6: Net-(M1-PadB074) -> /input_slots/SCKA+
- U5 pad 7: Net-(M1-PadB081) -> /input_slots/SCKB+
- U5 pad 8: Net-(M1-PadB083) -> /input_slots/SCKB-
Other:
- board text added: "+5VDIG bus top"
- board text added: "3V3 clock"
- board text added: "OVDD bus top"
- board text added: "Power and VREF busses, top and L2"
- board text added: "Power busses top and L2"
- board text added: "bus taps, bot vertical"
- board text removed: "OVDD pour L2"

Commit message: Various preparations for routing the main board. Cleaned up the BOM and reconciled it with the Digikey BOM, so lots of component attributes have changed. This involved pinning down some components which had been vague, especially ferrite beads and chip capacitors. 1uF capacitors have all been changed to 10uF. Changed CARDSEL lines to be buffered rather than filtered, since we had the unused buffers sitting there. Another pass on the Microzed pin mapping.  Brought out the DEBUG LVDS line, and tweaked orderings. Added RC filter and pullups on I2C and PROBE_CONFIG.  We might need level translators here to get >=3.3V Added mount holes for the low volt regulator daughtercard, and dimensioned the connector location.
Parts:
- removed the C1 at (206.8, 265.9)
- removed the C2 at (191.0, 270.6)
- removed the C3 at (206.8, 259.2)
- removed the R1 at (195.0, 270.6)
- removed the R2 at (199.0, 270.6)
- removed the REF** at (226.1, 153.4)
- removed the REF** at (195.6, 30.9)
- removed the REF** at (195.6, 153.4)
- removed the REF** at (165.1, 153.4)
- removed the REF** at (134.6, 153.4)
- removed the REF** at (104.1, 153.4)
- removed the REF** at (73.7, 153.4)
- removed the REF** at (43.2, 153.4)
- removed the REF** at (134.6, 30.9)
- removed the REF** at (73.7, 30.9)
- removed the REF** at (226.1, 164.3)
- added C72: 220pF, Capacitor_SMD:C_0603_1608Metric, F.Cu at (134.2, 91.8)
- added C73: 220pF, Capacitor_SMD:C_0603_1608Metric, F.Cu at (127.8, 91.8)
- added C74: 220pF, Capacitor_SMD:C_0603_1608Metric, F.Cu at (131.0, 91.8)
- added J3: DEBUG, Connector_Coaxial:MMCX_Molex_73415-1471_Vertical, F.Cu at (227.0, 44.3)
- added R13: 1.5K, Resistor_SMD:R_0603_1608Metric, F.Cu at (131.0, 88.4)
- added R18: 1.5K, Resistor_SMD:R_0603_1608Metric, F.Cu at (127.8, 88.4)
- added R19: 33, Resistor_SMD:R_0603_1608Metric, F.Cu at (131.0, 95.2)
- added R20: 33, Resistor_SMD:R_0603_1608Metric, F.Cu at (127.8, 95.2)
- added R21: 33, Resistor_SMD:R_0603_1608Metric, F.Cu at (134.2, 95.2)
- added R22: 100, Resistor_SMD:R_0603_1608Metric, F.Cu at (214.0, 110.4)
- added R26: 1.5K, Resistor_SMD:R_0603_1608Metric, F.Cu at (134.2, 88.4)
- added R27: 1K, Resistor_SMD:R_0603_1608Metric, F.Cu at (227.4, 108.6)
- added REF**: MountingHole_3.2mm_M3_Pad, MountingHole:MountingHole_3.2mm_M3_Pad, F.Cu at (36.7, 104.8)
- added REF**: MountingHole_3.2mm_M3_Pad, MountingHole:MountingHole_3.2mm_M3_Pad, F.Cu at (36.7, 55.2)
- C1, C10, C11, C2, C25, C26, C29, C30, C33, C34, C37, C38, C43, C45, C59, C7: value 1uF -> 10uF 16V
- C15, C16, C17, C18, C24, C27, C28, C31, C32, C35, C36, C39, C40, C47, C53, C57, C58, C63: value 1uF -> 10uF; footprint Capacitor_SMD:C_0805_2012Metric -> Capacitor_SMD:C_0603_1608Metric
- C3: value bulk >=16V -> 47uF
- C4, C5: value 3.3 uF -> 3.3uF
- C61, C62, C64, C65: value 200 pF -> 220pF
- FB3: value 1.2 A -> 300 Ohm; footprint Inductor_SMD:L_0805_2012Metric -> Capacitor_SMD:C_2220_5650Metric
- FB7: value 21 Ohm -> 300 Ohm; footprint Inductor_SMD:L_0805_2012Metric -> Capacitor_SMD:C_2220_5650Metric
- J1: value Conn_02x08_Odd_Even -> Power; moved to B.Cu
- P2, P3, P4, P5, P6: value my_pcie_8x -> PCIE 8x female
- R3: value 40K -> 40.2K
- RN1, RN2, RN3, RN4, RN5: value 33 -> 33x4
- U6: value AP3761C-25SP -> AP7361C-25SP-13
- X2: value Si570 -> 570CAC000121DG
- moved RN3 41.7 mm to (115.3, 133.6)
- moved RN5 41.2 mm to (115.3, 137.8)
- moved U9 41.1 mm to (107.2, 135.6)
- moved C71 41.0 mm to (110.0, 140.6)
- moved C70 34.5 mm to (110.0, 130.6), turned to 180 degrees
- moved REF** 15.2 mm to (210.8, 164.3)
- moved C6 15.2 mm to (180.8, 270.2)
- moved C49 14.7 mm to (110.0, 128.6), turned to 0 degrees
- moved C48 12.8 mm to (110.0, 118.7)
- moved U4 12.8 mm to (94.4, 124.0), turned to 90 degrees
- moved C58 12.4 mm to (92.1, 130.8), turned to 90 degrees
- moved RN2 12.0 mm to (115.2, 125.8)
- moved RN4 12.0 mm to (115.2, 121.7)
- moved U14 12.0 mm to (107.2, 123.7)
- moved FB7 10.5 mm to (204.8, 77.0)
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Connections:
- net Net-(C1-Pad2) renamed /reference/+10V_REF_1
- net Net-(C2-Pad2) renamed /reference/-6V_REF_1
- net Net-(C3-Pad1) renamed /reference/+10V_REF
- net Net-(C4-Pad1) renamed /reference/U1_NR
- net Net-(C5-Pad1) renamed /reference/U2_IN
- net Net-(C6-Pad1) renamed /reference/U2_V-
- net Net-(C7-Pad2) renamed /reference/U2_V+
- net Net-(C8-Pad1) renamed /reference/U2_OUT
- net Net-(C8-Pad2) renamed /reference/U2_-IN
- net Net-(FB4-Pad1) renamed /BIST_DAC/BIST++_DIST
- net Net-(FB5-Pad1) renamed /BIST_DAC/BIST-+_DIST
- net Net-(FB6-Pad1) renamed /BIST_DAC/BIST+-_DIST
- net Net-(FB8-Pad1) renamed /BIST_DAC/BIST--_DIST
- net Net-(M1-PadB017) renamed /BIST_DAC/BIST_MOSI_ZED
- net Net-(M1-PadB018) renamed /BIST_DAC/BIST_SYNC_ZED
- net Net-(M1-PadB019) renamed /BIST_DAC/BIST_SCLK_ZED
- net Net-(R3-Pad2) renamed /reference/U1_OUT
- net Net-(R40-Pad1) renamed /input_slots/SCKB_RX
- net Net-(R41-Pad1) renamed /input_slots/SCKA_RX
- net Net-(RN1-Pad1) renamed /input_slots/DEBUG_RX
- net Net-(RN1-Pad2) renamed /input_slots/MCLK_ENA_RX
- net Net-(RN2-Pad1) renamed /input_slots/SDI3
- net Net-(RN2-Pad2) renamed /input_slots/SDI2
- net Net-(RN2-Pad3) renamed /input_slots/SDI1
- net Net-(RN2-Pad4) renamed /input_slots/SDI0
- net Net-(RN3-Pad1) renamed /BIST_DAC/IN3_CARDSEL1
- net Net-(RN3-Pad2) renamed /BIST_DAC/IN2_CARDSEL1
- net Net-(RN3-Pad3) renamed /BIST_DAC/IN1_CARDSEL1
- net Net-(RN3-Pad4) renamed /BIST_DAC/IN0_CARDSEL1
- net Net-(RN4-Pad1) renamed /input_slots/SYNC3
- net Net-(RN4-Pad2) renamed /input_slots/SYNC2
- net Net-(RN4-Pad3) renamed /input_slots/SYNC1
- net Net-(RN4-Pad4) renamed /input_slots/SYNC0
- net Net-(RN5-Pad1) renamed /BIST_DAC/BIST_SYNC1
- net Net-(RN5-Pad2) renamed /BIST_DAC/BIST_MOSI1
- net Net-(RN5-Pad3) renamed /BIST_DAC/BIST_SCLK1
- net Net-(RN5-Pad4) renamed /BIST_DAC/UNUSED4
- J1 pad 1: GND -> +5_Zedboard_IN
- J1 pad 10: +5VANA -> GND
- J1 pad 11: GND -> +10V
- J1 pad 12: +10V -> GND
- J1 pad 13: GND -> -6V
- J1 pad 14: -6V -> GND
- J1 pad 2: +5_Zedboard_IN -> GND
- J1 pad 3: GND -> +5_CLOCK_IN
- J1 pad 4: +5_CLOCK_IN -> GND
- J1 pad 5: GND -> +5_DRIVERS_IN
- J1 pad 6: +5_DRIVERS_IN -> GND
- J1 pad 7: GND -> +5VDIG
- J1 pad 8: +5VDIG -> GND
- J1 pad 9: GND -> +5VANA
- M1 pad A009: /input_slots/card_slot0/CARDSEL -> /BIST_DAC/IN3_CARDSEL_ZED
- M1 pad A010: /input_slots/card_slot1/CARDSEL -> /BIST_DAC/IN2_CARDSEL_ZED
- M1 pad B001: SCL -> /microzed/SCL_ZED
- M1 pad B002: SDA -> /microzed/SDA_ZED
- M1 pad B003: PROBE_CONFIG -> /microzed/PROBE_CONFIG_ZED
- M1 pad B013: /input_slots/card_slot2/CARDSEL -> /BIST_DAC/IN1_CARDSEL_ZED
- M1 pad B014: /input_slots/card_slot3/CARDSEL -> /BIST_DAC/IN0_CARDSEL_ZED
- M1 pad B074: (no net) -> /input_slots/DEBUG+
- M1 pad B076: (no net) -> /input_slots/DEBUG-
- P2 pad A3: /input_slots/card_slot0/CARDSEL -> IN0_CARDSEL
- P3 pad A3: /input_slots/card_slot1/CARDSEL -> IN1_CARDSEL
- P4 pad A3: /input_slots/card_slot2/CARDSEL -> IN2_CARDSEL
- P5 pad A3: /input_slots/card_slot3/CARDSEL -> IN3_CARDSEL
- RN2 pad 5: /input_slots/card_slot3/SDI -> /input_slots/card_slot0/SDI
- RN2 pad 6: /input_slots/card_slot2/SDI -> /input_slots/card_slot1/SDI
- RN2 pad 7: /input_slots/card_slot1/SDI -> /input_slots/card_slot2/SDI
- RN2 pad 8: /input_slots/card_slot0/SDI -> /input_slots/card_slot3/SDI
- RN3 pad 5: Net-(RN3-Pad5) -> IN0_CARDSEL
- RN3 pad 6: Net-(RN3-Pad6) -> IN1_CARDSEL
- RN3 pad 7: Net-(RN3-Pad7) -> IN2_CARDSEL
- RN3 pad 8: Net-(RN3-Pad8) -> IN3_CARDSEL
- U5 pad 1: Net-(U5-Pad1) -> /input_slots/DEBUG-
- U5 pad 2: Net-(U5-Pad2) -> /input_slots/DEBUG+
- U9 pad 2: GND -> /BIST_DAC/IN3_CARDSEL_ZED
- U9 pad 3: GND -> /BIST_DAC/IN2_CARDSEL_ZED
- U9 pad 4: GND -> /BIST_DAC/IN1_CARDSEL_ZED
- U9 pad 5: GND -> /BIST_DAC/IN0_CARDSEL_ZED
Other:
- board text added: "OVDD pour bottom?"
