File: main/main_board/card_slot.sch (KiCad schematic (older format))
At the start: 5 parts, among them P1 my_pcie_8x

Commit message: Changes related to pin mapping. There's a new BIST unit in the Microzed symbol, and the unit ordering has changed. I also added SDI lines to the input slots which could be used to configure the ADC in a future version of the input board. Added some wire labels for easier routing.
Connections:
- net SDI: now reaches P1.A8
- no-connect marks 7 -> 6
Changed lines of the file:
@@
 $Descr A4 11693 8268
 encoding utf-8
-Sheet 10 12
+Sheet 7 12
 Title ""
 Date ""
@@
 AR Path="/5E525FFE/5EBAAF8F/5E67C68B" Ref="P4"  Part="3"
 AR Path="/5E525FFE/5EBAAFA1/5E67C68B" Ref="P5"  Part="3"
-F 0 "P5" H 2900 3550 50  0000 C CNN
+F 0 "P2" H 2900 3550 50  0000 C CNN
 F 1 "my_pcie_8x" H 2900 3050 50  0000 C CNN
 F 2 "input:PCIE_8x_female" H 2900 4050 50  0001 C CNN
@@
 AR Path="/5E525FFE/5EBAAF8F/5E682A6A" Ref="P4"  Part="5"
 AR Path="/5E525FFE/5EBAAFA1/5E682A6A" Ref="P5"  Part="5"
-F 0 "P5" H 6750 1550 50  0000 C CNN
+F 0 "P2" H 6750 1550 50  0000 C CNN
 F 1 "my_pcie_8x" H 6750 1050 50  0000 C CNN
 F 2 "input:PCIE_8x_female" H 6750 2050 50  0001 C CNN
@@
 AR Path="/5E525FFE/5EBAAF8F/5E625DE8" Ref="P4"  Part="6"
 AR Path="/5E525FFE/5EBAAFA1/5E625DE8" Ref="P5"  Part="6"
-F 0 "P5" H 6750 2600 50  0000 C CNN
+F 0 "P2" H 6750 2600 50  0000 C CNN
 F 1 "my_pcie_8x" H 6750 2100 50  0000 C CNN
 F 2 "input:PCIE_8x_female" H 6750 3100 50  0001 C CNN
@@
 AR Path="/5E525FFE/5EBAAF8F/5E625DE9" Ref="P4"  Part="7"
 AR Path="/5E525FFE/5EBAAFA1/5E625DE9" Ref="P5"  Part="7"
-F 0 "P5" H 6750 3650 50  0000 C CNN
+F 0 "P2" H 6750 3650 50  0000 C CNN
 F 1 "my_pcie_8x" H 6750 3150 50  0000 C CNN
 F 2 "input:PCIE_8x_female" H 6750 4150 50  0001 C CNN
@@
 AR Path="/5E525FFE/5EBAAF8F/5EC152A6" Ref="P4"  Part="2"
 AR Path="/5E525FFE/5EBAAFA1/5EC152A6" Ref="P5"  Part="2"
-F 0 "P5" H 2900 2500 50  0000 C CNN
+F 0 "P2" H 2900 2500 50  0000 C CNN
 F 1 "my_pcie_8x" H 2900 2000 50  0000 C CNN
 F 2 "input:PCIE_8x_female" H 2900 3000 50  0001 C CNN
@@
 AR Path="/5E525FFE/5EBAAF8F/5E681104" Ref="P4"  Part="1"
 AR Path="/5E525FFE/5EBAAFA1/5E681104" Ref="P5"  Part="1"
-F 0 "P5" H 2900 1500 50  0000 C CNN
+F 0 "P2" H 2900 1500 50  0000 C CNN
 F 1 "my_pcie_8x" H 2900 1000 50  0000 C CNN
 F 2 "input:PCIE_8x_female" H 2900 2000 50  0001 C CNN
@@
 NoConn ~ 3250 1800
 NoConn ~ 3250 4600
-NoConn ~ 2550 2200
 NoConn ~ 3250 2200
 Wire Wire Line
@@
 AR Path="/5E525FFE/5EBAAF8F/5EC152A7" Ref="P4"  Part="4"
 AR Path="/5E525FFE/5EBAAFA1/5EC152A7" Ref="P5"  Part="4"
-F 0 "P5" H 2900 4600 50  0000 C CNN
+F 0 "P2" H 2900 4600 50  0000 C CNN
 F 1 "my_pcie_8x" H 2900 4100 50  0000 C CNN
 F 2 "input:PCIE_8x_female" H 2900 5100 50  0001 C CNN
@@
 AR Path="/5E525FFE/5EBAAF8F/5ED81315" Ref="C32"  Part="1"
 AR Path="/5E525FFE/5EBAAFA1/5ED81315" Ref="C36"  Part="1"
-F 0 "C36" V 4221 6050 50  0000 C CNN
+F 0 "C24" V 4221 6050 50  0000 C CNN
 F 1 "1uF" V 4312 6050 50  0000 C CNN
 F 2 "Capacitor_SMD:C_0805_2012Metric" H 4450 6050 50  0001 C CNN
@@
 AR Path="/5E525FFE/5EBAAF8F/5EDA5F14" Ref="C33"  Part="1"
 AR Path="/5E525FFE/5EBAAFA1/5EDA5F14" Ref="C37"  Part="1"
-F 0 "C37" V 4671 6050 50  0000 C CNN
+F 0 "C25" V 4671 6050 50  0000 C CNN
 F 1 "1uF" V 4762 6050 50  0000 C CNN
 F 2 "Capacitor_SMD:C_0805_2012Metric" H 4900 6050 50  0001 C CNN
@@
 AR Path="/5E525FFE/5EBAAF8F/5EDBD896" Ref="C34"  Part="1"
 AR Path="/5E525FFE/5EBAAFA1/5EDBD896" Ref="C38"  Part="1"
-F 0 "C38" V 5121 6050 50  0000 C CNN
+F 0 "C26" V 5121 6050 50  0000 C CNN
 F 1 "1uF" V 5212 6050 50  0000 C CNN
 F 2 "Capacitor_SMD:C_0805_2012Metric" H 5350 6050 50  0001 C CNN
@@
 AR Path="/5E525FFE/5EBAAF8F/5EDCC5E2" Ref="C35"  Part="1"
 AR Path="/5E525FFE/5EBAAFA1/5EDCC5E2" Ref="C39"  Part="1"
-F 0 "C39" V 5571 6050 50  0000 C CNN
+F 0 "C27" V 5571 6050 50  0000 C CNN
 F 1 "1uF" V 5662 6050 50  0000 C CNN
 F 2 "Capacitor_SMD:C_0805_2012Metric" H 5800 6050 50  0001 C CNN
@@
 	1    0    0    -1
 $EndComp
+Text HLabel 2350 2200 0    50   Input ~ 0
+SDI
+Wire Wire Line
+	2550 2200 2350 2200
 $EndSCHEMATC

Commit message: Various preparations for routing the main board. Cleaned up the BOM and reconciled it with the Digikey BOM, so lots of component attributes have changed. This involved pinning down some components which had been vague, especially ferrite beads and chip capacitors. 1uF capacitors have all been changed to 10uF. Changed CARDSEL lines to be buffered rather than filtered, since we had the unused buffers sitting there. Another pass on the Microzed pin mapping.  Brought out the DEBUG LVDS line, and tweaked orderings. Added RC filter and pullups on I2C and PROBE_CONFIG.  We might need level translators here to get >=3.3V Added mount holes for the low volt regulator daughtercard, and dimensioned the connector location.
Parts:
- C24, C27: value 1uF -> 10uF; footprint Capacitor_SMD:C_0805_2012Metric -> Capacitor_SMD:C_0603_1608Metric; DK line 27 -> 20; Description CAP CER 1UF 16V X7R 0805 -> CAP CER 10UF 6.3V X5R 0603; Digikey 1276-6471-1-ND -> 478-5318-1-ND; MPN CL21B105KOFNNNG -> 06036D106MAT2A; Manufacturer (none) -> AVX
- C25, C26: value 1uF -> 10uF 16V; DK line 27 -> 10; Description CAP CER 1UF 16V X7R 0805 -> CAP CER 10UF 16V X5R 0805; Digikey 1276-6471-1-ND -> 399-8012-1-ND; MPN CL21B105KOFNNNG -> C0805C106K4PACTU; Manufacturer (none) -> KEMET
- P1: value my_pcie_8x -> PCIE 8x female; DK line (none) -> 2; Description (none) -> CONN PCI EXP FEMALE 98POS 0.039; Digikey (none) -> 609-1970-ND; MPN (none) -> 10018783-10102TLF; Manufacturer (none) -> Amphenol ICC (FCI)
Other:
- moved on the sheet: C36, C37, C38, C39, P5A, P5B, P5C, P5D, P5E, P5F, P5G
