File: dac/out_chan.sch (KiCad schematic (older format))
At the start: 22 parts, among them U101 OPA2210, U102 OPA1611

Commit message: Mainly BOM tweaks, working on setting up more systematic database of parts and BOMs in parts/
Parts:
- R107, R108, R109: DK line I.52 -> I.9; Description RES SMD 10 OHM 5% 1/2W 0805 -> RES SMD 10 OHM 5% 0.4W 0805; MPN CRCW080510R0JNEAHP -> ESR10EZPJ100; Manufacturer Vishay Dale -> Rohm Semiconductor
Changed lines of the file:
@@
 AR Path="/5F8C3863/5F8AE34F/5F81F6FE" Ref="#PWR0303"  Part="1"
 AR Path="/5F8C3863/5F8B0DF1/5F81F6FE" Ref="#PWR0403"  Part="1"
-F 0 "#PWR0203" H 2300 1550 50  0001 C CNN
+F 0 "#PWR0403" H 2300 1550 50  0001 C CNN
 F 1 "V+" H 2300 1840 50  0000 C CNN
 F 2 "" H 2300 1700 50  0001 C CNN
@@
 AR Path="/5F8C3863/5F8AE34F/5F81F704" Ref="#PWR0304"  Part="1"
 AR Path="/5F8C3863/5F8B0DF1/5F81F704" Ref="#PWR0404"  Part="1"
-F 0 "#PWR0204" H 2300 2700 50  0001 C CNN
+F 0 "#PWR0404" H 2300 2700 50  0001 C CNN
 F 1 "V-" H 2300 2800 50  0000 C CNN
 F 2 "" H 2300 2950 50  0001 C CNN
@@
 AR Path="/5F8C3863/5F8AE34F/5F82D372" Ref="#PWR0305"  Part="1"
 AR Path="/5F8C3863/5F8B0DF1/5F82D372" Ref="#PWR0405"  Part="1"
-F 0 "#PWR0205" H 2800 1550 50  0001 C CNN
+F 0 "#PWR0405" H 2800 1550 50  0001 C CNN
 F 1 "GND" V 2800 1600 50  0000 C CNN
 F 2 "" H 2800 1800 50  0001 C CNN
@@
 AR Path="/5F8C3863/5F8AE34F/5F8302F3" Ref="#PWR0306"  Part="1"
 AR Path="/5F8C3863/5F8B0DF1/5F8302F3" Ref="#PWR0406"  Part="1"
-F 0 "#PWR0206" H 2800 2400 50  0001 C CNN
+F 0 "#PWR0406" H 2800 2400 50  0001 C CNN
 F 1 "GND" V 2800 2450 50  0000 C CNN
 F 2 "" H 2800 2650 50  0001 C CNN
@@
 AR Path="/5F8C3863/5F8AE34F/5F836C8F" Ref="#PWR0301"  Part="1"
 AR Path="/5F8C3863/5F8B0DF1/5F836C8F" Ref="#PWR0401"  Part="1"
-F 0 "#PWR0201" H 1900 2200 50  0001 C CNN
+F 0 "#PWR0401" H 1900 2200 50  0001 C CNN
 F 1 "GND" H 1900 2300 50  0000 C CNN
 F 2 "" H 1900 2450 50  0001 C CNN
@@
 AR Path="/5F8C3863/5F8AE34F/5F8431A7" Ref="#PWR0308"  Part="1"
 AR Path="/5F8C3863/5F8B0DF1/5F8431A7" Ref="#PWR0408"  Part="1"
-F 0 "#PWR0208" H 5550 4900 50  0001 C CNN
+F 0 "#PWR0408" H 5550 4900 50  0001 C CNN
 F 1 "V-" H 5550 5000 50  0000 C CNN
 F 2 "" H 5550 5150 50  0001 C CNN
@@
 AR Path="/5F8C3863/5F8AE34F/5F8431B8" Ref="#PWR0310"  Part="1"
 AR Path="/5F8C3863/5F8B0DF1/5F8431B8" Ref="#PWR0410"  Part="1"
-F 0 "#PWR0210" H 6050 4600 50  0001 C CNN
+F 0 "#PWR0410" H 6050 4600 50  0001 C CNN
 F 1 "GND" V 6050 4650 50  0000 C CNN
 F 2 "" H 6050 4850 50  0001 C CNN
@@
 AR Path="/5F8C3863/5F8AE34F/5F8446CE" Ref="#PWR0307"  Part="1"
 AR Path="/5F8C3863/5F8B0DF1/5F8446CE" Ref="#PWR0407"  Part="1"
-F 0 "#PWR0207" H 5550 3750 50  0001 C CNN
+F 0 "#PWR0407" H 5550 3750 50  0001 C CNN
 F 1 "V+" H 5550 4040 50  0000 C CNN
 F 2 "" H 5550 3900 50  0001 C CNN
@@
 AR Path="/5F8C3863/5F8AE34F/5F8446D4" Ref="#PWR0309"  Part="1"
 AR Path="/5F8C3863/5F8B0DF1/5F8446D4" Ref="#PWR0409"  Part="1"
-F 0 "#PWR0209" H 6050 3750 50  0001 C CNN
+F 0 "#PWR0409" H 6050 3750 50  0001 C CNN
 F 1 "GND" V 6050 3800 50  0000 C CNN
 F 2 "" H 6050 4000 50  0001 C CNN
@@
 AR Path="/5F8C3863/5F8AE34F/5F85A57A" Ref="#PWR0302"  Part="1"
 AR Path="/5F8C3863/5F8B0DF1/5F85A57A" Ref="#PWR0402"  Part="1"
-F 0 "#PWR0202" H 1900 4500 50  0001 C CNN
+F 0 "#PWR0402" H 1900 4500 50  0001 C CNN
 F 1 "GND" H 1900 4600 50  0000 C CNN
 F 2 "" H 1900 4750 50  0001 C CNN
@@
 F 1 "10" V 7000 4400 50  0000 C CNN
 F 2 "Resistor_SMD:R_0805_2012Metric" V 7140 4390 50  0001 C CNN
-F 3 "http://www.vishay.com/docs/20043/crcwhpe3.pdf" H 7100 4400 50  0001 C CNN
-F 4 "RES SMD 10 OHM 5% 1/2W 0805" H 7100 4400 50  0001 C CNN "Description"
-F 5 "CRCW080510R0JNEAHP" H 7100 4400 50  0001 C CNN "MPN"
-F 6 "Vishay Dale" H 7100 4400 50  0001 C CNN "Manufacturer"
+F 3 "https://www.rohm.com/datasheet/ESR01MZPF/esr-e" H 7100 4400 50  0001 C CNN
+F 4 "RES SMD 10 OHM 5% 0.4W 0805" H 7100 4400 50  0001 C CNN "Description"
+F 5 "ESR10EZPJ100" H 7100 4400 50  0001 C CNN "MPN"
+F 6 "Rohm Semiconductor" H 7100 4400 50  0001 C CNN "Manufacturer"
 F 7 "541-10TACT-ND" H 7100 4400 50  0001 C CNN "Digikey"
 F 8 "Thick film surge resist" H 7100 4400 50  0001 C CNN "Notes"
-F 9 "I.52" H 7100 4400 50  0001 C CNN "DK line"
+F 9 "I.9" H 7100 4400 50  0001 C CNN "DK line"
 	1    7100 4400
 	0    1    1    0
@@
 F 1 "10" H 6200 2550 50  0000 C CNN
 F 2 "Resistor_SMD:R_0805_2012Metric" V 6390 2590 50  0001 C CNN
-F 3 "http://www.vishay.com/docs/20043/crcwhpe3.pdf" H 6350 2600 50  0001 C CNN
-F 4 "RES SMD 10 OHM 5% 1/2W 0805" H 6350 2600 50  0001 C CNN "Description"
-F 5 "CRCW080510R0JNEAHP" H 6350 2600 50  0001 C CNN "MPN"
-F 6 "Vishay Dale" H 6350 2600 50  0001 C CNN "Manufacturer"
+F 3 "https://www.rohm.com/datasheet/ESR01MZPF/esr-e" H 6350 2600 50  0001 C CNN
+F 4 "RES SMD 10 OHM 5% 0.4W 0805" H 6350 2600 50  0001 C CNN "Description"
+F 5 "ESR10EZPJ100" H 6350 2600 50  0001 C CNN "MPN"
+F 6 "Rohm Semiconductor" H 6350 2600 50  0001 C CNN "Manufacturer"
 F 7 "541-10TACT-ND" H 6350 2600 50  0001 C CNN "Digikey"
 F 8 "Thick film surge resist" H 6350 2600 50  0001 C CNN "Notes"
-F 9 "I.52" H 6350 2600 50  0001 C CNN "DK line"
+F 9 "I.9" H 6350 2600 50  0001 C CNN "DK line"
 	1    6350 2600
 	-1   0    0    1
@@
 AR Path="/5F8C3863/5F8AE34F/5F8A41D9" Ref="#PWR0311"  Part="1"
 AR Path="/5F8C3863/5F8B0DF1/5F8A41D9" Ref="#PWR0411"  Part="1"
-F 0 "#PWR0211" H 6350 2700 50  0001 C CNN
+F 0 "#PWR0411" H 6350 2700 50  0001 C CNN
 F 1 "GND" H 6350 2800 50  0000 C CNN
 F 2 "" H 6350 2950 50  0001 C CNN
@@
 F 1 "10" V 7750 4400 50  0000 C CNN
 F 2 "Resistor_SMD:R_0805_2012Metric" V 7890 4390 50  0001 C CNN
-F 3 "http://www.vishay.com/docs/20043/crcwhpe3.pdf" H 7850 4400 50  0001 C CNN
-F 4 "RES SMD 10 OHM 5% 1/2W 0805" H 7850 4400 50  0001 C CNN "Description"
-F 5 "CRCW080510R0JNEAHP" H 7850 4400 50  0001 C CNN "MPN"
-F 6 "Vishay Dale" H 7850 4400 50  0001 C CNN "Manufacturer"
+F 3 "https://www.rohm.com/datasheet/ESR01MZPF/esr-e" H 7850 4400 50  0001 C CNN
+F 4 "RES SMD 10 OHM 5% 0.4W 0805" H 7850 4400 50  0001 C CNN "Description"
+F 5 "ESR10EZPJ100" H 7850 4400 50  0001 C CNN "MPN"
+F 6 "Rohm Semiconductor" H 7850 4400 50  0001 C CNN "Manufacturer"
 F 7 "541-10TACT-ND" H 7850 4400 50  0001 C CNN "Digikey"
 F 8 "Thick film surge resist" H 7850 4400 50  0001 C CNN "Notes"
-F 9 "I.52" H 7850 4400 50  0001 C CNN "DK line"
+F 9 "I.9" H 7850 4400 50  0001 C CNN "DK line"
 	1    7850 4400
 	0    1    1    0
@@
 AR Path="/5F7EFEA4/5F8B0DF1/5F88DC3C" Ref="#PWR025"  Part="1"
 AR Path="/5F8C3863/5F8AE34F/5F88DC3C" Ref="#PWR036"  Part="1"
-F 0 "#PWR025" H 7450 3800 50  0001 C CNN
+F 0 "#PWR038" H 7450 3800 50  0001 C CNN
 F 1 "V+" H 7450 4090 50  0000 C CNN
 F 2 "" H 7450 3950 50  0001 C CNN
@@
 AR Path="/5F7EFEA4/5F8B0DF1/5F88E156" Ref="#PWR035"  Part="1"
 AR Path="/5F8C3863/5F8AE34F/5F88E156" Ref="#PWR037"  Part="1"
-F 0 "#PWR035" H 7500 4800 50  0001 C CNN
+F 0 "#PWR039" H 7500 4800 50  0001 C CNN
 F 1 "V-" H 7500 4910 50  0000 C CNN
 F 2 "" H 7500 5050 50  0001 C CNN

Commit message: BOM change to dac/, start of board revision in input/adc.sch
dac: changed 10 Ohm MPN on BOM

input:
Fixed SOIC-8 footprints
Got rid of bootstrapping of the reference buffer.  Now it runs from the 10 Ohm/330 uF filtered +8/-6.
Changed power input beads from 22 Ohm to 180 Ohm.
Added diode clamp between GND and Earth grounds.
Changed reference buffer to dual opamp.
Parts:
- R107, R108, R109: Digikey 541-10TACT-ND -> RHM10KCT-ND
Changed lines of the file:
@@
 F 5 "ESR10EZPJ100" H 7100 4400 50  0001 C CNN "MPN"
 F 6 "Rohm Semiconductor" H 7100 4400 50  0001 C CNN "Manufacturer"
-F 7 "541-10TACT-ND" H 7100 4400 50  0001 C CNN "Digikey"
+F 7 "RHM10KCT-ND" H 7100 4400 50  0001 C CNN "Digikey"
 F 8 "Thick film surge resist" H 7100 4400 50  0001 C CNN "Notes"
 F 9 "I.9" H 7100 4400 50  0001 C CNN "DK line"
@@
 F 5 "ESR10EZPJ100" H 6350 2600 50  0001 C CNN "MPN"
 F 6 "Rohm Semiconductor" H 6350 2600 50  0001 C CNN "Manufacturer"
-F 7 "541-10TACT-ND" H 6350 2600 50  0001 C CNN "Digikey"
+F 7 "RHM10KCT-ND" H 6350 2600 50  0001 C CNN "Digikey"
 F 8 "Thick film surge resist" H 6350 2600 50  0001 C CNN "Notes"
 F 9 "I.9" H 6350 2600 50  0001 C CNN "DK line"
@@
 F 5 "ESR10EZPJ100" H 7850 4400 50  0001 C CNN "MPN"
 F 6 "Rohm Semiconductor" H 7850 4400 50  0001 C CNN "Manufacturer"
-F 7 "541-10TACT-ND" H 7850 4400 50  0001 C CNN "Digikey"
+F 7 "RHM10KCT-ND" H 7850 4400 50  0001 C CNN "Digikey"
 F 8 "Thick film surge resist" H 7850 4400 50  0001 C CNN "Notes"
 F 9 "I.9" H 7850 4400 50  0001 C CNN "DK line"
