File: dac/dac.sch (KiCad schematic (older format))
At the start: 10 parts, among them U151 PCM1794A

Commit message: Mainly BOM tweaks, working on setting up more systematic database of parts and BOMs in parts/
Parts:
- R152, R153: DK line I.52 -> I.9; Description RES SMD 10 OHM 5% 1/2W 0805 -> RES SMD 10 OHM 5% 0.4W 0805; MPN CRCW080510R0JNEAHP -> ESR10EZPJ100; Manufacturer Vishay Dale -> Rohm Semiconductor
Changed lines of the file:
@@
 F 1 "10" V 5200 3350 50  0000 C CNN
 F 2 "Resistor_SMD:R_0805_2012Metric" V 5340 3340 50  0001 C CNN
-F 3 "http://www.vishay.com/docs/20043/crcwhpe3.pdf" H 5300 3350 50  0001 C CNN
+F 3 "https://www.rohm.com/datasheet/ESR01MZPF/esr-e" H 5300 3350 50  0001 C CNN
 F 4 "541-10TACT-ND" H 5300 3350 50  0001 C CNN "Digikey"
-F 5 "I.52" H 5300 3350 50  0001 C CNN "DK line"
-F 6 "RES SMD 10 OHM 5% 1/2W 0805" H 5300 3350 50  0001 C CNN "Description"
-F 7 "CRCW080510R0JNEAHP" H 5300 3350 50  0001 C CNN "MPN"
-F 8 "Vishay Dale" H 5300 3350 50  0001 C CNN "Manufacturer"
+F 5 "I.9" H 5300 3350 50  0001 C CNN "DK line"
+F 6 "RES SMD 10 OHM 5% 0.4W 0805" H 5300 3350 50  0001 C CNN "Description"
+F 7 "ESR10EZPJ100" H 5300 3350 50  0001 C CNN "MPN"
+F 8 "Rohm Semiconductor" H 5300 3350 50  0001 C CNN "Manufacturer"
 F 9 "Thick film surge resist" H 5300 3350 50  0001 C CNN "Notes"
 	1    5300 3350
@@
 F 1 "10" V 5200 3000 50  0000 C CNN
 F 2 "Resistor_SMD:R_0805_2012Metric" V 5340 2990 50  0001 C CNN
-F 3 "http://www.vishay.com/docs/20043/crcwhpe3.pdf" H 5300 3000 50  0001 C CNN
+F 3 "https://www.rohm.com/datasheet/ESR01MZPF/esr-e" H 5300 3000 50  0001 C CNN
 F 4 "541-10TACT-ND" H 5300 3000 50  0001 C CNN "Digikey"
-F 5 "I.52" H 5300 3000 50  0001 C CNN "DK line"
-F 6 "RES SMD 10 OHM 5% 1/2W 0805" H 5300 3000 50  0001 C CNN "Description"
-F 7 "CRCW080510R0JNEAHP" H 5300 3000 50  0001 C CNN "MPN"
-F 8 "Vishay Dale" H 5300 3000 50  0001 C CNN "Manufacturer"
+F 5 "I.9" H 5300 3000 50  0001 C CNN "DK line"
+F 6 "RES SMD 10 OHM 5% 0.4W 0805" H 5300 3000 50  0001 C CNN "Description"
+F 7 "ESR10EZPJ100" H 5300 3000 50  0001 C CNN "MPN"
+F 8 "Rohm Semiconductor" H 5300 3000 50  0001 C CNN "Manufacturer"
 F 9 "Thick film surge resist" H 5300 3000 50  0001 C CNN "Notes"
 	1    5300 3000
@@
 AR Path="/5F7EFEA4/5F9ED561" Ref="#PWR0113"  Part="1"
 AR Path="/5F8C3863/5F9ED561" Ref="#PWR0117"  Part="1"
-F 0 "#PWR0113" H 3600 3050 50  0001 C CNN
+F 0 "#PWR0117" H 3600 3050 50  0001 C CNN
 F 1 "VCC" H 3600 3350 50  0000 C CNN
 F 2 "" H 3600 3200 50  0001 C CNN
@@
 AR Path="/5F7EFEA4/5F9F1229" Ref="#PWR0116"  Part="1"
 AR Path="/5F8C3863/5F9F1229" Ref="#PWR0125"  Part="1"
-F 0 "#PWR0116" H 3100 6000 50  0001 C CNN
+F 0 "#PWR0125" H 3100 6000 50  0001 C CNN
 F 1 "VCC" H 3100 6300 50  0000 C CNN
 F 2 "" H 3100 6150 50  0001 C CNN
@@
 AR Path="/5F7EFEA4/5F8A8A2A" Ref="#PWR0146"  Part="1"
 AR Path="/5F8C3863/5F8A8A2A" Ref="#PWR0151"  Part="1"
-F 0 "#PWR0146" H 4700 4950 50  0001 C CNN
+F 0 "#PWR0151" H 4700 4950 50  0001 C CNN
 F 1 "GND" H 4700 5050 50  0000 C CNN
 F 2 "" H 4700 5200 50  0001 C CNN
@@
 AR Path="/5F7EFEA4/5F8AA834" Ref="#PWR0147"  Part="1"
 AR Path="/5F8C3863/5F8AA834" Ref="#PWR0152"  Part="1"
-F 0 "#PWR0147" H 3600 4800 50  0001 C CNN
+F 0 "#PWR0152" H 3600 4800 50  0001 C CNN
 F 1 "GND" H 3600 4900 50  0000 C CNN
 F 2 "" H 3600 5050 50  0001 C CNN
@@
 AR Path="/5F7EFEA4/5F8AABB7" Ref="#PWR0148"  Part="1"
 AR Path="/5F8C3863/5F8AABB7" Ref="#PWR0153"  Part="1"
-F 0 "#PWR0148" H 2800 3800 50  0001 C CNN
+F 0 "#PWR0153" H 2800 3800 50  0001 C CNN
 F 1 "GND" H 2800 3900 50  0000 C CNN
 F 2 "" H 2800 4050 50  0001 C CNN
@@
 AR Path="/5F7EFEA4/5F8AB0BD" Ref="#PWR0149"  Part="1"
 AR Path="/5F8C3863/5F8AB0BD" Ref="#PWR0154"  Part="1"
-F 0 "#PWR0149" H 4550 6650 50  0001 C CNN
+F 0 "#PWR0154" H 4550 6650 50  0001 C CNN
 F 1 "GND" H 4550 6750 50  0000 C CNN
 F 2 "" H 4550 6900 50  0001 C CNN
@@
 AR Path="/5F7EFEA4/5F8AB4CB" Ref="#PWR0150"  Part="1"
 AR Path="/5F8C3863/5F8AB4CB" Ref="#PWR0155"  Part="1"
-F 0 "#PWR0150" H 3100 6200 50  0001 C CNN
+F 0 "#PWR0155" H 3100 6200 50  0001 C CNN
 F 1 "GND" H 3100 6300 50  0000 C CNN
 F 2 "" H 3100 6450 50  0001 C CNN

Commit message: BOM change to dac/, start of board revision in input/adc.sch
dac: changed 10 Ohm MPN on BOM

input:
Fixed SOIC-8 footprints
Got rid of bootstrapping of the reference buffer.  Now it runs from the 10 Ohm/330 uF filtered +8/-6.
Changed power input beads from 22 Ohm to 180 Ohm.
Added diode clamp between GND and Earth grounds.
Changed reference buffer to dual opamp.
Parts:
- R152, R153: Digikey 541-10TACT-ND -> RHM10KCT-ND
Changed lines of the file:
@@
 F 2 "Resistor_SMD:R_0805_2012Metric" V 5340 3340 50  0001 C CNN
 F 3 "https://www.rohm.com/datasheet/ESR01MZPF/esr-e" H 5300 3350 50  0001 C CNN
-F 4 "541-10TACT-ND" H 5300 3350 50  0001 C CNN "Digikey"
+F 4 "RHM10KCT-ND" H 5300 3350 50  0001 C CNN "Digikey"
 F 5 "I.9" H 5300 3350 50  0001 C CNN "DK line"
 F 6 "RES SMD 10 OHM 5% 0.4W 0805" H 5300 3350 50  0001 C CNN "Description"
@@
 F 2 "Resistor_SMD:R_0805_2012Metric" V 5340 2990 50  0001 C CNN
 F 3 "https://www.rohm.com/datasheet/ESR01MZPF/esr-e" H 5300 3000 50  0001 C CNN
-F 4 "541-10TACT-ND" H 5300 3000 50  0001 C CNN "Digikey"
+F 4 "RHM10KCT-ND" H 5300 3000 50  0001 C CNN "Digikey"
 F 5 "I.9" H 5300 3000 50  0001 C CNN "DK line"
 F 6 "RES SMD 10 OHM 5% 0.4W 0805" H 5300 3000 50  0001 C CNN "Description"
